File: roam.kicad_pcb (KiCad board)
At the start: 4 copper layers, 100 x 60 mm, 110 parts, among them J1 nanoSIM-holder, J3 U.FL-R-SMT-1-GNSS_ANT, J4 U.FL-R-SMT-1-RF_ANT, J6 BAT, J7 MX23A18NF2, Q1 BC846A,215, Q2 BC846A,215, U1 SIP32408DNP-T1-GE4, U10 MCP2515-xST, U11 MCP2515-xST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

Commit message: Added DC booster
Parts:
- removed J6: BAT, Connector_JST:JST_GH_SM03B-GHS-TB_1x03-1MP_P1.25mm_Horizontal
- added C18: 1uF, Capacitor_SMD:C_0603_1608Metric, F.Cu at (116.5, 117.2)
- added C19: 1uF, Capacitor_SMD:C_0603_1608Metric, F.Cu at (119.6, 117.2)
- added C21: 18pF, Capacitor_SMD:C_0603_1608Metric, F.Cu at (172.7, 141.6)
- added C24: 22uF, Capacitor_SMD:C_0805_2012Metric, F.Cu at (127.4, 99.0)
- added C25: 22uF, Capacitor_SMD:C_0805_2012Metric, F.Cu at (139.5, 109.4)
- added C28: 22uF, Capacitor_SMD:C_0805_2012Metric, F.Cu at (141.6, 109.4)
- added C30: 22uF, Capacitor_SMD:C_0805_2012Metric, F.Cu at (139.5, 105.8)
- added D8: LED, LED_SMD:LED_0603_1608Metric, F.Cu at (122.2, 120.8)
- added J2: Battery, Connector_Molex:Molex_PicoBlade_53047-0310_1x03_P1.25mm_Vertical, F.Cu at (117.0, 89.2)
- added L3: 1.5uH, Inductor_SMD:L_Bourns-SRN4018, F.Cu at (122.5, 104.2)
- added R17: 1k1, Resistor_SMD:R_0603_1608Metric, F.Cu at (114.7, 119.2)
- added R23: DNP, Resistor_SMD:R_0603_1608Metric, F.Cu at (114.7, 120.7)
- added R26: 1k5, Resistor_SMD:R_0603_1608Metric, F.Cu at (122.2, 119.2)
- added R27: DNP, Resistor_SMD:R_0603_1608Metric, F.Cu at (229.7, 66.4)
- added R28: 10k, Resistor_SMD:R_0603_1608Metric, F.Cu at (226.6, 62.9)
- added R29: 10k, Resistor_SMD:R_0603_1608Metric, F.Cu at (229.7, 70.0)
- added R30: 93k1, Resistor_SMD:R_0603_1608Metric, F.Cu at (131.2, 101.8)
- added R33: 348k, Resistor_SMD:R_0603_1608Metric, F.Cu at (132.9, 94.3)
- added R34: 71.5k, Resistor_SMD:R_0603_1608Metric, F.Cu at (132.9, 96.9)
- added TH1: 10k (103A), Resistor_SMD:R_0603_1608Metric, F.Cu at (121.5, 89.5)
- added U18: MP3423, TC-Power:MP3423, F.Cu at (126.2, 109.3)
- added U8: BQ24040DSQR, TC-Power:BQ24040DSQR, F.Cu at (118.3, 120.1)
- added Y2: 16MHz, Crystal:Crystal_SMD_Abracon_ABM8G-4Pin_3.2x2.5mm, F.Cu at (172.7, 139.1)
- C22: value 100nF -> 18pF
- C23: value 100nF -> 22uF; footprint Capacitor_SMD:C_0603_1608Metric -> Capacitor_SMD:C_0805_2012Metric
- C31: value 10uF -> 22uF; footprint Capacitor_SMD:C_1206_3216Metric -> Capacitor_SMD:C_0805_2012Metric
- R14: value 10k -> 0
- R15: value 10k -> 100k
- moved F1 148.1 mm to (114.9, 124.8)
- moved C31 127.7 mm to (141.6, 105.8)
- moved U4 104.7 mm to (192.0, 118.8)
- moved R18 96.4 mm to (162.5, 142.2), turned to 180 degrees
- moved C23 89.6 mm to (124.6, 94.6)
- moved C4 86.7 mm to (158.7, 93.7)
- moved C5 86.7 mm to (158.7, 98.1)
- moved CP1 86.7 mm to (155.5, 96.2)
- moved CP2 86.7 mm to (151.7, 96.2)
- moved CP3 86.7 mm to (147.9, 96.2)
- moved FB1 86.7 mm to (144.7, 96.9)
- moved J1 81.1 mm to (192.4, 129.5)
- moved U16 80.2 mm to (157.1, 132.8), turned to 180 degrees
- moved U2 79.4 mm to (191.7, 108.3)
- moved R15 78.8 mm to (127.2, 101.8)
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Connections:
- C16 pad 1: /CAN_OSC1 -> /CAN_250_OSC_1
- C17 pad 1: /CAN_OSC2 -> /CAN_250_OSC_2
- C20 pad 1: +100V -> /100V
- C22 pad 1: GND -> /CAN_500_OSC_2
- C22 pad 2: 3V3_CAN -> GND
- C23 pad 1: GND -> CHG_BAT
- C23 pad 2: 3V3_CAN -> GND
- C26 pad 1: +100V -> /100V
- C27 pad 1: +100V -> /100V
- C31 pad 1: VBAT -> 4V7_BOOST
- C36 pad 1: 4V0 -> 5V0
- F1 pad 1: VBAT -> +100V
- F1 pad 2: Net-(F1-Pad2) -> /100V
- R15 pad 1: Net-(R15-Pad1) -> CHG_BAT
- R15 pad 2: /CAN_CS -> Net-(R15-Pad2)
- R18 pad 1: Net-(R18-Pad1) -> /CS_INT
- R19 pad 1: VBAT -> CHG_BAT
- R21 pad 1: +100V -> /100V
- R46 pad 1: 4V0 -> 5V0
- U10 pad 18: Net-(R15-Pad1) -> /CS_INT
- U10 pad 3: /CAN_CLK_CHAIN -> unconnected-(U10-Pad3)
- U10 pad 8: /CAN_OSC2 -> /CAN_500_OSC_2
- U10 pad 9: /CAN_OSC1 -> /CAN_500_OSC_1
- U11 pad 18: Net-(R18-Pad1) -> /CS_INT
- U11 pad 3: /CAN_CLK_CHAIN -> unconnected-(U11-Pad3)
- U11 pad 8: /CAN_OSC2 -> /CAN_250_OSC_2
- U11 pad 9: /CAN_OSC1 -> /CAN_250_OSC_1
- U12 pad 1: 4V0 -> 5V0
- U4 pad GND: (no net) -> GND
- U6 pad 3: +100V -> /100V
- U7 pad 5: unconnected-(U7-Pad5) -> Net-(R27-Pad2)
- U9 pad 5: unconnected-(U9-Pad5) -> Net-(R29-Pad1)
- Y1 pad 1: /CAN_OSC1 -> /CAN_250_OSC_1
- Y1 pad 3: /CAN_OSC2 -> /CAN_250_OSC_2
Routing:
- net /NTC: track 0.00 -> 43.1 mm, vias 0 -> 2
- net 5V0_BUCK: track 16.3 -> 56.0 mm, vias 2 -> 17
- net CHG_BAT: track 0.00 -> 35.7 mm, vias 0 -> 4
- net /100V: track 0.00 -> 27.2 mm, vias 0 -> 2
- net +100V: track 27.6 -> 3.63 mm, vias 2 -> 0
- net Net-(D8-Pad1): track 0.00 -> 2.53 mm
- net Net-(R17-Pad1): track 0.00 -> 1.94 mm
- net Net-(R23-Pad1): track 0.00 -> 1.82 mm
- net Net-(D8-Pad2): track 0.00 -> 1.60 mm
- net GND: track 0.00 -> 1.05 mm, vias 58 -> 80
- net /3423_SW: vias 0 -> 8
- added copper zone on F.Cu, net /100V
- added copper zone on B.Cu, net /3423_SW
- added copper zone on F.Cu, net /3423_SW
- added copper zone on F.Cu, net 4V0_MODEM
- added copper zone on F.Cu, net 4V7_BOOST
- added copper zone on B.Cu, net 5V0_BUCK
- added copper zone on F.Cu, net CHG_BAT
- removed copper zone on F.Cu, net +100V

Commit message: Save
Parts:
- moved R27 112.1 mm to (142.9, 137.3)
- moved R29 111.8 mm to (142.9, 140.5)
- moved U7 111.8 mm to (139.8, 135.7)
- moved R28 111.2 mm to (147.6, 141.2)
- moved U9 107.3 mm to (139.8, 132.8)
- moved R14 104.0 mm to (146.8, 134.3)
- moved C45 56.5 mm to (185.4, 98.6), turned to 180 degrees
- moved C44 53.9 mm to (185.3, 100.2), turned to 180 degrees
- moved U13 51.7 mm to (188.7, 99.4), turned to 180 degrees
- moved R37 50.4 mm to (191.8, 98.6), turned to 180 degrees
- moved R38 47.5 mm to (191.8, 100.2), turned to 180 degrees
- moved R23 38.0 mm to (132.9, 87.3), turned to 0 degrees
- moved R17 35.4 mm to (132.9, 88.8), turned to 0 degrees
- moved U8 34.0 mm to (129.3, 87.9), turned to 180 degrees
- moved D8 33.8 mm to (125.4, 87.2), turned to 180 degrees
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- renumbered J7 to locked
Routing:
- net Net-(R33-Pad1): track 0.00 -> 32.6 mm, vias 0 -> 2
- net /NTC: track 43.1 -> 18.4 mm, vias 2 -> 1
- net CHG_BAT: track 35.7 -> 52.8 mm, vias 4 -> 6
- net 5V0_BUCK: track 56.0 -> 67.8 mm, vias 17 -> 11
- net Net-(R15-Pad2): track 0.00 -> 8.19 mm, vias 0 -> 2
- net 3V3_ALWAYS_ON: track 0.00 -> 4.83 mm
- net 4V7_BOOST: track 0.00 -> 4.42 mm
- net 5V0: track 0.00 -> 3.86 mm
- net Net-(L5-Pad1): track 0.00 -> 2.99 mm
- net Net-(R46-Pad2): track 0.00 -> 1.96 mm
- net GND: vias 80 -> 92

Commit message: Routing
Parts:
- added C35: 47uF, Inductor_SMD:L_1206_3216Metric, F.Cu at (130.9, 106.3)
- added C37: 100nF, Inductor_SMD:L_0603_1608Metric, F.Cu at (130.2, 104.3)
- added C39: 33pF, Inductor_SMD:L_0402_1005Metric, F.Cu at (124.0, 105.7)
- added C42: 22uF, Inductor_SMD:L_0805_2012Metric, F.Cu at (133.9, 96.5)
- added C43: 22uF, Inductor_SMD:L_0805_2012Metric, F.Cu at (130.3, 96.5)
- added C50: 22uF, Inductor_SMD:L_0805_2012Metric, F.Cu at (133.9, 94.7)
- added C51: 22uF, Inductor_SMD:L_0805_2012Metric, F.Cu at (130.3, 94.7)
- added C52: 100nF, Inductor_SMD:L_0603_1608Metric, F.Cu at (130.0, 98.2)
- added L4: 2.2uH, Inductor_SMD:L_Bourns-SRN4018, F.Cu at (133.8, 100.0)
- added R35: 10k, Resistor_SMD:R_0603_1608Metric, F.Cu at (176.7, 142.3)
- added R36: 100k, Inductor_SMD:L_0603_1608Metric, F.Cu at (124.9, 102.0)
- added R39: 34.8k, Inductor_SMD:L_0603_1608Metric, F.Cu at (123.3, 102.0)
- added R40: 169k, Inductor_SMD:L_0603_1608Metric, F.Cu at (124.1, 104.3)
- added R41: 30k, Inductor_SMD:L_0603_1608Metric, F.Cu at (127.1, 104.3)
- added U19: SN74AHC1G04DBVR, Package_TO_SOT_SMD:SOT-23-5, F.Cu at (186.4, 139.6)
- added U20: TPS566242DRLR, TC-Power:TPS566242DRLR, F.Cu at (129.0, 101.3)
- moved Z1 152.6 mm to (114.5, 101.6), turned to 180 degrees
- moved R20 92.4 mm to (121.0, 91.8)
- moved J3 91.9 mm to (170.7, 92.2), turned to -90 degrees
- moved R19 89.4 mm to (122.6, 91.8), turned to -90 degrees
- moved C10 88.2 mm to (170.3, 95.5), turned to 180 degrees
- moved J4 88.2 mm to (163.4, 92.1), turned to -90 degrees
- moved R6 88.0 mm to (143.0, 105.9), turned to 90 degrees
- moved C7 86.6 mm to (174.0, 96.0), turned to 90 degrees
- moved C8 86.4 mm to (171.2, 98.6)
- moved R1 82.1 mm to (175.0, 129.9)
- moved R2 81.6 mm to (175.0, 128.3)
- moved R3 81.3 mm to (175.0, 126.7)
- moved C14 80.4 mm to (180.9, 100.2), turned to 90 degrees
- moved C6 80.3 mm to (181.3, 113.4)
- moved D2 78.0 mm to (140.4, 99.9), turned to -90 degrees
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Connections:
- C1 pad 1: 3V3 -> 3V3_ALWAYS_ON
- D1 pad 4: /SIM_CHIP_CLK -> /SIM_CHIP_DATA
- D1 pad 5: /SIM_CHIP_DATA -> /SIM_CHIP_CLK
- R18 pad 1: /CS_INT -> Net-(R18-Pad1)
- R18 pad 2: /CAN_CS -> /CAN_CS_250
- R31 pad 1: 12V -> 5V0_BUCK
- U1 pad 1: 3V3 -> 3V3_ALWAYS_ON
- U10 pad 14: /CAN_SCK -> /CAN_SCK_500
- U10 pad 16: /CAN_MOSI -> /CAN_MOSI_500
- U10 pad 17: /CAN_MISO -> /CAN_MISO_500
- U10 pad 18: /CS_INT -> Net-(U10-Pad18)
- U11 pad 14: /CAN_SCK -> /CAN_SCK_250
- U11 pad 16: /CAN_MOSI -> /CAN_MOSI_250
- U11 pad 17: /CAN_MISO -> /CAN_MISO_250
- U11 pad 18: /CS_INT -> Net-(R18-Pad1)
- U14 pad 3: /~{P_EN} -> /~{ACC_EN}
- U15 pad 3: /P0.00 -> /CAN_EN
- U16 pad 8: unconnected-(U16-Pad8) -> /CAN_SHDN
- U17 pad 8: unconnected-(U17-Pad8) -> /CAN_SHDN
- U2 pad 10: /P0.29_AIN5 -> unconnected-(U2-Pad10)
- U2 pad 11: /P0.02_AIN0 -> unconnected-(U2-Pad11)
- U2 pad 13: /P0.28_AIN4 -> /CAN_INT_500
- U2 pad 16: /I2C1_SCL -> /SCL
- U2 pad 17: /SERIAL_TX -> /AUX_LED
- U2 pad 18: /SERIAL_RX -> /CAN_EN
- U2 pad 19: /I2C1_SDA -> /SDA
- U2 pad 20: /P0.04_AIN2 -> unconnected-(U2-Pad20)
- U2 pad 21: /P0.05_AIN3 -> unconnected-(U2-Pad21)
- U2 pad 22: /AUX_LED -> unconnected-(U2-Pad22)
- U2 pad 25: /~{CE} -> unconnected-(U2-Pad25)
- U2 pad 26: /CAN_INT -> unconnected-(U2-Pad26)
- U2 pad 29: /P0.12 -> /CAN_SCK_250
- U2 pad 3: /CONN_LED -> /NET_LED
- U2 pad 36: /CAN_MISO -> /CAN_MOSI_250
- U2 pad 37: /CAN_SCK -> /CAN_MISO_250
- U2 pad 38: /I2C2_SDA -> /CAN_MISO_500
- U2 pad 39: /CAN_MOSI -> /CAN_SCK_500
- U2 pad 4: /NET_LED -> /STATUS_LED_3V3
- U2 pad 41: /I2C2_SCL -> /CAN_MOSI_500
- U2 pad 49: /ACC_INT -> unconnected-(U2-Pad49)
- U2 pad 5: /GPS_ANT_EN -> /NRF_LED
- U2 pad 50: /CAN_CS -> /CAN_CS_500
- U2 pad 57: /~{PE} -> /MODEM_RI_3V3
- U2 pad 58: /STATUS_LED_3V3 -> /CONN_LED
- U2 pad 6: /P1.13 -> /GPS_ANT_EN
- U2 pad 61: /P1.01 -> /CAN_CS_250
- U2 pad 7: /NRF_LED -> /~{ACC_EN}
- U2 pad 8: /MODEM_RI_3V3 -> /ACC_INT
- U2 pad 9: /P0.03_AIN1 -> /CAN_INT_250
- locked pad 15: /USB_D- -> unconnected-(J7-Pad15)
- locked pad 16: /USB_D+ -> unconnected-(J7-Pad16)
- locked pad 17: /VUSB -> unconnected-(J7-Pad17)
Routing:
- net 3V3_ALWAYS_ON: track 4.83 -> 177.3 mm, vias 0 -> 8
- net /SWDIO: track 0.00 -> 139.0 mm, vias 0 -> 6
- net /SWDCLK: track 0.00 -> 133.8 mm, vias 0 -> 5
- net 5V0: track 3.86 -> 106.1 mm, vias 0 -> 8
- net /IBL: track 0.00 -> 77.7 mm, vias 0 -> 5
- net /CAN_500_L: track 0.00 -> 73.6 mm, vias 0 -> 3
- net /CAN_500_H: track 0.00 -> 73.1 mm, vias 0 -> 3
- net /EBL: track 0.00 -> 67.8 mm, vias 0 -> 4
- net /NRESET: track 0.00 -> 65.3 mm, vias 0 -> 3
- net /CAN_CS_250: track 0.00 -> 63.7 mm, vias 0 -> 3
- net 3V3_CAN: track 0.00 -> 62.1 mm, vias 0 -> 8
- net /CAN_INT_250: track 0.00 -> 61.4 mm, vias 0 -> 3
- net /CAN_EN: track 0.00 -> 60.1 mm, vias 0 -> 4
- net /CAN_250_H: track 0.00 -> 55.5 mm, vias 0 -> 3
- net 1V8: track 0.00 -> 55.2 mm, vias 0 -> 5
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- added copper zone on F.Cu, net 5V0

Commit message: Routed
Parts:
- added C53: 1nF, Capacitor_SMD:C_0603_1608Metric, F.Cu at (115.5, 95.0)
- added D9: 3v3, Diode_SMD:D_0603_1608Metric, F.Cu at (113.9, 95.0)
- added R42: 10k, Resistor_SMD:R_0603_1608Metric, F.Cu at (113.9, 98.1)
- added R43: 3.9k, Resistor_SMD:R_0603_1608Metric, F.Cu at (115.5, 98.1)
- U20: value TPS566242DRLR -> SOT5x3_DRL_TEX
- U8: value BQ24040DSQR -> DSQ10_P9X1P5
- moved J1 0.30 mm to (193.0, 128.7)
Connections:
- net CHG_BAT renamed VBAT
- C14 pad 1: 3.3V -> 3V3_ALWAYS_ON
- C6 pad 1: 3V3 -> 3V3_ALWAYS_ON
- U2 pad 10: unconnected-(U2-Pad10) -> /IGN_IN_3V3
- U2 pad 28: 3V3 -> 3V3_ALWAYS_ON
- U3 pad 24: /USB_VBUS -> unconnected-(U3-Pad24)
- U3 pad 27: /USB_D+ -> unconnected-(U3-Pad27)
- U3 pad 28: /USB_D- -> unconnected-(U3-Pad28)
- U4 pad 8: 3V3 -> 3V3_ALWAYS_ON
- U5 pad 19: 3.3V -> 3V3_ALWAYS_ON
Routing:
- net /IGN_IN_3V3: track 0.00 -> 91.2 mm, vias 0 -> 5
- net 3V3_ALWAYS_ON: track 177.3 -> 205.6 mm, vias 8 -> 11
- net /IGN_IN_12V: track 0.00 -> 18.4 mm, vias 0 -> 2
- net 3V3: track 17.2 -> 0.00 mm, vias 2 -> 0
- net 3.3V: track 7.61 -> 0.00 mm
- net +100V: track 0.00 -> 3.49 mm
- net 5V0_BUCK: track 89.0 -> 90.9 mm
- net /FLASH_SCK: track 8.36 -> 7.01 mm
- net /ACC_INT: track 8.98 -> 10.3 mm
- net /STATUS_LED_3V3: track 26.8 -> 28.1 mm
- net /MODEM_RI_3V3: track 18.0 -> 19.2 mm
- net /CAN_MOSI_500: track 32.9 -> 34.0 mm
- net /SIM_CHIP_CLK: track 25.7 -> 24.6 mm
- net /CAN_SCK_500: track 33.8 -> 34.8 mm
- net 3V3_CAN: track 62.1 -> 61.2 mm
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
Commit message: Routing
Parts:
- U20: value SOT5x3_DRL_TEX -> TPS566242DRLR
- U8: value DSQ10_P9X1P5 -> BQ24040DSQR
- moved J4 4.55 mm to (160.5, 88.6)
- moved J3 3.63 mm to (171.2, 88.6)
Routing:
- net Net-(D6-Pad1): track 3.05 -> 7.62 mm
- net Net-(C10-Pad1): track 3.84 -> 7.64 mm
- net GND: vias 92 -> 529
- net /NRESET: vias 3 -> 4
