File: roam.kicad_pcb (KiCad board)
At the start: 4 copper layers, 100 x 60 mm, 226 parts, among them IC2 MCP73833T-FCI/MF, J1 SIM8060-6-0-14-00-A, J2 Battery, Q1 BC846A,215, Q2 BC846A,215, U1 SIP32408DNP-T1-GE4, U11 W25N512GVEIG, U12 LM3671MF-3.3/NOPB, U13 LIS2DH12TR, U14 MAX17643ATC+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

Commit message: Fullfill the info for all components
Parts:
- C73, C78, C79: value 0.1uF -> 100nF
- U16, U6: value MCP2562-E-MF -> MCP2562-E/MF
- U18: value MP3423 -> MP3423GG
- U3: value SIMCOM-7000G -> SIM7000G
- U7, U9: value LM66100 -> LM66100DCKR
- U8: value MAX2659ELT -> MAX2659ELT+T

Commit message: reday to produce
Parts:
- removed D6: D_Schottky, Package_TO_SOT_SMD:TO-277A_alt
- added D23: MM3Z18VT1G, Diode_SMD:D_SOD-323F, B.Cu at (119.0, 139.6)
- added R61: 20k, Resistor_SMD:R_1206_3216Metric, B.Cu at (117.2, 135.2)
- added R62: 220k, Resistor_SMD:R_0805_2012Metric, B.Cu at (116.3, 139.6)
- added U15: FDMC86139P, TC-ICs:WDFN8-511DH-O_3p3x3p3x0p65_OSI, B.Cu at (112.3, 135.3)
- turned L9 to 180 degrees
Connections:
- L9 pad 1: Net-(U14-LX) -> 5V0_BUCK
- L9 pad 2: 5V0_BUCK -> Net-(U14-LX)
Routing:
- net Net-(D23-A): track 0.00 -> 28.3 mm
- net /EBL_60V: track 15.1 -> 30.7 mm
- net 3V3_ALWAYS_ON: track 319.1 -> 318.4 mm
- net GND: vias 448 -> 454
- removed copper zone on B.Cu, net /EBL_60V
Other:
- board text added: "ROAM P6"
- board text removed: "ROAM P5"

Commit message: Fixed production issue
Routing:
- net GND: vias 454 -> 452
Changed lines of the file:
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@@
   (via (at 103 143.5) (size 0.5) (drill 0.3) (layers "F.Cu" "B.Cu") (free) (net 2))
   (via (at 179.5 119) (size 0.5) (drill 0.3) (layers "F.Cu" "B.Cu") (free) (net 2))
-  (via (at 119.1 139.6) (size 0.5) (drill 0.3) (layers "F.Cu" "B.Cu") (free) (net 2))
   (via (at 118.125 105.975) (size 0.5) (drill 0.3) (layers "F.Cu" "B.Cu") (free) (net 2))
   (via (at 177.5 85.6) (size 0.5) (drill 0.3) (layers "F.Cu" "B.Cu") (free) (net 2))
@@
   (via (at 127.45 134.55) (size 0.5) (drill 0.3) (layers "F.Cu" "B.Cu") (free) (net 2))
   (via (at 173.5 144.43) (size 0.5) (drill 0.3) (layers "F.Cu" "B.Cu") (free) (net 2))
-  (via (at 107.25 127.35) (size 0.5) (drill 0.3) (layers "F.Cu" "B.Cu") (free) (net 2))
   (via (at 132.22 93.69) (size 0.5) (drill 0.3) (layers "F.Cu" "B.Cu") (free) (net 2))
   (via (at 124.9 132.9) (size 0.5) (drill 0.3) (layers "F.Cu" "B.Cu") (free) (net 2))
