File: roam.kicad_sch (KiCad schematic)
At the start: 148 parts, among them J1 nanoSIM-holder, J2 Battery, J3 U.FL-R-SMT-1-GNSS_ANT, J4 U.FL-R-SMT-1-RF_ANT, J7 MX23A18NF2, Q1 BC846A,215, Q2 BC846A,215, U1 SIP32408DNP-T1-GE4, U10 MCP2515-xST, U11 MCP2515-xST, U12 LM3671MF-3.3/NOPB, U13 LIS2DH12TR, U14 SiP32408, U15 SiP32408, U16 MCP2562-E-MF, U17 MCP2562-E-MF, U18 MP3423, U19 SN74AHC1G04DBVR, U2 MDBT50Q-1M, U20 TPS566242DRLR, U3 SIMCOM-7000G, U4 MX25L3233FZBI-08Q, U5 TXB0108PWR, U6 MP9486A, U7 LM66100, U8 BQ24040DSQR, U9 LM66100, Y1 16MHz, Y2 16MHz

Commit message: Routed
Parts:
- added C53: 1nF, Capacitor_SMD:C_0603_1608Metric, symbol Device:C
- added D9: 3v3, Diode_SMD:D_0603_1608Metric, symbol Device:D_Zener
- added R42: 10k, Resistor_SMD:R_0603_1608Metric, symbol Device:R_Small
- added R43: 3.9k, Resistor_SMD:R_0603_1608Metric, symbol Device:R_Small
Connections:
- net 3.3V is gone; now on net 3V3_ALWAYS_ON: C14.1, U5.19 (VCCB)
- net 3V3 is gone; now on net 3V3_ALWAYS_ON: C6.1, U2.28 (VDD), U4.8 (VCC)
- net GND: now also C53.2, D9.2 (A), R43.2
- net IGN_IN_12V: now also R42.1
- net IGN_IN_3V3: now reaches U2.10 (P0.29/AIN5)
- net IGN_IN_3V3: now also C53.1, D9.1 (K), R42.2, R43.1
- net CHG_BAT renamed VBAT
- net USB_D+: no longer names the net of U3.27 (USB_D+)
- net USB_D-: no longer names the net of U3.28 (USB_D-)
- net USB_VBUS: no longer names the net of U3.24 (USB_VBUS)
- no-connect marks 52 -> 54

Commit message: Routing
Other:
- moved on the sheet: J3, J4

Commit message: Component selection in progress
Parts:
- added FID1, FID2: Fiducial, Fiducial:Fiducial_1mm_Mask2mm, symbol Mechanical:Fiducial
- added H5: LOGO, TC-Logo:THETC_LOGO_FOOTPRINT_MASK, symbol TC-logo:LOGO
- C1: MPN (none) -> GRM188C71C475KE21D
- C10, C13, C7, C8: MPN NC -> DNP; now left out of the parts list
- C11, C12, C14, C15, C2, C3, C5, C52: MPN (none) -> 06036C104KAT4A
- C16, C17, C21, C22: MPN (none) -> 251R14S180JV4T
- C18, C19, C4: MPN (none) -> GCJ188R71H104KA12D
- C20, C26: MPN GRM32ER72A225K -> GRM31CC72A475KE11
- C27: value 0.1uF -> 100nF
- C29, C32: value 0.1uF -> 100nF; MPN GRM188R71E104KL -> GRM188R72A104KA35
- C34: MPN GRM21AR71E475KL -> GRM188C71C475KE21D
- C36, C38: MPN CL21A226MOQNNNE -> GRM21BR60J226M
- C37: footprint Inductor_SMD:L_0603_1608Metric -> Capacitor_SMD:C_0603_1608Metric; MPN (none) -> 06036C104KAT4A
- C40, C41: Digi-key PN 445-12541-1-ND -> (none); MF TDK -> (none); MPN (none) -> 06036C104KAT4A; Rating X7R -> (none); Spec 0.1 µF, 25V, X7R, 0603, 20% -> (none); V 25 -> (none)
- C42, C43, C50, C51: footprint Inductor_SMD:L_0805_2012Metric -> Capacitor_SMD:C_0805_2012Metric; MPN GRM21BR61A226ME44L -> GRM21BR60J226M
- C44: Digi-key PN 445-12541-1-ND -> (none); MF TDK -> (none); MPN (none) -> 06036C104KAT4A; Rating X7R -> (none); Spec 0.1uF, 25V, X7R, 0603, 20% -> (none); V 25 -> (none)
- C48, C49: Digi-key PN 1276-1005-1-ND -> (none); MPN (none) -> 06036C104KAT4A; Spec CAP CER 0.1UF 16V X7R 0603 -> (none)
- C53: value 1nF -> 100nF; MPN (none) -> 06036C104KAT4A
- C6: Digi-key PN (none) -> 445-6853-1-ND; MPN (none) -> C1608X5R1A106M080AC
- D8: MPN (none) -> SML-D12U1WT86
- D9: MPN (none) -> CZRU52C3
- F1: MPN (none) -> 0685T1000-01
- H1, H2, H3, H4: MPN (none) -> DNP; now left out of the parts list
- J2: MPN (none) -> 53047-0310
- J7: MPN (none) -> MX23A18NF2
- R23, R27: MPN (none) -> NC
- U10, U11: MPN (none) -> MCP2515-xST
- U16, U17: MPN (none) -> MCP2562-E-MF
- U18, U20: MPN (none) -> MP3423
- U7, U9: MPN (none) -> LM66100
- U8: MPN (none) -> BQ24040DSQR

Commit message: phase 2 start
Parts:
- added F?: 4A, Fuse:Fuse_1206_3216Metric, symbol Device:Fuse
- added FID3, FID4, FID5, FID6: Fiducial, Fiducial:Fiducial_0.5mm_Mask1.5mm, symbol Mechanical:Fiducial
- added SW1: SW_SPST ESE-13V01A, symbol Switch:SW_SPST
- D2: value T3V3S5-7 -> DNP; now left out of the parts list
- U20: MPN MP3423 -> TPS566242DRLR
Connections:
- net BAT_SENS_3V3: now also U2.20 (P0.04/AIN2)
- net IM_OUT_3V3: now also U2.21 (P0.05/AIN3)
- net VBAT: now also F?.1; no longer J2.2 (Pin_2)
- new net: F?.2, J2.2 (Pin_2)
- no-connect marks 54 -> 52
Other:
- note added: "HOW DOES IT WORK"
- note added: "Orderd wrong"

Commit message: single shield on vin dcdc
Parts:
- added J5: RFShield_OnePiece, RF_Shielding:SMS-409N, symbol Device:RFShield_OnePiece
- added J6: RFShield_OnePiece, RF_Shielding:SMS-402C, symbol Device:RFShield_OnePiece
- added J8: RFShield_OnePiece, RF_Shielding:Laird_Technologies_BMI-S-205-F_38.10x25.40mm, symbol Device:RFShield_OnePiece
- added J9: RFShield_OnePiece, RF_Shielding:SMS-455-N-F, symbol Device:RFShield_OnePiece
- C29, C32: footprint Capacitor_SMD:C_0603_1608Metric -> Capacitor_SMD:C_0402_1005Metric
- R21, R22, R24, R25, R33, R34: footprint Resistor_SMD:R_0603_1608Metric -> Resistor_SMD:R_0402_1005Metric
- gave numbers to parts that had none: 1
Connections:
- net GND: now also J9.1 (Shield)
Other:
- moved on the sheet: C20, C26, C27, C29, C32, C33, C34, D7, F1, L2, R21, R22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

Commit message: updated layout, not done
Parts:
- removed R14: 0, Resistor_SMD:R_0603_1608Metric, symbol Device:R
- removed R27: DNP, Resistor_SMD:R_0603_1608Metric, symbol Device:R
- removed SW1: SW_SPST ESE-13V01A, symbol Switch:SW_SPST
- removed U5: TXB0108PWR, Package_SON:USON-20_2x4mm_P0.4mm, symbol TC-ICs:TXB0108PWR
- added C54, C55: 100nF, Capacitor_SMD:C_0603_1608Metric, symbol Device:C
- added C56: 4.7uF, Capacitor_SMD:C_0603_1608Metric, symbol Device:C_Small
- added C57, C59: 10pF, Capacitor_SMD:C_0402_1005Metric, symbol Device:C_Small
- added C58: 100nF, Capacitor_SMD:C_0402_1005Metric, symbol Device:C_Small
- added C60: 100nF, Capacitor_SMD:C_0603_1608Metric, symbol Device:C_Small
- added C? (x2): 1uF, Capacitor_SMD:C_0603_1608Metric, symbol Device:C
- added D10, D11, D12, D13: BAT54FILMY, Diode_SMD:D_SOT-23_ANK, symbol Device:D_Schottky
- added D14, D15, D16, D17, D18, D19, D20, D? (x2): LED, LED_SMD:LED_0603_1608Metric, symbol Device:LED
- added D21: D_Schottky, Package_TO_SOT_SMD:TO-277A, symbol Device:D_Schottky
- added IC1: STM32G030K8T6, STM32G030K8T6:QFP80P900X900X160-32N, symbol STM32G030K8T6:STM32G030K8T6
- added IC?: MCP73833-CNI_MF, SON50P300X300X100-11N-D, symbol MCP73833-CNI_MF:MCP73833-CNI_MF
- added J10: Conn_01x04_Male, Connector_PinHeader_1.27mm:PinHeader_1x04_P1.27mm_Vertical, symbol Connector:Conn_01x04_Male
- added R44, R45: 10, Resistor_SMD:R_0603_1608Metric, symbol Device:R_Small
- added R47, R49: 1k, Resistor_SMD:R_0603_1608Metric, symbol Device:R_Small
- added R50, R51, R52, R53, R54, R55, R56: 750, Resistor_SMD:R_0603_1608Metric, symbol Device:R_Small
- added R? (x2): 1k5, Resistor_SMD:R_0603_1608Metric, symbol Device:R_Small
- added SW2: SW_SPST, Button_Switch_SMD:Nidec_Copal_SH-7010B, symbol Switch:SW_SPST
- added U5: TXB0108DQSR, Package_SON:USON-20_2x4mm_P0.4mm, symbol Logic_LevelTranslator:TXB0108DQSR
- added Y3: Crystal_GND24, Crystal:Crystal_SMD_2016-4Pin_2.0x1.6mm_modified, symbol Device:Crystal_GND24
- R28, R29: footprint Resistor_SMD:R_0603_1608Metric -> Resistor_SMD:R_0402_1005Metric
- R31: value 820k -> 300k
- R32: value 190k -> 5k
- R36, R39, R40, R41: footprint Inductor_SMD:L_0603_1608Metric -> Inductor_SMD:L_0402_1005Metric
Connections:
- net 100V: now also R31.1, D21.1 (K); no longer F1.2
- net 1V8: now also U5.5 (VCCA), U5.6 (OE)
- net 3V3_ALWAYS_ON: now also C56.1, C58.1, D10.1 (K), D12.1 (K), IC1.4 (VDD/VDDA), J10.4 (Pin_4), U5.16 (VCCB); no longer J7.9 (Pin_9)
- net 3V3_ANT: now also D14.2 (A)
- net 3V3_CAN: now also D19.2 (A)
- net 3V3_SENS: now also D18.2 (A)
- net 5V0: now also D15.2 (A)
- net 5V0_BUCK: now also R28.1, U7.5 (ST), U9.3 (~{CE}), C?.1, D?.2 (A), D?.2 (A), IC?.1 (VDD_1), IC?.2 (VDD_2); no longer R31.1
- net BAT_SENS_3V3: now also R45.1; no longer U2.20 (P0.04/AIN2)
- net CTS_1V8: now also U5.4 (A4)
- net CTS_3V3: now also U5.17 (B4)
- net DCD_1V8: now also U5.3 (A3)
- net DCD_3V3: now also U5.18 (B3)
- net GND: now also J5.1 (Shield), C54.2, C55.2, C56.2, C57.2, C58.2, C59.2, C60.2, C?.2, C?.2, D11.2 (A), D13.2 (A), IC1.5 (VSS/VSSA), IC?.11 (EP), IC?.5 (VSS), J10.1 (Pin_1), R50.1, R51.1, R52.1, R53.1, R54.1, R55.1, R56.1, SW2.1 (A), U5.15 (GND)
- net IGN_IN_3V3: no longer U2.10 (P0.29/AIN5)
- net IM_OUT_3V3: now also R44.1; no longer U2.21 (P0.05/AIN3), Z1.5
- net MODEM_DTR_1V8: now also U5.1 (A1)
- net MODEM_DTR_3V3: now also U5.20 (B1)
- net MODEM_RI_1V8: now also U5.2 (A2)
- net MODEM_RI_3V3: now also U5.19 (B2)
- net MODEM_RX_1V8: now also U5.9 (A7)
- net MODEM_RX_3V3: now also U5.12 (B7)
- net MODEM_TX_1V8: now also U5.8 (A6)
- net MODEM_TX_3V3: now also U5.13 (B6)
- net NET_LED: now also D16.2 (A)
- net NTC: now also IC?.8 (THERM)
- net RTS_1V8: now also U5.7 (A5)
- net RTS_3V3: now also U5.14 (B5)
- net SIM_CHIP_DATA: now also D1.6 (IO5); no longer D1.4 (IO3)
- net SIM_CHIP_RST: now also D1.4 (IO3); no longer D1.6 (IO5)
- net STATUS_LED: now also U5.10 (A8)
- net STATUS_LED_3V3: now also D17.2 (A), U5.11 (B8)
- net VBAT: now also C?.1, IC?.10 (VBAT_2), IC?.9 (VBAT_1)
- net STM32_TX: now reaches U2.22 (P0.06)
- net STM32_TX: now also IC1.19 (PA9)
- net VCU_RX: no longer names the net of J7.13 (Pin_13)
- net VCU_TX: no longer names the net of J7.12 (Pin_12)
- new net: D?.1 (K), R?.1 (x2)
- new net: C54.1, D10.2 (A), D11.1 (K), R44.2, R49.1
- new net: D12.2 (A), D13.1 (K), R45.2, R47.1
- new net: D18.1 (K), R52.2
- new net: D21.2 (A), F1.2
- new net: D19.1 (K), R53.2
- new net: C57.1, IC1.3 (PC15-OSC32_OUT), Y3.1
- new net: C59.1, IC1.2 (PC14-OSC32_IN), Y3.3
- new net: D17.1 (K), R51.2
- new net: D20.1 (K), R56.2
- new net: D14.1 (K), R54.2
- new net: IC?.3 (STAT1), R?.2
- new net: IC?.4 (STAT2), R?.2
- new net: D16.1 (K), R50.2
- new net: D15.1 (K), R55.2
- new net BAT_SENS_3V3_STM: C55.1, IC1.27 (PB3), R47.2
- new net IGN_IN_3V3_STM: IC1.26 (PA15)
- new net IM_OUT_3V3_STM: IC1.28 (PB4), R49.2
- new net STM32_IO: D20.2 (A), IC1.18 (PA8), U2.20 (P0.04/AIN2)
- new net STM32_RX: IC1.21 (PA10), U2.21 (P0.05/AIN3)
- new net STM32_SWCLK: IC1.25 (PA14-BOOT0), J10.3 (Pin_3)
- new net STM32_SWDIO: IC1.24 (PA13), J10.2 (Pin_2)
- new net TAMPER: C60.1, IC1.8 (PA1), SW2.2 (B)
- no-connect marks 52 -> 77
Other:
- note added: "?"
- note added: "Change this to output"
- note added: "DEBUG LEDs (Not for production)"
- note added: "Estimated stray cap to be 5pF C load of crystal = 10pF C(load) = (10*10)/(10+10)+5 = 10pF"
- note added: "STM32 prog"
- note added: "USART1 TX = 19 USART1 RX = 21 SWDIO = 24 SWCLK = 25 TAMP_IN2 = 8"
- moved on the sheet: C18, C19, C53, D8, D9, F1, F2, J2, J5, R13, R17, R19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

Commit message: Done, execpt ERC
Parts:
- removed C? (x2): 1uF, Capacitor_SMD:C_0603_1608Metric, symbol Device:C
- removed D?: LED, LED_SMD:LED_0603_1608Metric, symbol Device:LED
- removed FID3, FID4, FID5, FID6: Fiducial, Fiducial:Fiducial_0.5mm_Mask1.5mm, symbol Mechanical:Fiducial
- removed J1: nanoSIM-holder, TC-Connector:SIM8051-6-0-14-01-A, symbol TC-Connector:nanoSIM-holder
- removed R?: 1k5, Resistor_SMD:R_0603_1608Metric, symbol Device:R_Small
- removed SW2: SW_SPST, Button_Switch_SMD:Nidec_Copal_SH-7010B, symbol Switch:SW_SPST
- removed U8: BQ24040DSQR, TC-Power:BQ24040DSQR, symbol TC-Power:BQ24040DSQR
- added C61: 100nF, Capacitor_SMD:C_0603_1608Metric, symbol Device:C
- added C62: 1uF, Capacitor_SMD:C_0402_1005Metric, symbol Device:C
- added J1: SIM8060-6-0-14-00-A, SIM8060-6-0-14-00-A:SIM8060601400A, symbol SIM8060-6-0-14-00-A:SIM8060-6-0-14-00-A
- added S1: ESE-11MV9, ESE11MV9, symbol ESE-11MV9:ESE-11MV9
- D3, D4, D5: mpn LY L29K-H1K2-26-Z -> QBLP601D-IG
- R17: value 1k1 -> 2k
- R23: value DNP -> 10k; MPN NC -> (none)
- U4: value MX25L3233FZBI-08Q -> MX25L25645GZNI-08G; footprint TC-ICs:4x3-8-USON -> Package_SON:WSON-8-1EP_6x5mm_P1.27mm_EP3.4x4mm; MPN MX25L3233FZBI-08Q -> MX25L25645GZNI-08G
- gave numbers to parts that had none: 3
Connections:
- net 3V3_ALWAYS_ON: now also C61.1
- net 4V7_BOOST: now also C62.1
- net 5V0_BUCK: now also D8.2 (A)
- net GND: now also C61.2, C62.2, J1.C5 (GND_1), J1.G1 (GND_2), J1.G2 (GND_3), J1.G3 (GND_4), J1.G4 (GND_5), S1.C1 (COM_1), S1.C2 (COM_2); no longer R23.2, U4.GND
- net SIM_CHIP_CLK: now also J1.C3 (CLK)
- net SIM_CHIP_DATA: now also J1.C7 (I/O)
- net SIM_CHIP_RST: now also J1.C2 (RST)
- net SIM_VDD: now also J1.C1 (VCC)
- net TAMPER: now also R23.2; no longer C60.1
- net VBAT: no longer R26.2
- net at R17.1: now also IC2.6 (PROG)
- net at R23.1: now also C60.1, S1.1 (NO_1), S1.2 (NO_2)
- net at IC2.3 (STAT1): now also R26.2
- net at R26.1: now also D8.1 (K); no longer D8.2 (A)
- no-connect marks 77 -> 76
Other:
- note added: "Flash memory 256MBit"
- note removed: "Flash memory 32MBit"
- moved on the sheet: C18, C19, C25, C28, C3, C30, C31, C60, D22, D8, IC2, R14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

Commit message: ready for production
Parts:
- removed J6: RFShield_OnePiece, RF_Shielding:SMS-402C, symbol Device:RFShield_OnePiece
- removed J8: RFShield_OnePiece, RF_Shielding:Laird_Technologies_BMI-S-205-F_38.10x25.40mm, symbol Device:RFShield_OnePiece
Changed lines of the file:
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@@
     (pin "1")
   )
-  (symbol (lib_id "Device:RFShield_OnePiece") (at 248.92 502.92 0) (unit 1)
-    (in_bom yes) (on_board yes) (fields_autoplaced)
-    (property "Reference" "J8" (id 0) (at 265.43 501.6499 0)
-      (effects (font (size 1.27 1.27)) (justify left))
-    )
-    (property "Value" "RFShield_OnePiece" (id 1) (at 265.43 504.1899 0)
-      (effects (font (size 1.27 1.27)) (justify left))
-    )
-    (property "Footprint" "RF_Shielding:Laird_Technologies_BMI-S-205-F_38.10x25.40mm" (id 2) (at 248.92 505.46 0)
-      (effects (font (size 1.27 1.27)) hide)
-    )
-    (property "Datasheet" "~" (id 3) (at 248.92 505.46 0)
-      (effects (font (size 1.27 1.27)) hide)
-    )
-    (pin "1")
-  )
   (symbol (lib_id "Device:C_Small") (at 420.37 111.76 0) (unit 1)
     (in_bom yes) (on_board yes)
@@
     (pin "3")
   )
-  (symbol (lib_id "Device:RFShield_OnePiece") (at 248.92 473.71 0) (unit 1)
-    (in_bom yes) (on_board yes) (fields_autoplaced)
-    (property "Reference" "J6" (id 0) (at 265.43 472.4399 0)
-      (effects (font (size 1.27 1.27)) (justify left))
-    )
-    (property "Value" "RFShield_OnePiece" (id 1) (at 265.43 474.9799 0)
-      (effects (font (size 1.27 1.27)) (justify left))
-    )
-    (property "Footprint" "RF_Shielding:SMS-402C" (id 2) (at 248.92 476.25 0)
-      (effects (font (size 1.27 1.27)) hide)
-    )
-    (property "Datasheet" "https://www.leadertechinc.com/assets/files/EngineeringDrawings/SMS-402.PDF" (id 3) (at 248.92 476.25 0)
-      (effects (font (size 1.27 1.27)) hide)
-    )
-    (property "MPN" "SMS-402C" (id 4) (at 248.92 473.71 0)
-      (effects (font (size 1.27 1.27)) hide)
-    )
-    (pin "1")
-  )
   (symbol (lib_id "Device:LED") (at 767.715 268.605 180) (unit 1)
     (in_bom yes) (on_board yes)
@@
       (reference "J5") (unit 1) (value "RFShield_OnePiece") (footprint "RF_Shielding:SMS-409N")
     )
-    (path "/6109e549-92d5-4993-a164-fd0af07db971"
-      (reference "J6") (unit 1) (value "RFShield_OnePiece") (footprint "RF_Shielding:SMS-402C")
-    )
     (path "/c227d7e3-ee3d-449d-b72a-7c4d9fc5832b"
       (reference "J7") (unit 1) (value "MX23A18NF2") (footprint "TC-Connector:MX23A18NF1")
     )
-    (path "/2e8d9018-272d-4934-9eb6-ea3a587acbcb"
-      (reference "J8") (unit 1) (value "RFShield_OnePiece") (footprint "RF_Shielding:Laird_Technologies_BMI-S-205-F_38.10x25.40mm")
-    )
     (path "/cab0b7ca-f826-4145-9c2e-f76d675969b2"
