File: roam.kicad_sch (KiCad schematic)
At the start: 232 parts, among them IC2 MCP73833T-FCI/MF, J1 SIM8060-6-0-14-00-A, J2 Battery, J7 MX23A18NF1, Q1 BC846A,215, Q2 BC846A,215, U1 SIP32408DNP-T1-GE4, U10 LTV-217, U12 LM3671MF-3.3/NOPB, U13 LIS2DH12TR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

Commit message: rm leds, added trace for u20
Parts:
- removed D14, D15, D19, D22, D8: LED, LED_SMD:LED_0603_1608Metric, symbol Device:LED
- removed R26, R50, R54: 750, Resistor_SMD:R_0603_1608Metric, symbol Device:R_Small
- removed R39: 34.8k, Resistor_SMD:R_0402_1005Metric, symbol Device:R
- removed R55: 2k, Resistor_SMD:R_0603_1608Metric, symbol Device:R_Small
- added R21: 4K7, Resistor_SMD:R_0603_1608Metric, symbol Device:R_Small
- R14: value 750 -> 4K7; MF (none) -> Stackpole; MPN RC0603JR-07750RL -> RC0603FR-074K7L
- R36: value 100k -> 10k
Connections:
- net 3V3_ALWAYS_ON: now also R14.2, R36.1, R21.2
- net 5V0: no longer R36.1
- net CHARGER_STAT_1: now also R14.1
- net CHARGER_STAT_2: now also R21.1; no longer R14.2
- net U20_EN: now reaches R36.2, U20.5 (EN)
- net U20_EN: now also U2.10 (P0.29/AIN5)
- net VCU_LED: no longer names the net of U4.40 (PC9)
Other:
- note removed: "For production, the LEDs should be removed and the resistor val changed to 4k7"
- moved on the sheet: C35, C37, R36

Commit message: Added a jumper for CAN termination and updated mpns for status LEDs
Parts:
- added J3, J4: Conn_01x02_Pin, Connector_PinHeader_2.54mm:PinHeader_1x02_P2.54mm_Vertical, symbol Connector:Conn_01x02_Pin
- added R26, R30: 120, Resistor_SMD:R_0603_1608Metric, symbol Device:R_Small
- D3, D4: If 1mA -> 20mA; MPN SML-D12U1WT86 -> QBLP601D-IB; Vf 1.8V -> 3.2V; mpn QBLP601D-IG -> QBLP601D-IB
- D5: If 1mA -> 20mA; MPN SML-D12U1WT86 -> QBLP601D-IG; Vf 1.8V -> 3.2V
Connections:
- net CAN_250_H: now also J4.1 (Pin_1)
- net CAN_250_L: now also R30.2
- net CAN_500_H: now also J3.1 (Pin_1)
- net CAN_500_L: now also R26.2
- new net: J4.2 (Pin_2), R30.1
- new net: J3.2 (Pin_2), R26.1
Other:
- note added: "These LEDs are tested with the case and is bright enough with 750 Ohm/1mA current Can be driven directly on MCU pin"

Commit message: clean up
Parts:
- removed J3, J4: Conn_01x02_Pin, Connector_PinHeader_2.54mm:PinHeader_1x02_P2.54mm_Vertical, symbol Connector:Conn_01x02_Pin
- added J3, J5: Conn_01x03_Pin, Connector_PinHeader_1.27mm:PinHeader_1x03_P1.27mm_Vertical_SMD_Pin1Left, symbol Connector:Conn_01x03_Pin
- added TCLOGO3: SYM_Magnet_Large, TC-Logo:Sticker-frame, symbol Graphic:SYM_Magnet_Large
- added TCLOGO4: SYM_Magnet_Large, TC-Logo:SIM-instruction, symbol Graphic:SYM_Magnet_Large
- TCLOGO2: footprint TC-Logo:Logo-Text-Silk -> TC-Logo:Logo-Text-Silk-Smaller
Connections:
- net CAN_250_H: now also J3.2 (Pin_2)
- net CAN_500_H: now also J5.2 (Pin_2)
- net GPIO_3V3_4: now also U4.15 (PA1); no longer U4.62 (PB9)
- net GPIO_3V3_5: now also U4.14 (PA0); no longer U4.61 (PB8)
- net VCU_CAN1_RX: now also U4.61 (PB8); no longer U4.44 (PA11)
- net VCU_CAN1_TX: now also U4.62 (PB9); no longer U4.45 (PA12)
- net VCU_USART2_CTS: now also U4.44 (PA11); no longer U4.14 (PA0)
- net VCU_USART2_RTS: now also U4.45 (PA12); no longer U4.15 (PA1)
- net VCU_USART2_RX: now also U4.43 (PA10); no longer U4.17 (PA3)
- net VCU_USART2_TX: now also U4.42 (PA9); no longer U4.16 (PA2)
- net at R30.1: now also J3.1 (Pin_1)
- net at R26.1: now also J5.1 (Pin_1)
- no-connect marks 65 -> 67
Other:
- note added: "CAN1_RX / CAN1_TX Need to be remapped due to confilct with USART1_CTS / RTS"
- note removed: "CAN TX/TX or TX/RX??"
- note removed: "Do we need a RT clock?"
- note removed: "TODO Check footprint and pinmap Check resistor values"
- note removed: "TODO Correct colors on LEDs"
- moved on the sheet: C72, C74, C80, D21, L12, R26, R30, R51, R56, R59, R60, U16

Commit message: some cleanup and new comments on the schematic
Connections:
- net GPIO_3V3_5 renamed IGN_3V3
- net GPIO_5 renamed IGN_IN
- net VCU_USART2_CTS renamed VCU_USART1_CTS
- net VCU_USART2_RTS renamed VCU_USART1_RTS
- net VCU_USART2_RX renamed VCU_USART1_RX
- net VCU_USART2_TX renamed VCU_USART1_TX
Other:
- note added: "12 bit = 24mV steps 10 bit = 100mV steps"
- note added: "BOOT1 pin always pulled low"
- note added: "CZRU52C3V3 replace to: CZRU52C3V9 CZRU52C4V3"
- note added: "IGN and IMOB"
- note added: "In sleep mode or not used: CS need to be HIGH and the other pins need to be grounded to achive low consumption"
- note added: "MODEM / NRF lvl shigt"
- note added: "Main Connector"
- note added: "Max 30V input"
- note added: "SIM CARD"
- note added: "Tested with R64 = 6k8 and R66 = 4k7 The HIGH/LOW thresshold is 3-4V instead of ~1.7V the upper limit is 60V+ and the current / heat / diode warnout is reduced. D2 should be behind R64 and maybe be a TVS instead?"
- note added: "Testpoints"
- note added: "These LEDs are tested with the enclosure and is bright enough with 750 Ohm/1mA current Can be driven directly on MCU pin"
- note added: "VCU"
- note removed: "16 USART2_TX 17 USART2_RX 14 USART2_CTS 15 USART2_RTS"
- note removed: "2 Tamper switch"
- note removed: "33 CAN2_RX 34 CAN2_TX 44 CAN1_RX 45 CAN1_TX"
- note removed: "42 USART1_TX 43 USART1_RX 44 USART1_CTS 45 USART1_RTS"
- note removed: "46 JTMS-SWDIO 49 JTMS-SWCLK 28 BOOT1 60 BOOT0"
- note removed: "7 NRST (week internal pullup)"
- note removed: "Connector"
- note removed: "EN (divider for undervoltage?)"
- note removed: "LSE Clock pins: OSC32_IN: 3 OSC32_OUT: 4 HSE Clock pins: OSC_IN: 5 OSC32_OUT: 6"
- note removed: "Llv shift modem serial"
- note removed: "MODEM"
- note removed: "SIM"
- note removed: "These LEDs are tested with the case and is bright enough with 750 Ohm/1mA current Can be driven directly on MCU pin"
- note removed: "https://www.st.com/resource/en/application_note/an2586-getting-started-with-stm32f10xxx-hardware-development-stmicroelectronics.pdf"
- note removed: "https://www.st.com/resource/en/datasheet/stm32f105rb.pdf"
- note removed: "https://www.st.com/resource/en/product_training/STM32MP1-Security-Tamper_TAMP.pdf"
- company: (none) -> TTC
- title: (none) -> ROAM 
- moved on the sheet: C14, C15, C16, C17, C18, C19, C20, C21, C26, C3, C41, C47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

Commit message: revision for production
Parts:
- D2: value BAT54AW -> VCAN36A2-03GHE3-08; symbol Diode:BAT54AW -> TC-Transistors:VCAN36A2-03GHE3-08; MPN BAT54AW -> VCAN36A2-03GHE3-08
- D9: value 3v3 -> 4v3; MPN CZRU52C3V3 -> CZRU52C4V3
- R26, R30: MPN (none) -> RES 120K OHM 1% 1/10W 0603
- R64: value 680 -> 6k8; MPN ERJ-PB6B6800V -> RMCF0805JT6K80
- R66: value 1k -> 4K7; MF Stackpole -> (none); MPN PFR05S-102-FNH -> RC0402FR-074K7L
Other:
- note added: "CTR=Ic/If x 100%"
- note added: "If = ~1.5mA"
- note added: "Power dissipation R64 = 15,9mW"
- note removed: "If = 15mA"
- note removed: "Power dissipation R64 = 153mW"
Changed lines of the file:
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@@
   (junction (at 55.88 236.22) (diameter 0) (color 0 0 0 0)
   )
+  (junction (at 613.41 325.12) (diameter 0) (color 0 0 0 0)
+  )
   (junction (at 480.06 396.24) (diameter 0) (color 0 0 0 0)
   )
@@
   (junction (at 662.94 275.59) (diameter 0) (color 0 0 0 0)
   )
+  (junction (at 613.41 281.94) (diameter 0) (color 0 0 0 0)
+  )
   (junction (at 67.31 172.72) (diameter 0) (color 0 0 0 0)
   )
@@
   (junction (at 415.29 161.29) (diameter 0) (color 0 0 0 0)
   )
-  (junction (at 615.95 281.94) (diameter 0) (color 0 0 0 0)
-  )
   (junction (at 276.225 52.07) (diameter 0) (color 0 0 0 0)
   )
@@
   (junction (at 495.935 396.24) (diameter 0) (color 0 0 0 0)
   )
-  (junction (at 615.95 325.12) (diameter 0) (color 0 0 0 0)
-  )
   (junction (at 373.38 106.68) (diameter 0) (color 0 0 0 0)
   )
@@
     (stroke (width 0) (type default))
   )
+  (wire (pts (xy 618.49 304.8) (xy 622.3 304.8))
+    (stroke (width 0) (type default))
+  )
   (wire (pts (xy 462.28 396.24) (xy 462.28 398.78))
     (stroke (width 0) (type default))
@@
     (stroke (width 0) (type default))
   )
-  (wire (pts (xy 615.95 325.12) (xy 629.92 325.12))
+  (wire (pts (xy 603.25 325.12) (xy 613.41 325.12))
     (stroke (width 0) (type default))
   )
@@
     (stroke (width 0) (type default))
   )
-  (wire (pts (xy 603.25 325.12) (xy 615.95 325.12))
-    (stroke (width 0) (type default))
-  )
   (wire (pts (xy 462.915 288.29) (xy 462.915 292.1))
     (stroke (width 0) (type default))
@@
     (stroke (width 0) (type default))
   )
-  (wire (pts (xy 605.79 281.94) (xy 615.95 281.94))
-    (stroke (width 0) (type default))
-  )
   (polyline (pts (xy 302.26 85.09) (xy 397.51 85.09))
     (stroke (width 0) (type default))
@@
     (stroke (width 0) (type default))
   )
-  (wire (pts (xy 626.11 297.18) (xy 628.65 297.18))
-    (stroke (width 0) (type default))
-  )
-  (wire (pts (xy 615.95 312.42) (xy 615.95 325.12))
-    (stroke (width 0) (type default))
-  )
   (wire (pts (xy 16.51 215.9) (xy 33.02 215.9))
     (stroke (width 0) (type default))
@@
     (stroke (width 0) (type default))
   )
-  (wire (pts (xy 615.95 281.94) (xy 624.84 281.94))
+  (wire (pts (xy 605.79 281.94) (xy 613.41 281.94))
     (stroke (width 0) (type default))
   )
@@
     (stroke (width 0) (type default))
   )
-  (wire (pts (xy 615.95 297.18) (xy 615.95 281.94))
-    (stroke (width 0) (type default))
-  )
   (wire (pts (xy 403.225 391.795) (xy 403.225 393.065))
     (stroke (width 0) (type default))
@@
     (stroke (width 0) (type default))
   )
-  (wire (pts (xy 621.03 304.8) (xy 622.3 304.8))
-    (stroke (width 0) (type default))
-  )
   (wire (pts (xy 442.595 396.24) (xy 462.28 396.24))
     (stroke (width 0) (type default))
@@
     (stroke (width 0) (type default))
   )
+  (wire (pts (xy 613.41 316.23) (xy 613.41 325.12))
+    (stroke (width 0) (type default))
+  )
   (wire (pts (xy 577.85 177.8) (xy 577.85 205.74))
     (stroke (width 0) (type default))
@@
     (stroke (width 0) (type default))
   )
+  (wire (pts (xy 613.41 281.94) (xy 624.84 281.94))
+    (stroke (width 0) (type default))
+  )
   (wire (pts (xy 121.92 237.49) (xy 102.87 237.49))
     (stroke (width 0) (type default))
@@
     (stroke (width 0) (type default))
   )
+  (wire (pts (xy 613.41 325.12) (xy 629.92 325.12))
+    (stroke (width 0) (type default))
+  )
   (wire (pts (xy 290.83 129.54) (xy 290.83 132.08))
     (stroke (width 0) (type default))
@@
     (stroke (width 0) (type default))
   )
+  (wire (pts (xy 613.41 281.94) (xy 613.41 293.37))
+    (stroke (width 0) (type default))
+  )
   (wire (pts (xy 182.245 347.345) (xy 182.245 350.52))
     (stroke (width 0) (type default))
@@
     (stroke (width 0) (type default))
   )
+  (wire (pts (xy 626.11 297.18) (xy 628.65 297.18))
+    (stroke (width 0) (type default))
+  )
   (wire (pts (xy 690.88 189.23) (xy 697.23 189.23))
     (stroke (width 0) (type default))
@@
     (effects (font (size 1.27 1.27)) (justify left bottom))
   )
-  (text "Power dissipation R64 = 153mW" (at 600.71 278.13 0)
+  (text "Power dissipation R64 = 15,9mW" (at 600.71 278.13 0)
     (effects (font (size 1.27 1.27)) (justify left bottom))
   )
@@
     (effects (font (size 1.27 1.27)) (justify left bottom))
   )
-  (text "If = 15mA" (at 619.76 295.91 0)
+  (text "If = ~1.5mA" (at 618.49 294.64 0)
     (effects (font (size 1.27 1.27)) (justify left bottom))
   )
@@
     (effects (font (size 2.54 2.54)) (justify left bottom))
   )
+  (text "CTR=Ic/If x 100%" (at 581.66 293.37 0)
+    (effects (font (size 1.27 1.27)) (justify left bottom))
+  )
   (text "C63\nVibration tolerant variant:\nEEE-FK1K330V\n(Not currently in stock)"
     (at 195.58 138.43 0)
@@
       (effects (font (size 1.27 1.27)) (justify left))
     )
-    (property "Value" "3v3" (at 48.26 320.0399 90)
+    (property "Value" "4v3" (at 48.26 320.0399 90)
       (effects (font (size 1.27 1.27)) (justify left))
     )
@@
       (effects (font (size 1.27 1.27)) hide)
     )
-    (property "MPN" "CZRU52C3V3" (at 45.72 318.77 0)
+    (property "MPN" "CZRU52C4V3" (at 45.72 318.77 0)
       (effects (font (size 1.27 1.27)) hide)
     )
-    (property "Description" "DIODE ZENER 3.3V 150MW 0603" (at 45.72 318.77 0)
+    (property "Description" "DIODE ZENER 4.3V 150MW 0603" (at 45.72 318.77 0)
       (effects (font (size 1.27 1.27)) hide)
     )
@@
       (effects (font (size 1.27 1.27)) (justify left))
     )
-    (property "Value" "1k" (at 643.6614 285.623 0)
+    (property "Value" "4K7" (at 643.6614 285.623 0)
       (effects (font (size 1.27 1.27)) (justify left))
     )
@@
       (effects (font (size 1.27 1.27)) hide)
     )
-    (property "Datasheet" "~" (at 645.16 284.48 0)
+    (property "Datasheet" "https://www.digikey.cn/zh/products/detail/yageo/RC0402FR-074K7L/2827563?amp%3BWT.z_header=search_go&s=N4IgTCBcDaIEoGEAMAWJYBicC0SDsKA0ngDIgC6AvkA" (at 645.16 284.48 0)
       (effects (font (size 1.27 1.27)) hide)
     )
-    (property "MF" "Stackpole" (at 645.16 284.48 0)
+    (property "MF" "" (at 645.16 284.48 0)
       (effects (font (size 1.27 1.27)) hide)
     )
-    (property "MPN" "PFR05S-102-FNH" (at 645.16 284.48 0)
+    (property "MPN" "RC0402FR-074K7L" (at 645.16 284.48 0)
       (effects (font (size 1.27 1.27)) hide)
     )
-    (property "Description" "RES SMD 1 KOHM 1% 1/16W 0402" (at 645.16 284.48 0)
+    (property "Description" "RES 4.7K OHM 1% 1/16W 0402" (at 645.16 284.48 0)
       (effects (font (size 1.27 1.27)) hide)
     )
@@
       (effects (font (size 1.27 1.27)) (justify left))
     )
-    (property "Value" "680" (at 626.3386 288.163 0)
+    (property "Value" "6k8" (at 626.3386 288.163 0)
       (effects (font (size 1.27 1.27)) (justify left))
     )
@@
       (effects (font (size 1.27 1.27)) hide)
     )
-    (property "Datasheet" "https://www.digikey.sg/en/products/detail/panasonic-electronic-components/ERJ-PB6B6800V/6213358" (at 624.84 287.02 0)
+    (property "Datasheet" "https://www.digikey.cn/zh/products/detail/stackpole-electronics-inc/RMCF0805JT6K80/1757931" (at 624.84 287.02 0)
       (effects (font (size 1.27 1.27)) hide)
     )
-    (property "MPN" "ERJ-PB6B6800V" (at 624.84 287.02 0)
+    (property "MPN" "RMCF0805JT6K80" (at 624.84 287.02 0)
       (effects (font (size 1.27 1.27)) hide)
     )
-    (property "Description" "RES SMD 680 OHM 0.1% 1/4W 0805" (at 624.84 287.02 0)
+    (property "Description" "RES 6.8K OHM 5% 1/8W 0805" (at 624.84 287.02 0)
       (effects (font (size 1.27 1.27)) hide)
     )
@@
     )
   )
-  (symbol (lib_id "Diode:BAT54AW") (at 615.95 304.8 90) (unit 1)
-    (in_bom yes) (on_board yes) (dnp no) (fields_autoplaced)
-    (property "Reference" "D2" (at 613.41 304.165 90)
+  (symbol (lib_id "TC-Transistors:VCAN36A2-03GHE3-08") (at 610.87 309.88 0) (mirror y) (unit 1)
+    (in_bom yes) (on_board yes) (dnp no)
+    (property "Reference" "D2" (at 610.87 303.53 0)
       (effects (font (size 1.27 1.27)) (justify left))
     )
-    (property "Value" "BAT54AW" (at 613.41 306.705 90)
+    (property "Value" "VCAN36A2-03GHE3-08" (at 610.87 306.07 0)
       (effects (font (size 1.27 1.27)) (justify left))
     )
-    (property "Footprint" "Package_TO_SOT_SMD:SOT-323_SC-70" (at 612.775 302.895 0)
-      (effects (font (size 1.27 1.27)) (justify left) hide)
+    (property "Footprint" "Package_TO_SOT_SMD:SOT-323_SC-70" (at 605.79 332.74 0)
+      (effects (font (size 1.27 1.27)) hide)
     )
-    (property "Datasheet" "https://assets.nexperia.com/documents/data-sheet/BAT54W_SER.pdf" (at 615.95 307.848 0)
+    (property "Datasheet" "https://www.vishay.com/docs/86164/vcan36a2-03g.pdf" (at 603.25 334.01 0)
       (effects (font (size 1.27 1.27)) hide)
     )
-    (property "MPN" "BAT54AW" (at 615.95 304.8 90)
+    (property "MPN" "VCAN36A2-03GHE3-08" (at 608.33 331.47 0)
       (effects (font (size 1.27 1.27)) hide)
     )
-    (property "Description" "DIODE SCHOTTKY 30V 100MA SOT323" (at 615.95 304.8 0)
+    (property "Description" "TVS DIODE 36VWM 63VC SOT323" (at 609.6 328.93 0)
       (effects (font (size 1.27 1.27)) hide)
     )
@@
       (effects (font (size 1.27 1.27)) hide)
     )
-    (property "MPN" "" (at 522.605 411.48 0)
+    (property "MPN" "RES 120K OHM 1% 1/10W 0603" (at 522.605 411.48 0)
       (effects (font (size 1.27 1.27)) hide)
     )
-    (property "Description" "" (at 522.605 411.48 0)
+    (property "Description" "RES 120K OHM 1% 1/10W 0603" (at 522.605 411.48 0)
       (effects (font (size 1.27 1.27)) hide)
     )
@@
       (effects (font (size 1.27 1.27)) hide)
     )
-    (property "MPN" "" (at 521.335 359.41 0)
+    (property "MPN" "RES 120K OHM 1% 1/10W 0603" (at 521.335 359.41 0)
       (effects (font (size 1.27 1.27)) hide)
     )
-    (property "Description" "" (at 521.335 359.41 0)
+    (property "Description" "RES 120K OHM 1% 1/10W 0603" (at 521.335 359.41 0)
       (effects (font (size 1.27 1.27)) hide)
     )

Commit message: update bom
Parts:
- R26, R30: MPN RES 120K OHM 1% 1/10W 0603 -> RMCF0603JG120R
Changed lines of the file:
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@@
       (effects (font (size 1.27 1.27)) hide)
     )
-    (property "MPN" "RES 120K OHM 1% 1/10W 0603" (at 522.605 411.48 0)
-      (effects (font (size 1.27 1.27)) hide)
-    )
-    (property "Description" "RES 120K OHM 1% 1/10W 0603" (at 522.605 411.48 0)
+    (property "MPN" "RMCF0603JG120R" (at 522.605 411.48 0)
+      (effects (font (size 1.27 1.27)) hide)
+    )
+    (property "Description" "RES 120 OHM 5% 1/10W 0603" (at 522.605 411.48 0)
       (effects (font (size 1.27 1.27)) hide)
     )
@@
       (effects (font (size 1.27 1.27)) hide)
     )
-    (property "MPN" "RES 120K OHM 1% 1/10W 0603" (at 521.335 359.41 0)
-      (effects (font (size 1.27 1.27)) hide)
-    )
-    (property "Description" "RES 120K OHM 1% 1/10W 0603" (at 521.335 359.41 0)
-      (effects (font (size 1.27 1.27)) hide)
-    )
+    (property "MPN" "RMCF0603JG120R" (at 521.335 359.41 0)
+      (effects (font (size 1.27 1.27)) hide)
+    )
+    (property "Description" "RES 120 OHM 5% 1/10W 0603" (at 521.335 359.41 0)
+      (effects (font (size 1.27 1.27)) hide)
+    )

Commit message: bom update
Parts:
- C52: footprint Inductor_SMD:L_0402_1005Metric -> Capacitor_SMD:C_0402_1005Metric
- R36: MPN 667-ERJ-2RKF1003X -> RMCF0402FT10K0
Changed lines of the file:
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@@
       (effects (font (size 1.27 1.27)) hide)
     )
-    (property "MPN" "667-ERJ-2RKF1003X" (at 447.04 38.1 0)
+    (property "MPN" "RMCF0402FT10K0" (at 447.04 38.1 0)
       (effects (font (size 1.27 1.27)) hide)
     )
-    (property "Description" "RES SMD 100K OHM 1% 1/10W 0402" (at 447.04 38.1 0)
+    (property "Description" "RES 10K OHM 1% 1/16W 0402" (at 447.04 38.1 0)
       (effects (font (size 1.27 1.27)) hide)
     )
@@
       (effects (font (size 1.27 1.27)) (justify left))
     )
-    (property "Footprint" "Inductor_SMD:L_0402_1005Metric" (at 567.3852 55.88 0)
+    (property "Footprint" "Capacitor_SMD:C_0402_1005Metric" (at 567.3852 55.88 0)
       (effects (font (size 1.27 1.27)) hide)
     )

Commit message: LOGO update
Parts:
- added Anti-static1: SYM_Magnet_Large, Symbol:ESD-Logo_6.6x6mm_SilkScreen, symbol Graphic:SYM_Magnet_Large
- added CE_LOGO1: SYM_Magnet_Large, TC-Logo:CE_LOGO, symbol Graphic:SYM_Magnet_Large
- added RoHs_LOGO1: SYM_Magnet_Large, TC-Logo:RoHs-LOGO, symbol Graphic:SYM_Magnet_Large
Changed lines of the file:
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@@
+    )
+  )
+  (symbol (lib_id "Graphic:SYM_Magnet_Large") (at 784.86 477.52 0) (unit 1)
+    (in_bom no) (on_board yes) (dnp no)
+    (property "Reference" "RoHs_LOGO1" (at 784.86 473.71 0)
+      (effects (font (size 1.27 1.27)))
+    )
+    (property "Value" "SYM_Magnet_Large" (at 784.86 483.87 0)
+      (effects (font (size 1.27 1.27)) hide)
+    )
+    (property "Footprint" "TC-Logo:RoHs-LOGO" (at 784.86 482.6 0)
+      (effects (font (size 1.27 1.27)) hide)
+    )
+    (property "Datasheet" "~" (at 785.622 482.6 0)
+      (effects (font (size 1.27 1.27)) hide)
+    )
+    (property "Sim.Enable" "0" (at 784.86 477.52 0)
+      (effects (font (size 1.27 1.27)) hide)
+    )
+    (instances
+      (project "roam"
+        (path "/e63e39d7-6ac0-4ffd-8aa3-1841a4541b55"
+          (reference "RoHs_LOGO1") (unit 1)
+        )
+      )
     )
   )
@@
         (path "/e63e39d7-6ac0-4ffd-8aa3-1841a4541b55"
           (reference "R12") (unit 1)
+        )
+      )
+    )
+  )
+  (symbol (lib_id "Graphic:SYM_Magnet_Large") (at 801.37 464.82 0) (unit 1)
+    (in_bom no) (on_board yes) (dnp no)
+    (property "Reference" "Anti-static1" (at 801.37 461.01 0)
+      (effects (font (size 1.27 1.27)))
+    )
+    (property "Value" "SYM_Magnet_Large" (at 801.37 471.17 0)
+      (effects (font (size 1.27 1.27)) hide)
+    )
+    (property "Footprint" "Symbol:ESD-Logo_6.6x6mm_SilkScreen" (at 801.37 469.9 0)
+      (effects (font (size 1.27 1.27)) hide)
+    )
+    (property "Datasheet" "~" (at 802.132 469.9 0)
+      (effects (font (size 1.27 1.27)) hide)
+    )
+    (property "Sim.Enable" "0" (at 801.37 464.82 0)
+      (effects (font (size 1.27 1.27)) hide)
+    )
+    (instances
+      (project "roam"
+        (path "/e63e39d7-6ac0-4ffd-8aa3-1841a4541b55"
+          (reference "Anti-static1") (unit 1)
         )
       )
@@
         )
       )
+    )
+  )
+  (symbol (lib_id "Graphic:SYM_Magnet_Large") (at 784.86 464.82 0) (unit 1)
+    (in_bom no) (on_board yes) (dnp no)
+    (property "Reference" "CE_LOGO1" (at 784.86 461.01 0)
+      (effects (font (size 1.27 1.27)))
+    )
+    (property "Value" "SYM_Magnet_Large" (at 784.86 471.17 0)
+      (effects (font (size 1.27 1.27)) hide)
+    )
+    (property "Footprint" "TC-Logo:CE_LOGO" (at 784.86 469.9 0)
+      (effects (font (size 1.27 1.27)) hide)
+    )
+    (property "Datasheet" "~" (at 785.622 469.9 0)
+      (effects (font (size 1.27 1.27)) hide)
+    )
+    (property "Sim.Enable" "0" (at 784.86 464.82 0)
+      (effects (font (size 1.27 1.27)) hide)
+    )
+    (instances
+      (project "roam"
+        (path "/e63e39d7-6ac0-4ffd-8aa3-1841a4541b55"
+          (reference "CE_LOGO1") (unit 1)
+        )
+      )
