File: roam.kicad_sch (KiCad schematic)
At the start: 305 parts, among them IC2 MCP73833T-FCI/MF, J1 SIM8060-6-0-14-00-A, J2 Battery, J3 Conn_01x03_Pin, J5 Conn_01x03_Pin, J7 MX23A18NF1, P1 USB_C_USB2.0, Q2 MMBT3904, Q3 MMBT3904, Q5 BC846A,215, Q6 BC846A,215, Q7 BC846A,215, U1 NUP4202, U10 LTV-217, U11 MAX13487EESAT, U12 LM3671MF-3.3/NOPB, U13 LIS2DH12TR, U14 MAX17643ATC+, U15 FDMC86139P, U16 MCP2562-E/MF, U17 LTV-217, U18 MP3423GG, U2 MDBT50Q-1M, U20 TPS566242DRLR, U23 TXS0102DCU, U24 LP5907MFX-3.3, U27 EG915ULAAB-N05-SNNSA, U28 LC29H, U29 USBLC6-2SC6, U31 B8389, U32 LP5907MFX-3.3, U4 STM32F105RBT6, U5 TXB0108DQSR, U6 MCP2562-E/MF, U6 MX25R6435FZNIL0, U6 W25N512GVEIG, U7 LM66100DCKR, U8 GP.1575.25.2.A.02, U9 LM66100DCKR, Y1 25MHz

Commit message: done for review
Parts:
- removed F1: 1A, Fuse:Fuse_0603_1608Metric, symbol Device:Fuse
- removed P1: USB_C_USB2.0, Connector_USB:USB_C_Receptacle_G-Switch_GT-USB-7010ASV, symbol Connector:USB_C_Receptacle_USB2.0
- removed R24, R77: 5K1, Resistor_SMD:R_0402_1005Metric, symbol Device:R
- removed R78: 20, Resistor_SMD:R_0402_1005Metric, symbol Device:R
- removed R80: 1k5, Resistor_SMD:R_0603_1608Metric, symbol Device:R
- added D1: AXGD10402, Diode_SMD:D_0402_1005Metric, symbol Device:D_TVS_Filled
- added J4: USB_B_Micro, Connector_USB:USB_Micro-B_XKB_U254-051T-4BH83-F1S, symbol Connector:USB_B_Micro
- added R5: 20, Resistor_SMD:R_0402_1005Metric, symbol Device:R
- C90: footprint Capacitor_SMD:C_0805_2012Metric_Pad1.18x1.45mm_HandSolder -> Capacitor_SMD:C_0402_1005Metric
Connections:
- net GND: now also D1.1 (A1), D1.2 (A2), J4.5 (GND), J4.6 (Shield)
- net USB_DM: now also R5.2
- net USB_VBUS: now also J4.1 (VBUS)
- net at R79.1: now also J4.3 (D+)
- new net: J4.2 (D-), R5.1
Other:
- note added: "0.04pF at 250Mhz"
- note removed: "DNP"
- note removed: "Define if high speed USB device"
- moved on the sheet: C100, C101, C108, C115, C90, D15, D16, D19, FID1, FID2, H1, H2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

Commit message: saved
Parts:
- removed C14, C15: 100nF, Capacitor_SMD:C_0402_1005Metric, symbol Device:C
- removed R13: 100k, Resistor_SMD:R_0402_1005Metric, symbol Device:R
- removed U5: TXB0108DQSR, Package_SON:USON-20_2x4mm_P0.4mm, symbol Logic_LevelTranslator:TXB0108DQSR
- added C5, C7: 100nF, Capacitor_SMD:C_0402_1005Metric, symbol Device:C
- added R6: 100k, Resistor_SMD:R_0402_1005Metric, symbol Device:R
- added U3: TXB0108DQSR, Package_SON:USON-20_2x4mm_P0.4mm, symbol Logic_LevelTranslator:TXB0108DQSR
Connections:
- net 1V8: now also C7.1, U3.5 (VCCA), U3.6 (OE)
- net 3V3_ALWAYS_ON: now also C5.1, U3.16 (VCCB)
- net CTS_1V8: now also U3.4 (A4)
- net CTS_3V3: now also U3.17 (B4)
- net DCD_1V8: now also U3.7 (A5)
- net DCD_3V3: now also U3.14 (B5)
- net GND: now also C5.2, C7.2, R6.1, U3.15 (GND)
- net MODEM_DTR_1V8: now also U3.9 (A7)
- net MODEM_DTR_3V3: now also U3.12 (B7)
- net MODEM_RI_1V8: now also U3.8 (A6)
- net MODEM_RI_3V3: now also U3.13 (B6)
- net MODEM_RX_1V8: now also U3.1 (A1)
- net MODEM_RX_3V3: now also U3.20 (B1)
- net MODEM_TX_1V8: now also U3.2 (A2)
- net MODEM_TX_3V3: now also U3.19 (B2)
- net RTS_1V8: now also U3.3 (A3)
- net RTS_3V3: now also U3.18 (B3)
- net STATUS_LED: now also U3.10 (A8)
- net STATUS_LED_3V3: now also R6.2, U3.11 (B8)
Other:
- note added: "EG915U"
- note added: "Immobilizer & Ignition detect"
- note added: "Llv shifter GNSS IIC"
- note added: "RS485 auto tranciever"
- note added: "SIM CARD SLOT"
- note removed: "SIM CARD"
- moved on the sheet: C100, C101, C102, C103, C104, C105, C106, C107, C108, C110, C112, C115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

Commit message: saved
Parts:
- R1, R2, R3: footprint Resistor_SMD:R_0603_1608Metric -> Resistor_SMD:R_0402_1005Metric; MPN CRGCQ0603J22R -> RMCF0402ZT0R00
Changed lines of the file:
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@@
       (effects (font (size 1.27 1.27)))
     )
-    (property "Footprint" "Resistor_SMD:R_0603_1608Metric" (at 954.405 266.192 90)
+    (property "Footprint" "Resistor_SMD:R_0402_1005Metric" (at 954.405 266.192 90)
       (effects (font (size 1.27 1.27)) hide)
     )
@@
       (effects (font (size 1.27 1.27)) hide)
     )
-    (property "MPN" "CRGCQ0603J22R" (at 954.405 267.97 0)
+    (property "MPN" "RMCF0402ZT0R00" (at 954.405 267.97 0)
       (effects (font (size 1.27 1.27)) hide)
     )
@@
       (effects (font (size 1.27 1.27)))
     )
-    (property "Footprint" "Resistor_SMD:R_0603_1608Metric" (at 954.405 262.382 90)
+    (property "Footprint" "Resistor_SMD:R_0402_1005Metric" (at 954.405 262.382 90)
       (effects (font (size 1.27 1.27)) hide)
     )
@@
       (effects (font (size 1.27 1.27)) hide)
     )
-    (property "MPN" "CRGCQ0603J22R" (at 954.405 264.16 0)
+    (property "MPN" "RMCF0402ZT0R00" (at 954.405 264.16 0)
       (effects (font (size 1.27 1.27)) hide)
     )
@@
       (effects (font (size 1.27 1.27)))
     )
-    (property "Footprint" "Resistor_SMD:R_0603_1608Metric" (at 954.405 270.002 90)
+    (property "Footprint" "Resistor_SMD:R_0402_1005Metric" (at 954.405 270.002 90)
       (effects (font (size 1.27 1.27)) hide)
     )
@@
       (effects (font (size 1.27 1.27)) hide)
     )
-    (property "MPN" "CRGCQ0603J22R" (at 954.405 271.78 0)
+    (property "MPN" "RMCF0402ZT0R00" (at 954.405 271.78 0)
       (effects (font (size 1.27 1.27)) hide)
     )

Commit message: nrf flash done
Connections:
- net +100V renamed +60V_IN
Changed lines of the file:
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@@
     (stroke (width 0) (type default))
   )
-  (wire (pts (xy 332.74 30.48) (xy 332.74 31.75))
-    (stroke (width 0) (type default))
-  )
   (wire (pts (xy 45.72 322.58) (xy 55.88 322.58))
     (stroke (width 0) (type default))
@@
     )
   )
+  (symbol (lib_id "TC-Power:+60V_IN") (at 38.1 347.98 0) (unit 1)
+    (in_bom yes) (on_board yes) (dnp no) (fields_autoplaced)
+    (property "Reference" "#PWR014" (at 38.1 351.79 0)
+      (effects (font (size 1.27 1.27)) hide)
+    )
+    (property "Value" "+60V_IN" (at 38.1 342.9 0)
+      (effects (font (size 1.27 1.27)))
+    )
+    (property "Footprint" "" (at 38.1 347.98 0)
+      (effects (font (size 1.27 1.27)) hide)
+    )
+    (property "Datasheet" "" (at 38.1 347.98 0)
+      (effects (font (size 1.27 1.27)) hide)
+    )
+    (pin "1")
+    (instances
+      (project "roam"
+        (path "/e63e39d7-6ac0-4ffd-8aa3-1841a4541b55"
+          (reference "#PWR014") (unit 1)
+        )
+      )
+    )
+  )
   (symbol (lib_id "Device:C_Small") (at 631.19 543.56 0) (unit 1)
     (in_bom yes) (on_board yes) (dnp no)
@@
     )
   )
+  (symbol (lib_id "TC-Power:+60V_IN") (at 92.71 105.41 0) (unit 1)
+    (in_bom yes) (on_board yes) (dnp no) (fields_autoplaced)
+    (property "Reference" "#PWR093" (at 92.71 109.22 0)
+      (effects (font (size 1.27 1.27)) hide)
+    )
+    (property "Value" "+60V_IN" (at 92.71 100.33 0)
+      (effects (font (size 1.27 1.27)))
+    )
+    (property "Footprint" "" (at 92.71 105.41 0)
+      (effects (font (size 1.27 1.27)) hide)
+    )
+    (property "Datasheet" "" (at 92.71 105.41 0)
+      (effects (font (size 1.27 1.27)) hide)
+    )
+    (pin "1")
+    (instances
+      (project "roam"
+        (path "/e63e39d7-6ac0-4ffd-8aa3-1841a4541b55"
+          (reference "#PWR093") (unit 1)
+        )
+      )
+    )
+  )
   (symbol (lib_id "power:GND") (at 330.2 515.62 0) (unit 1)
     (in_bom yes) (on_board yes) (dnp no) (fields_autoplaced)
@@
     )
   )
-  (symbol (lib_id "TC-Power:+100V") (at 38.1 347.98 0) (unit 1)
-    (in_bom yes) (on_board yes) (dnp no) (fields_autoplaced)
-    (property "Reference" "#PWR0135" (at 38.1 351.79 0)
-      (effects (font (size 1.27 1.27)) hide)
-    )
-    (property "Value" "+60V" (at 38.1 344.17 0)
-      (effects (font (size 1.27 1.27)))
-    )
-    (property "Footprint" "" (at 38.1 347.98 0)
-      (effects (font (size 1.27 1.27)) hide)
-    )
-    (property "Datasheet" "" (at 38.1 347.98 0)
-      (effects (font (size 1.27 1.27)) hide)
-    )
-    (pin "1")
-    (instances
-      (project "roam"
-        (path "/e63e39d7-6ac0-4ffd-8aa3-1841a4541b55"
-          (reference "#PWR0135") (unit 1)
-        )
-      )
-    )
-  )
   (symbol (lib_id "power:GND") (at 318.77 135.89 0) (unit 1)
     (in_bom yes) (on_board yes) (dnp no) (fields_autoplaced)
@@
     )
   )
-  (symbol (lib_id "TC-Power:+100V") (at 19.05 24.13 0) (unit 1)
-    (in_bom yes) (on_board yes) (dnp no)
-    (property "Reference" "#PWR0145" (at 19.05 27.94 0)
-      (effects (font (size 1.27 1.27)) hide)
-    )
-    (property "Value" "+100V" (at 19.05 19.05 0)
-      (effects (font (size 1.27 1.27)))
-    )
-    (property "Footprint" "" (at 19.05 24.13 0)
-      (effects (font (size 1.27 1.27)) hide)
-    )
-    (property "Datasheet" "" (at 19.05 24.13 0)
-      (effects (font (size 1.27 1.27)) hide)
-    )
-    (pin "1")
-    (instances
-      (project "roam"
-        (path "/e63e39d7-6ac0-4ffd-8aa3-1841a4541b55"
-          (reference "#PWR0145") (unit 1)
-        )
-      )
-    )
-  )
   (symbol (lib_id "Device:C") (at 678.18 492.76 0) (mirror y) (unit 1)
     (in_bom yes) (on_board yes) (dnp no)
@@
     )
   )
+  (symbol (lib_id "TC-Power:+60V_IN") (at 19.05 24.13 0) (unit 1)
+    (in_bom yes) (on_board yes) (dnp no) (fields_autoplaced)
+    (property "Reference" "#PWR092" (at 19.05 27.94 0)
+      (effects (font (size 1.27 1.27)) hide)
+    )
+    (property "Value" "+60V_IN" (at 19.05 19.05 0)
+      (effects (font (size 1.27 1.27)))
+    )
+    (property "Footprint" "" (at 19.05 24.13 0)
+      (effects (font (size 1.27 1.27)) hide)
+    )
+    (property "Datasheet" "" (at 19.05 24.13 0)
+      (effects (font (size 1.27 1.27)) hide)
+    )
+    (pin "1")
+    (instances
+      (project "roam"
+        (path "/e63e39d7-6ac0-4ffd-8aa3-1841a4541b55"
+          (reference "#PWR092") (unit 1)
+        )
+      )
+    )
+  )
   (symbol (lib_id "Device:C") (at 264.16 119.38 0) (unit 1)
     (in_bom yes) (on_board yes) (dnp no) (fields_autoplaced)
@@
         )
       )
-    )
-  )
-  (symbol (lib_id "TC-Power:+100V") (at 92.71 105.41 0) (unit 1)
-    (in_bom yes) (on_board yes) (dnp no)
-    (property "Reference" "#PWR014" (at 92.71 109.22 0)
-      (effects (font (size 1.27 1.27)) hide)
-    )
-    (property "Value" "+60V" (at 92.71 100.33 0)
-      (effects (font (size 1.27 1.27)))
-    )
-    (property "Footprint" "" (at 92.71 105.41 0)
-      (effects (font (size 1.27 1.27)) hide)
-    )
-    (property "Datasheet" "" (at 92.71 105.41 0)
-      (effects (font (size 1.27 1.27)) hide)
-    )
-    (pin "1")
-    (instances
-      (project "roam"
-        (path "/e63e39d7-6ac0-4ffd-8aa3-1841a4541b55"
-          (reference "#PWR014") (unit 1)
-        )
-      )

Commit message: saved
Parts:
- removed J3: Conn_01x03_Pin, Connector_PinHeader_1.27mm:PinHeader_1x03_P1.27mm_Vertical_SMD_Pin1Left, symbol Connector:Conn_01x03_Pin
- removed TP18: USB_DM_T, TestPoint:TestPoint_Pad_D1.0mm, symbol Connector:TestPoint
- removed TP19: USB_DP_T, TestPoint:TestPoint_Pad_D1.0mm, symbol Connector:TestPoint
- removed TP20: USB_VBUS_T, TestPoint:TestPoint_Pad_D1.0mm, symbol Connector:TestPoint
- removed TP21: USB_GND, TestPoint:TestPoint_Pad_D1.0mm, symbol Connector:TestPoint
- removed U1: NUP4202, Package_TO_SOT_SMD:SOT-363_SC-70-6, symbol Power_Protection:NUP4202
- added D18, D22, D24, D25: ESD9C5.0ST5G, Diode_SMD:D_SOD-923, symbol Diode:ESD9B5.0ST5G
- added J3: Conn_01x03_Pin, Connector_PinHeader_1.27mm:PinHeader_1x02_P1.27mm_Vertical_SMD_Pin1Right, symbol Connector:Conn_01x02_Pin
- C56: footprint Capacitor_SMD:C_0603_1608Metric -> Capacitor_SMD:C_0402_1005Metric; MPN CL10B105KO8NNNC -> (none)
- C90: MPN C15850 -> (none)
- C91, C92: footprint Capacitor_SMD:C_0603_1608Metric -> Capacitor_SMD:C_0402_1005Metric; MPN GRM188R71A225KE15J -> 0402X225K100NT
- C96, C98: footprint Capacitor_SMD:C_0603_1608Metric -> Capacitor_SMD:C_0402_1005Metric; MPN GRM188R61E105K -> (none)
- J5: footprint Connector_PinHeader_1.27mm:PinHeader_1x03_P1.27mm_Vertical_SMD_Pin1Left -> Connector_PinHeader_1.27mm:PinHeader_1x02_P1.27mm_Vertical_SMD_Pin1Left; symbol Connector:Conn_01x03_Pin -> Connector:Conn_01x02_Pin
- R11, R16, R51, R56: footprint Resistor_SMD:R_0603_1608Metric -> Resistor_SMD:R_0402_1005Metric; MPN RC0603FR-072K8L -> (none)
- R26, R30: footprint Resistor_SMD:R_0603_1608Metric -> Resistor_SMD:R_0402_1005Metric
- R37, R38: footprint Resistor_SMD:R_0603_1608Metric -> Resistor_SMD:R_0402_1005Metric; MPN RC0603FR-074K7L -> (none)
- TP1, TP2, TP3, TP4, TP5, TP6, TP7, TP8, TP9: footprint TestPoint:TestPoint_Pad_D1.5mm -> TestPoint:TestPoint_Pad_D1.0mm
Connections:
- net CAN_250_H: now also J3.2 (Pin_2)
- net GND: now also D18.1 (A1), D22.1 (A1), D24.1 (A1), D25.1 (A1)
- net SIM_CHIP_CLK: now also C3.1, D22.2 (A2)
- net SIM_CHIP_DATA: now also C2.1, D18.2 (A2)
- net SIM_CHIP_RST: now also C4.1, D24.2 (A2)
- net SIM_CLK: no longer C3.1
- net SIM_DATA: no longer C2.1
- net SIM_RST: no longer C4.1
- net SIM_VDD: now also D25.2 (A2)
- net USB-: now reaches U27.10 (USB_DM), U29.4 (I/O2)
- net USB+: now reaches U27.9 (USB_DP), U29.6 (I/O1)
- net at R30.1: now also J3.1 (Pin_1)
- no-connect marks 85 -> 83
Other:
- moved on the sheet: C1, R1, R2, R3, R4

Commit message: saved 4/1
Parts:
- C102, C103, C41, C45, C6: footprint Capacitor_SMD:C_0603_1608Metric -> Capacitor_SMD:C_0402_1005Metric; MPN CL10A106MP8NNNC -> CL05A106MP8NUB8
- J4: footprint Connector_USB:USB_Micro-B_XKB_U254-051T-4BH83-F1S -> Connector_USB:USB_Micro-B_Molex_47346-0001
Connections:
- net CAN_250_H: now also J5.2 (Pin_2), L11.2, R16.1, R35.1; no longer J3.2 (Pin_2), L12.2, R51.1, R59.1
- net CAN_250_L: now also L11.3, R11.2, R26.2, R49.1; no longer L12.3, R30.2, R56.2, R60.1
- net CAN_500_H: now also J3.2 (Pin_2), L12.2, R51.1, R59.1; no longer J5.2 (Pin_2), L11.2, R16.1, R35.1
- net CAN_500_L: now also L12.3, R30.2, R56.2, R60.1; no longer L11.3, R11.2, R26.2, R49.1
- net VCU_CAN1_RX: now also U16.4 (RXD); no longer U6.4 (RXD)
- net VCU_CAN1_TX: now also U16.1 (TXD); no longer U6.1 (TXD)
- net VCU_CAN2_RX: now also U6.4 (RXD); no longer U16.4 (RXD)
- net VCU_CAN2_TX: now also U6.1 (TXD); no longer U16.1 (TXD)
Other:
- note added: "100n near VBAT, VDD_1 - VDD_4 10u near VDD_3"
- note removed: "100n near VBAT, VDD_1 - VDD_4 4.7u near VDD_3"
Changed lines of the file:
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@@
     (effects (font (size 1.27 1.27)) (justify left bottom))
   )
-  (text "100n near VBAT, VDD_1 - VDD_4 \n4.7u near VDD_3" (at 463.55 154.94 0)
+  (text "100n near VBAT, VDD_1 - VDD_4 \n10u near VDD_3" (at 463.55 154.94 0)
     (effects (font (size 1.27 1.27)) (justify left bottom))
   )
@@
     (effects (font (size 1.27 1.27)) (justify left bottom))
   )
-  (label "CAN_500_L" (at 572.77 360.68 180) (fields_autoplaced)
-    (effects (font (size 1.27 1.27)) (justify right bottom))
-  )
   (label "USB_VBUS" (at 1043.94 80.01 0) (fields_autoplaced)
     (effects (font (size 1.27 1.27)) (justify left bottom))
@@
     (effects (font (size 1.27 1.27)) (justify right bottom))
   )
-  (label "VCU_CAN1_RX" (at 411.48 346.075 0) (fields_autoplaced)
-    (effects (font (size 1.27 1.27)) (justify left bottom))
-  )
   (label "SWDIO" (at 191.77 213.36 180) (fields_autoplaced)
     (effects (font (size 1.27 1.27)) (justify right bottom))
   )
-  (label "VCU_CAN2_RX" (at 411.48 405.765 0) (fields_autoplaced)
-    (effects (font (size 1.27 1.27)) (justify left bottom))
+  (label "CAN_500_H" (at 571.5 396.24 180) (fields_autoplaced)
+    (effects (font (size 1.27 1.27)) (justify right bottom))
   )
   (label "ACC_INT" (at 300.99 196.85 0) (fields_autoplaced)
@@
     (effects (font (size 1.27 1.27)) (justify left bottom))
   )
+  (label "CAN_500_L" (at 571.5 420.37 180) (fields_autoplaced)
+    (effects (font (size 1.27 1.27)) (justify right bottom))
+  )
   (label "GNSS_ANT" (at 1064.26 504.19 180) (fields_autoplaced)
     (effects (font (size 1.27 1.27)) (justify right bottom))
@@
     (effects (font (size 1.27 1.27)) (justify left bottom))
   )
-  (label "VCU_SWDIO" (at 477.52 212.09 180) (fields_autoplaced)
-    (effects (font (size 1.27 1.27)) (justify right bottom))
+  (label "VCU_CAN1_TX" (at 411.48 403.225 0) (fields_autoplaced)
+    (effects (font (size 1.27 1.27)) (justify left bottom))
   )
-  (label "CAN_500_H" (at 572.77 336.55 180) (fields_autoplaced)
+  (label "VCU_SWDIO" (at 477.52 212.09 180) (fields_autoplaced)
     (effects (font (size 1.27 1.27)) (justify right bottom))
   )
@@
     (effects (font (size 1.27 1.27)) (justify left bottom))
   )
-  (label "CAN_250_H" (at 571.5 396.24 180) (fields_autoplaced)
-    (effects (font (size 1.27 1.27)) (justify right bottom))
-  )
   (label "MODEM_RX_3V3" (at 713.74 281.94 180) (fields_autoplaced)
     (effects (font (size 1.27 1.27)) (justify right bottom))
@@
     (effects (font (size 1.27 1.27)) (justify left bottom))
   )
-  (label "VCU_CAN2_TX" (at 411.48 403.225 0) (fields_autoplaced)
-    (effects (font (size 1.27 1.27)) (justify left bottom))
-  )
   (label "MODEM_DTR_1V8" (at 650.24 297.18 0) (fields_autoplaced)
     (effects (font (size 1.27 1.27)) (justify left bottom))
@@
     (effects (font (size 1.27 1.27)) (justify left bottom))
   )
+  (label "CAN_250_L" (at 572.77 360.68 180) (fields_autoplaced)
+    (effects (font (size 1.27 1.27)) (justify right bottom))
+  )
   (label "FLASH_SCK" (at 100.33 217.17 0) (fields_autoplaced)
     (effects (font (size 1.27 1.27)) (justify left bottom))
@@
     (effects (font (size 1.27 1.27)) (justify left bottom))
   )
-  (label "CAN_250_L" (at 571.5 420.37 180) (fields_autoplaced)
-    (effects (font (size 1.27 1.27)) (justify right bottom))
+  (label "VCU_CAN2_RX" (at 411.48 346.075 0) (fields_autoplaced)
+    (effects (font (size 1.27 1.27)) (justify left bottom))
   )
   (label "RTS_1V8" (at 892.81 137.16 0) (fields_autoplaced)
@@
     (effects (font (size 1.27 1.27)) (justify left bottom))
   )
+  (label "CAN_250_H" (at 572.77 336.55 180) (fields_autoplaced)
+    (effects (font (size 1.27 1.27)) (justify right bottom))
+  )
   (label "LC29_RESET_ESP32" (at 201.93 275.59 180) (fields_autoplaced)
     (effects (font (size 1.27 1.27)) (justify right bottom))
@@
     (effects (font (size 1.27 1.27)) (justify left bottom))
   )
+  (label "VCU_CAN2_TX" (at 411.48 343.535 0) (fields_autoplaced)
+    (effects (font (size 1.27 1.27)) (justify left bottom))
+  )
   (label "RTS_1V8" (at 650.24 287.02 0) (fields_autoplaced)
     (effects (font (size 1.27 1.27)) (justify left bottom))
@@
     (effects (font (size 1.27 1.27)) (justify right bottom))
   )
-  (label "VCU_CAN1_TX" (at 411.48 343.535 0) (fields_autoplaced)
-    (effects (font (size 1.27 1.27)) (justify left bottom))
-  )
   (label "VCU_USART2_RTS" (at 96.52 234.95 0) (fields_autoplaced)
     (effects (font (size 1.27 1.27)) (justify left bottom))
@@
     (effects (font (size 1.27 1.27)) (justify right bottom))
   )
+  (label "VCU_CAN1_RX" (at 411.48 405.765 0) (fields_autoplaced)
+    (effects (font (size 1.27 1.27)) (justify left bottom))
+  )
   (label "CTS_3V3" (at 96.52 247.65 0) (fields_autoplaced)
     (effects (font (size 1.27 1.27)) (justify left bottom))
@@
       (effects (font (size 1.27 1.27)) (justify left))
     )
-    (property "Footprint" "Capacitor_SMD:C_0603_1608Metric" (at 697.5348 546.1 0)
+    (property "Footprint" "Capacitor_SMD:C_0402_1005Metric" (at 697.5348 546.1 0)
       (effects (font (size 1.27 1.27)) hide)
     )
@@
       (effects (font (size 1.27 1.27)) hide)
     )
-    (property "Description" "CAP CER 10UF 10V X5R 0603" (at 698.5 542.29 0)
+    (property "Description" "CAP CER 10UF 10V X5R 0402" (at 698.5 542.29 0)
       (effects (font (size 1.27 1.27)) hide)
     )
@@
       (effects (font (size 1.27 1.27)) hide)
     )
-    (property "MPN" "CL10A106MP8NNNC" (at 698.5 542.29 0)
+    (property "MPN" "CL05A106MP8NUB8" (at 698.5 542.29 0)
       (effects (font (size 1.27 1.27)) hide)
     )
@@
       (effects (font (size 1.27 1.27)) (justify left))
     )
-    (property "Footprint" "Capacitor_SMD:C_0603_1608Metric" (at 701.3448 492.76 0)
+    (property "Footprint" "Capacitor_SMD:C_0402_1005Metric" (at 701.3448 492.76 0)
       (effects (font (size 1.27 1.27)) hide)
     )
@@
       (effects (font (size 1.27 1.27)) hide)
     )
-    (property "Description" "CAP CER 10UF 10V X5R 0603" (at 702.31 488.95 0)
+    (property "Description" "CAP CER 10UF 10V X5R 0402" (at 702.31 488.95 0)
       (effects (font (size 1.27 1.27)) hide)
     )
@@
       (effects (font (size 1.27 1.27)) hide)
     )
-    (property "MPN" "CL10A106MP8NNNC" (at 702.31 488.95 0)
+    (property "MPN" "CL05A106MP8NUB8" (at 702.31 488.95 0)
       (effects (font (size 1.27 1.27)) hide)
     )
@@
       (effects (font (size 1.27 1.27)))
     )
-    (property "Footprint" "Capacitor_SMD:C_0603_1608Metric" (at 321.0052 198.12 0)
+    (property "Footprint" "Capacitor_SMD:C_0402_1005Metric" (at 321.0052 198.12 0)
       (effects (font (size 1.27 1.27)) hide)
     )
@@
       (effects (font (size 1.27 1.27)) hide)
     )
-    (property "MPN" "CL10A106MP8NNNC" (at 320.04 194.31 0)
+    (property "MPN" "CL05A106MP8NUB8" (at 320.04 194.31 0)
       (effects (font (size 1.27 1.27)) hide)
     )
@@
       (effects (font (size 1.27 1.27)) hide)
     )
-    (property "Description" "CAP CER 10UF 10V X5R 0603" (at 320.04 194.31 0)
+    (property "Description" "CAP CER 10UF 10V X5R 0402" (at 320.04 194.31 0)
       (effects (font (size 1.27 1.27)) hide)
     )
@@
       (effects (font (size 1.27 1.27)) (justify left))
     )
-    (property "Footprint" "Capacitor_SMD:C_0603_1608Metric" (at 202.2348 213.995 0)
+    (property "Footprint" "Capacitor_SMD:C_0402_1005Metric" (at 202.2348 213.995 0)
       (effects (font (size 1.27 1.27)) hide)
     )
@@
       (effects (font (size 1.27 1.27)) hide)
     )
-    (property "Description" "CAP CER 10UF 10V X5R 0603" (at 203.2 210.185 0)
+    (property "Description" "CAP CER 10UF 10V X5R 0402" (at 203.2 210.185 0)
       (effects (font (size 1.27 1.27)) hide)
     )
@@
       (effects (font (size 1.27 1.27)) hide)
     )
-    (property "MPN" "CL10A106MP8NNNC" (at 203.2 210.185 0)
+    (property "MPN" "CL05A106MP8NUB8" (at 203.2 210.185 0)
       (effects (font (size 1.27 1.27)) hide)
     )
@@
       (effects (font (size 1.27 1.27)) (justify left))
     )
-    (property "Footprint" "Capacitor_SMD:C_0603_1608Metric" (at 504.19 162.56 0)
+    (property "Footprint" "Capacitor_SMD:C_0402_1005Metric" (at 504.19 162.56 0)
       (effects (font (size 1.27 1.27)) hide)
     )
@@
       (effects (font (size 1.27 1.27)) hide)
     )
-    (property "Description" "CAP CER 10UF 10V X5R 0603" (at 504.19 162.56 0)
+    (property "Description" "CAP CER 10UF 10V X5R 0402" (at 504.19 162.56 0)
       (effects (font (size 1.27 1.27)) hide)
     )
@@
       (effects (font (size 1.27 1.27)) hide)
     )
-    (property "MPN" "CL10A106MP8NNNC" (at 504.19 162.56 0)
+    (property "MPN" "CL05A106MP8NUB8" (at 504.19 162.56 0)
       (effects (font (size 1.27 1.27)) hide)
     )
@@
       (effects (font (size 1.27 1.27)))
     )
-    (property "Footprint" "Connector_USB:USB_Micro-B_XKB_U254-051T-4BH83-F1S" (at 628.65 184.15 0)
+    (property "Footprint" "Connector_USB:USB_Micro-B_Molex_47346-0001" (at 628.65 184.15 0)
       (effects (font (size 1.27 1.27)) hide)
     )

Commit message: updated 4/12
Parts:
- J3: footprint Connector_PinHeader_1.27mm:PinHeader_1x02_P1.27mm_Vertical_SMD_Pin1Right -> Connector_PinHeader_1.27mm:PinHeader_1x02_P1.27mm_Vertical_SMD_Pin1Left
Connections:
- net CAN_250_H: now also D20.2 (A2)
- net CAN_250_L: now also D20.1 (A1)
- net CAN_500_H: now also D21.2 (A2)
- net CAN_500_L: now also D21.1 (A1)
- net at L12.1, R59.2, U16.7 (CANH): no longer D21.2 (A2)
- net at L12.4, R60.2, U16.6 (CANL): no longer D21.1 (A1)
- net at L11.4, R49.2, U6.6 (CANL): no longer D20.1 (A1)
- net at L11.1, R35.2, U6.7 (CANH): no longer D20.2 (A2)
Other:
- moved on the sheet: C16, C80, J3, J5, L11, L12, R11, R16, R26, R30, R35, R49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
