File: roam.kicad_sch (KiCad schematic)
At the start: 301 parts, among them IC2 MCP73833T-FCI/MF, J1 SIM8060-6-0-14-00-A, J2 Battery, J3 Conn_01x03_Pin, J4 USB_B_Micro, J5 Conn_01x03_Pin, J7 MX23A18NF1, Q2 MMBT3904, Q3 MMBT3904, Q5 BC846A,215, Q6 BC846A,215, Q7 BC846A,215, U10 LTV-217, U11 MAX13487EESAT, U12 LM3671MF-3.3/NOPB, U13 LIS2DH12TR, U14 MAX17643ATC+, U15 FDMC86139P, U16 MCP2562-E/MF, U17 LTV-217, U18 MP3423GG, U2 MDBT50Q-1M, U20 TPS566242DRLR, U23 TXS0102DCU, U24 LP5907MFX-3.3, U27 EG915ULAAB-N05-SNNSA, U28 LC29H, U29 USBLC6-2SC6, U3 TXB0108DQSR, U31 B8389, U32 LP5907MFX-3.3, U4 STM32F105RBT6, U6 MCP2562-E/MF, U6 MX25R6435FZNIL0, U6 W25N512GVEIG, U7 LM66100DCKR, U8 GP.1575.25.2.A.02, U9 LM66100DCKR, Y1 25MHz

Commit message: Printed
Parts:
- removed R100, R12: 0, Resistor_SMD:R_0402_1005Metric, symbol Device:R_Small
- added L1, L6: 0nH, Inductor_SMD:L_0402_1005Metric, symbol Device:L_Small
- C100: value 100nF -> 10nF; MPN CL05B104KP5NNNC -> (none)
- R5, R79: value 20 -> 0
- R60, R61: MPN (none) -> PFR05S-102-FNH
- U28: value LC29H -> LC29HAAMD
- U31: value B8389 -> B39162B8389P810
Connections:
- net GND: now also L1.2
- net RF_ANT: now also L1.1
- net at C116.1, L10.2: now also L6.1
- net at C117.1, L13.2: now also L6.2
Changed lines of the file:
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@@
     (stroke (width 0) (type dash))
   )
-  (wire (pts (xy 660.4 115.57) (xy 669.29 115.57))
-    (stroke (width 0) (type default))
-  )
   (wire (pts (xy 203.2 190.5) (xy 203.2 204.47))
     (stroke (width 0) (type default))
@@
     (stroke (width 0) (type default))
   )
+  (wire (pts (xy 659.765 115.57) (xy 669.29 115.57))
+    (stroke (width 0) (type default))
+  )
   (wire (pts (xy 351.79 401.955) (xy 351.79 415.29))
     (stroke (width 0) (type default))
@@
     (stroke (width 0) (type default))
   )
-  (wire (pts (xy 648.97 115.57) (xy 655.32 115.57))
+  (wire (pts (xy 648.97 115.57) (xy 654.685 115.57))
     (stroke (width 0) (type default))
   )
@@
     (effects (font (size 1.27 1.27)) (justify left bottom))
   )
-  (text "NO CAP in spec" (at 873.76 64.77 0)
-    (effects (font (size 1.27 1.27)) (justify left bottom))
-  )
   (text "ACTIVE_LOW" (at 94.615 485.14 0)
     (effects (font (size 1.27 1.27)) (justify left bottom))
@@
       (effects (font (size 1.27 1.27)))
     )
-    (property "Value" "100nF" (at 880.11 73.66 0)
+    (property "Value" "10nF" (at 880.11 73.66 0)
       (effects (font (size 1.27 1.27)))
     )
@@
       (effects (font (size 1.27 1.27)) hide)
     )
-    (property "MPN" "CL05B104KP5NNNC" (at 876.3 71.12 0)
+    (property "MPN" "" (at 876.3 71.12 0)
       (effects (font (size 1.27 1.27)) hide)
     )
-    (property "Description" "CAP CER 0.1UF 10V X7R 0402" (at 876.3 71.12 0)
+    (property "Description" "CAP CER 0.01UF 10V X7R 0402" (at 876.3 71.12 0)
       (effects (font (size 1.27 1.27)) hide)
     )
@@
       (effects (font (size 1.27 1.27)))
     )
-    (property "Value" "B8389" (at 1037.59 495.3 0)
+    (property "Value" "B39162B8389P810" (at 1037.59 495.3 0)
       (effects (font (size 1.27 1.27)))
     )
@@
       (effects (font (size 1.27 1.27)))
     )
-    (property "Value" "LC29H" (at 900.43 383.54 0)
+    (property "Value" "LC29HAAMD" (at 900.43 383.54 0)
       (effects (font (size 1.27 1.27)))
     )
@@
   (symbol (lib_id "Device:R") (at 665.48 182.88 90) (unit 1)
     (in_bom yes) (on_board yes) (dnp no)
-    (property "Reference" "R79" (at 670.56 180.34 90)
+    (property "Reference" "R79" (at 672.465 181.61 90)
       (effects (font (size 1.27 1.27)) (justify left))
     )
-    (property "Value" "20" (at 666.623 181.102 90)
+    (property "Value" "0" (at 666.623 181.102 90)
       (effects (font (size 1.27 1.27)) (justify left))
     )
@@
     )
   )
+  (symbol (lib_id "Device:L_Small") (at 657.225 115.57 90) (unit 1)
+    (in_bom yes) (on_board yes) (dnp no)
+    (property "Reference" "L1" (at 655.955 111.76 0)
+      (effects (font (size 1.27 1.27)))
+    )
+    (property "Value" "0nH" (at 653.415 113.03 0)
+      (effects (font (size 1.27 1.27)))
+    )
+    (property "Footprint" "Inductor_SMD:L_0402_1005Metric" (at 657.225 115.57 0)
+      (effects (font (size 1.27 1.27)) hide)
+    )
+    (property "Datasheet" "~" (at 657.225 115.57 0)
+      (effects (font (size 1.27 1.27)) hide)
+    )
+    (property "Description" "" (at 657.225 115.57 0)
+      (effects (font (size 1.27 1.27)) hide)
+    )
+    (property "MPN" "" (at 657.225 115.57 0)
+      (effects (font (size 1.27 1.27)) hide)
+    )
+    (pin "1")
+    (pin "2")
+    (instances
+      (project "roam"
+        (path "/e63e39d7-6ac0-4ffd-8aa3-1841a4541b55"
+          (reference "L1") (unit 1)
+        )
+      )
+    )
+  )
   (symbol (lib_id "Device:R") (at 384.175 179.07 270) (unit 1)
     (in_bom yes) (on_board yes) (dnp no)
@@
     )
   )
-  (symbol (lib_id "Device:R_Small") (at 979.17 504.19 90) (unit 1)
-    (in_bom yes) (on_board yes) (dnp no)
-    (property "Reference" "R100" (at 981.71 506.73 90)
-      (effects (font (size 1.27 1.27)) (justify left))
-    )
-    (property "Value" "0" (at 980.44 504.19 90)
-      (effects (font (size 1.27 1.27)) (justify left))
-    )
-    (property "Footprint" "Resistor_SMD:R_0402_1005Metric" (at 979.17 504.19 0)
-      (effects (font (size 1.27 1.27)) hide)
-    )
-    (property "Datasheet" "~" (at 979.17 504.19 0)
-      (effects (font (size 1.27 1.27)) hide)
-    )
-    (property "MPN" "RMCF0402ZT0R00" (at 979.17 504.19 90)
-      (effects (font (size 1.27 1.27)) hide)
-    )
-    (property "Description" "RES 0 OHM JUMPER 1/16W 0402" (at 979.17 504.19 0)
-      (effects (font (size 1.27 1.27)) hide)
-    )
-    (pin "1")
-    (pin "2")
-    (instances
-      (project "roam"
-        (path "/e63e39d7-6ac0-4ffd-8aa3-1841a4541b55"
-          (reference "R100") (unit 1)
-        )
-      )
-    )
-  )
   (symbol (lib_id "Device:R") (at 826.77 516.89 270) (unit 1)
     (in_bom yes) (on_board yes) (dnp no)
@@
     )
   )
+  (symbol (lib_id "Device:L_Small") (at 979.17 504.19 90) (unit 1)
+    (in_bom yes) (on_board yes) (dnp no)
+    (property "Reference" "L6" (at 977.9 500.38 0)
+      (effects (font (size 1.27 1.27)))
+    )
+    (property "Value" "0nH" (at 975.36 501.65 0)
+      (effects (font (size 1.27 1.27)))
+    )
+    (property "Footprint" "Inductor_SMD:L_0402_1005Metric" (at 979.17 504.19 0)
+      (effects (font (size 1.27 1.27)) hide)
+    )
+    (property "Datasheet" "~" (at 979.17 504.19 0)
+      (effects (font (size 1.27 1.27)) hide)
+    )
+    (property "Description" "" (at 979.17 504.19 0)
+      (effects (font (size 1.27 1.27)) hide)
+    )
+    (property "MPN" "" (at 979.17 504.19 0)
+      (effects (font (size 1.27 1.27)) hide)
+    )
+    (pin "1")
+    (pin "2")
+    (instances
+      (project "roam"
+        (path "/e63e39d7-6ac0-4ffd-8aa3-1841a4541b55"
+          (reference "L6") (unit 1)
+        )
+      )
+    )
+  )
   (symbol (lib_id "power:GND") (at 99.695 541.02 0) (unit 1)
     (in_bom yes) (on_board yes) (dnp no)
@@
     )
   )
-  (symbol (lib_id "Device:R_Small") (at 657.86 115.57 90) (unit 1)
-    (in_bom yes) (on_board yes) (dnp no)
-    (property "Reference" "R12" (at 660.4 118.11 90)
-      (effects (font (size 1.27 1.27)) (justify left))
-    )
-    (property "Value" "0" (at 659.13 115.57 90)
-      (effects (font (size 1.27 1.27)) (justify left))
-    )
-    (property "Footprint" "Resistor_SMD:R_0402_1005Metric" (at 657.86 115.57 0)
-      (effects (font (size 1.27 1.27)) hide)
-    )
-    (property "Datasheet" "~" (at 657.86 115.57 0)
-      (effects (font (size 1.27 1.27)) hide)
-    )
-    (property "MPN" "RMCF0402ZT0R00" (at 657.86 115.57 90)
-      (effects (font (size 1.27 1.27)) hide)
-    )
-    (property "Description" "RES 0 OHM JUMPER 1/16W 0402" (at 657.86 115.57 0)
-      (effects (font (size 1.27 1.27)) hide)
-    )
-    (pin "1")
-    (pin "2")
-    (instances
-      (project "roam"
-        (path "/e63e39d7-6ac0-4ffd-8aa3-1841a4541b55"
-          (reference "R12") (unit 1)
-        )
-      )
-    )
-  )
   (symbol (lib_id "Device:R_Small") (at 124.46 46.99 90) (unit 1)
     (in_bom yes) (on_board yes) (dnp no)
@@
   (symbol (lib_id "Device:R") (at 665.48 185.42 90) (unit 1)
     (in_bom yes) (on_board yes) (dnp no)
-    (property "Reference" "R5" (at 670.56 182.88 90)
+    (property "Reference" "R5" (at 671.195 186.69 90)
       (effects (font (size 1.27 1.27)) (justify left))
     )
-    (property "Value" "20" (at 666.75 188.595 90)
+    (property "Value" "0" (at 666.75 188.595 90)
       (effects (font (size 1.27 1.27)) (justify left))
     )
@@
       (effects (font (size 1.27 1.27)) hide)
     )
+    (property "MPN" "PFR05S-102-FNH" (at 293.37 551.18 0)
+      (effects (font (size 1.27 1.27)) hide)
+    )
     (pin "1")
     (pin "2")
@@
       (effects (font (size 1.27 1.27)) hide)
     )
+    (property "MPN" "PFR05S-102-FNH" (at 229.87 551.18 0)
+      (effects (font (size 1.27 1.27)) hide)
+    )
