File: orange_compact.kicad_pcb (KiCad board)
At the start: 6 copper layers, 60 x 50 mm, 235 parts, among them IC4 MAX13487EESA+T, J1 Battery, J2 Conn_Coaxial, J3 Conn_Coaxial, J4 USB_B_Micro, J6 USB_B_Micro, J7 Conn_01x11_Pin, Q12 Q_NPN_BEC_BRT, Q2 Q_NPN_BEC_BRT, Q5 Q_NPN_BEC_BRT, Q6 Q_NPN_BEC_BRT, Q8 Q_NPN_BEC_BRT, SW1 SW_Push, SW2 SW_Push, U1 EG916QGLLG-N03-SGNSA, U10 LP5907MFX-3.3, U11 TXB0104RUT, U13 LIS2DH12TR, U14 LP5907MFX-1.8, U15 LM66100DCKR, U16 LM66100DCKR, U18 TPS61022, U19 LTV-217, U2 TXB0102DCU, U20 TPS566242DRLR, U22 TP4056, U25 ESP32-S3-MINI-1, U26 MCP2562-E/MF, U27 LP5907MFX-3.3, U28 USBLC6-2SC6, U29 TXB0108RGY, U4 LP5907MFX-3.3, U5 LTV-217, U6 LMR14030SDDAR, U7 LP5907MFX-3.3, U8 1NCE IoT SIMs Chip, U9 USBLC6-2SC6

Commit message: changed
Routing:
- net VBAT: track 38.2 -> 29.9 mm, vias 2 -> 0
- net 5V0_BUCK: track 143.8 -> 144.8 mm, vias 7 -> 8
- net +1V8: track 10.5 -> 11.0 mm
- net GND: vias 208 -> 210

Commit message: lite v3 done
Parts:
- added TP28: TestPoint, TestPoint:TestPoint_Pad_D1.0mm, B.Cu at (159.4, 73.8)
- moved C1 0.35 mm to (149.1, 87.5)
Routing:
- net VBAT: track 29.9 -> 36.9 mm, vias 0 -> 1
- net GND: track 4.44 -> 7.16 mm, vias 210 -> 232
- net /GNSS_RST_3V3: track 11.3 -> 10.7 mm
Other:
- board text added: "IO3"
- board text added: "IO34"
- board text added: "IO37"
- board text added: "RXD"
- board text added: "TXD"
- board text removed: "CON"
- board text removed: "GNSS"
- board text removed: "PWR"
- board text removed: "RX"
- board text removed: "TX"

Commit message: saved
Parts:
- removed C114, C118, C60, C66, C85: 100nF, Capacitor_SMD:C_0402_1005Metric
- removed C62, C63, C64, C86: 33pF, Inductor_SMD:L_0402_1005Metric
- removed C65, C67: 10nF, Capacitor_SMD:C_0402_1005Metric
- removed C68, C98, C99: 1uF, Capacitor_SMD:C_0402_1005Metric
- removed C71: 2.2uF, Capacitor_SMD:C_0402_1005Metric
- removed C84, C87: 10pF, Capacitor_SMD:C_0402_1005Metric
- removed CP4, CP5: 100u, Capacitor_Tantalum_SMD:CP_EIA-6032-28_Kemet-C
- removed D15, D23: LED, LED_SMD:LED_0603_1608Metric
- removed D20, D21, D22, D24: D4V5H1BS2LP-7B, Diode_SMD:D_0402_1005Metric
- removed L4: 2.2uH, Inductor_SMD:L_Bourns-SRN4018
- removed Q12, Q5, Q6, Q8: Q_NPN_BEC_BRT, Package_TO_SOT_SMD:SOT-23
- removed R36: 10k, Resistor_SMD:R_0402_1005Metric
- removed R40: 169k, Resistor_SMD:R_0402_1005Metric
- removed R41: 30k, Resistor_SMD:R_0402_1005Metric
- removed R53: 15k, Resistor_SMD:R_0402_1005Metric
- removed R58, R59: 20, Resistor_SMD:R_0402_1005Metric
- removed R64: 4k7, Resistor_SMD:R_0402_1005Metric
- removed R70, R71, R78: 750, Resistor_SMD:R_0603_1608Metric
- removed TP11, TP12, TP13, TP9: TestPoint, TestPoint:TestPoint_Pad_D1.0mm
- removed TP19: gnss_tx, TestPoint:TestPoint_Pad_D1.0mm
- removed TP20: gnss_rx, TestPoint:TestPoint_Pad_D1.0mm
- removed TP21: gnss_en, TestPoint:TestPoint_Pad_D1.0mm
- removed U20: TPS566242DRLR, TC-Power:TPS566242DRLR
- removed U29: TXB0108RGY, Package_DFN_QFN:Texas_RGY_R-PVQFN-N20_EP2.05x3.05mm
- removed U8: 1NCE IoT SIMs Chip, Package_DFN_QFN:DFN-8-1EP_6x5mm_P1.27mm_EP4x4mm
- added C10: 33pF, Inductor_SMD:L_0402_1005Metric, F.Cu at (222.2, 103.2)
- added C12: 33pF, Inductor_SMD:L_0402_1005Metric, F.Cu at (222.2, 101.2)
- added C16: 10nF, Capacitor_SMD:C_0402_1005Metric, F.Cu at (269.0, 75.5)
- added C17: 10nF, Capacitor_SMD:C_0402_1005Metric, F.Cu at (269.0, 77.5)
- added C18: 33pF, Inductor_SMD:L_0402_1005Metric, F.Cu at (222.2, 99.2)
- added C21: 2.2uF, Capacitor_SMD:C_0402_1005Metric, F.Cu at (269.0, 79.4)
- added C22: 100nF, Capacitor_SMD:C_0402_1005Metric, F.Cu at (269.0, 81.4)
- added C23: 1uF, Capacitor_SMD:C_0402_1005Metric, F.Cu at (223.6, 68.9)
- added C28: 100nF, Capacitor_SMD:C_0402_1005Metric, F.Cu at (271.9, 75.5)
- added C30: 10pF, Capacitor_SMD:C_0402_1005Metric, F.Cu at (271.9, 77.5)
- added C31: 3.9pF, Capacitor_SMD:C_0402_1005Metric, F.Cu at (271.9, 79.4)
- added C36: 100nF, Capacitor_SMD:C_0402_1005Metric, F.Cu at (271.9, 81.4)
- added C38: 22uF, Capacitor_SMD:C_0805_2012Metric, F.Cu at (290.3, 74.0)
- added C40: 22uF, Capacitor_SMD:C_0805_2012Metric, F.Cu at (290.3, 77.0)
- added C41: 22uF, Capacitor_SMD:C_0805_2012Metric, F.Cu at (290.3, 80.1)
- added C8: 100nF, Capacitor_SMD:C_0402_1005Metric, F.Cu at (222.4, 106.1)
- added CP2: 100u, Capacitor_Tantalum_SMD:CP_EIA-6032-28_Kemet-C, F.Cu at (277.6, 82.1)
- added D2: D4V5H1BS2LP-7B, Diode_SMD:D_0402_1005Metric, F.Cu at (269.3, 83.4)
- added D7: D4V5H1BS2LP-7B, Diode_SMD:D_0402_1005Metric, F.Cu at (269.3, 85.4)
- added J5: USB_B_Micro, Connector_USB:USB_Micro-B_Molex-105017-0001, F.Cu at (220.1, 63.6)
- added J7: Conn_01x11_Pin, Connector_JST:JST_XH_B11B-XH-A_1x11_P2.50mm_Vertical, F.Cu at (154.1, 99.1)
- added JP2: Jumper_2_Bridged, Resistor_SMD:R_0805_2012Metric, F.Cu at (164.1, 92.1)
- added L1: 2.2uH, Inductor_SMD:L_Bourns-SRN4018, F.Cu at (291.1, 84.3)
- added Q1: Q_NPN_BEC_BRT, Package_TO_SOT_SMD:SOT-23, F.Cu at (285.6, 74.9)
- added Q3: Q_NPN_BEC_BRT, Package_TO_SOT_SMD:SOT-23, F.Cu at (285.6, 79.6)
- added R1: 15k, Resistor_SMD:R_0402_1005Metric, F.Cu at (222.2, 97.3)
- added R14: 20, Resistor_SMD:R_0402_1005Metric, F.Cu at (216.8, 70.0)
- added R16: 20, Resistor_SMD:R_0402_1005Metric, F.Cu at (216.8, 68.0)
- added R18: 10k, Resistor_SMD:R_0402_1005Metric, F.Cu at (289.7, 65.2)
- added R19: 169k, Resistor_SMD:R_0402_1005Metric, F.Cu at (289.7, 67.2)
- added R20: 30k, Resistor_SMD:R_0402_1005Metric, F.Cu at (289.7, 69.1)
- added R21: 100k, Resistor_SMD:R_0402_1005Metric, F.Cu at (188.4, 76.8)
- added R23: 47k, Resistor_SMD:R_0402_1005Metric, F.Cu at (186.4, 76.7)
- added R24: 330, Resistor_SMD:R_0603_1608Metric, F.Cu at (196.6, 88.9)
- added R25: 10k, Resistor_SMD:R_0402_1005Metric, F.Cu at (292.6, 65.2)
- added R7: 4k7, Resistor_SMD:R_0402_1005Metric, F.Cu at (286.7, 69.1)
- added R8: 750, Resistor_SMD:R_0603_1608Metric, F.Cu at (285.2, 83.0)
- added U17: MIC29302WU, Package_TO_SOT_SMD:TO-263-5_TabPin3, F.Cu at (181.8, 84.3)
- C1, C102, C103, C104, C115, C117, C119, C120, C48, C49, C5, C54, C58, C72, C73, D12, D16, D17, IC4, J4, L11, L15, R3, R31, R32, R33, R35, R43, R44, R45, R47, R48, R57, R60, R61, R79, R80, R93, R94, TP25, TP26, U18, U19, U2, U25, U27, U28, U5, U9: moved to F.Cu
- C29, C37: value 100nF -> 33pF; footprint Capacitor_SMD:C_0402_1005Metric -> Inductor_SMD:L_0402_1005Metric
- C32: value 33pF -> 1.8pF; footprint Inductor_SMD:L_0402_1005Metric -> Capacitor_SMD:C_0402_1005Metric
- C39: value 33pF -> 22uF; footprint Inductor_SMD:L_0402_1005Metric -> Capacitor_SMD:C_0805_2012Metric
- C42: value 22uF -> 100nF; footprint Capacitor_SMD:C_0805_2012Metric -> Capacitor_SMD:C_0402_1005Metric
- C43: value 22uF -> 470uF; footprint Capacitor_SMD:C_0805_2012Metric -> Capacitor_SMD:CP_Elec_6.3x7.7
- C50: value 22uF -> 220uF; footprint Capacitor_SMD:C_0805_2012Metric -> Capacitor_SMD:CP_Elec_6.3x7.7
- C51: value 22uF -> 100nF; footprint Capacitor_SMD:C_0805_2012Metric -> Capacitor_SMD:C_0603_1608Metric
- C52: footprint Capacitor_SMD:C_0402_1005Metric -> Capacitor_SMD:C_0603_1608Metric
- H1, H2, H3, H4: value MountingHole -> MountingHole_with_conection; footprint MountingHole:MountingHole_2.7mm_M2.5_DIN965_Pad -> MountingHole:MountingHole_2.7mm_M2.5_DIN965_Pad_TopBottom
- J6: value USB_B_Micro -> EG800; footprint Connector_USB:USB_Micro-B_Molex-105017-0001 -> TC-RF-module:XCVR_EG800Q-EU; moved to F.Cu
- J7: footprint Connector_PinHeader_2.00mm:PinHeader_1x11_P2.00mm_Vertical -> Connector_JST:JST_XH_B11B-XH-A_1x11_P2.50mm_Vertical
- U1: value EG916QGLLG-N03-SGNSA -> 1NCE IoT SIMs Chip; footprint TC-RF-module:XCVR_EG9xQ -> Package_DFN_QFN:DFN-8-1EP_6x5mm_P1.27mm_EP4x4mm; moved to F.Cu
- U11: value TXB0104RUT -> TXB0108RGY; footprint Package_DFN_QFN:Texas_R-PUQFN-N12 -> Package_DFN_QFN:Texas_RGY_R-PVQFN-N20_EP2.05x3.05mm
- U14: value LP5907MFX-1.8 -> TPS566242DRLR; footprint Package_TO_SOT_SMD:SOT-23-5 -> TC-Power:TPS566242DRLR
- moved C117 126.8 mm to (270.9, 111.6), turned to 0 degrees
- moved H4 126.1 mm to (247.5, 115.8)
- moved D5 124.4 mm to (271.1, 107.1), turned to 180 degrees
- moved H1 123.4 mm to (247.5, 63.8)
- moved R65 122.9 mm to (271.1, 105.5), turned to 0 degrees
- moved D4 119.5 mm to (271.0, 102.0), turned to 180 degrees
- moved R10 118.0 mm to (271.0, 100.4), turned to 0 degrees
- moved D3 113.8 mm to (270.9, 95.8), turned to 180 degrees
- moved R9 112.4 mm to (270.9, 94.2), turned to 0 degrees
- moved TP4 111.2 mm to (271.6, 91.8), turned to 90 degrees
- moved L11 100.3 mm to (223.8, 141.4)
- moved R93 99.8 mm to (239.9, 110.8), turned to 90 degrees
- moved J1 99.6 mm to (237.1, 114.9)
- moved R94 96.6 mm to (238.3, 110.7), turned to -90 degrees
- moved C115 93.9 mm to (236.9, 111.3), turned to -90 degrees
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Connections:
- C32 pad 1: 4V0 -> GND
- C32 pad 2: GND -> 4V0
- C37 pad 1: 5V0 -> 4V0
- C37 pad 2: GND -> Net-(U14-FB)
- C39 pad 2: Net-(U20-FB) -> GND
- C43 pad 1: 4V0 -> 5V0
- C52 pad 1: 4V0 -> 5V0
- H1 pad 1: (no net) -> GND
- H2 pad 1: (no net) -> GND
- H3 pad 1: (no net) -> GND
- H4 pad 1: (no net) -> GND
- J6 pad 1: /USB_VBUS -> GND
- J6 pad 2: Net-(J6-D-) -> unconnected-(J6A-GNSS_ANT-Pad2)
- J6 pad 3: Net-(J6-D+) -> unconnected-(J6B-RESERVED-Pad3)
- J6 pad 5: GND -> unconnected-(J6B-RESERVED-Pad5)
- J6 pad 6: GND -> unconnected-(J6B-RESERVED-Pad6)
- Q2 pad 1: /NET_LED -> /PWRKEY
- Q2 pad 3: Net-(Q2-C) -> Net-(J6A-~{PWRKEY})
- R37 pad 1: 3V3_CONM -> 3V3_ALWAYS_ON
- R38 pad 1: 3V3_CONM -> 3V3_ALWAYS_ON
- TP1 pad 1: Net-(U1-GNSS_DBG_TXD) -> Net-(D2-K)
- TP10 pad 1: Net-(D22-K) -> Net-(D7-K)
- U1 pad 1: /PSM_IND -> GND
- U1 pad 3: GND -> /SIM_DATA
- U1 pad 6: unconnected-(U1-PCM_DIN-Pad6) -> /SIM_CLK
- U1 pad 7: unconnected-(U1-PCM_DOUT-Pad7) -> /SIM_RST
- U1 pad 8: /USB_VBUS -> /SIM_VDD
- U1 pad 9: Net-(U1-USB_DP) -> (no net)
- U11 pad 1: +1V8 -> /MODEM_TX_1V8
- U11 pad 10: /GNSS_EN_3V3 -> VDD_EXT
- U11 pad 11: 3V3_CONM -> GND
- U11 pad 12: +1V8 -> /STATUS_LED_3V3
- U11 pad 2: /GNSS_EN_1V8 -> VDD_EXT
- U11 pad 3: /GNSS_RST_1V8 -> /MODEM_RX_1V8
- U11 pad 4: /GNSS_TXD_1V8 -> /RTS_1V8
- U11 pad 5: /GNSS_RXD_1V8 -> /CTS_1V8
- U11 pad 6: GND -> /DCD_1V8
- U11 pad 7: /GNSS_RXD_3V3 -> /MODEM_RI_1V8
- U11 pad 8: /GNSS_TXD_3V3 -> /MODEM_DTR_1V8
- U11 pad 9: /GNSS_RST_3V3 -> /STATUS_LED
- U14 pad 1: 3V3_ALWAYS_ON -> 5V0
- U14 pad 2: GND -> Net-(U14-SW)
- U14 pad 3: /GNSS_EN_3V3 -> GND
- U14 pad 4: unconnected-(U14-NC-Pad4) -> GND
- U14 pad 5: +1V8 -> /U20_EN
- U25 pad 20: /U20_EN -> /Modem_EN
- U9 pad 4: Net-(U1-USB_DP) -> Net-(J6A-USB_DP)
- U9 pad 6: Net-(U1-USB_DM) -> Net-(J6A-USB_DM)
Routing:
- net GND: track 7.16 -> 221.9 mm, vias 232 -> 236
- net (no net): track 0.00 -> 100.6 mm, vias 0 -> 15
- net 3V3_ALWAYS_ON: track 120.4 -> 57.7 mm
- net /SDA: track 64.3 -> 3.72 mm
- net /SCL: track 63.4 -> 3.87 mm
- net 5V0: track 136.5 -> 77.2 mm
- net /3V3_COMU_EN: track 60.0 -> 3.65 mm
- net 5V0_BUCK: track 144.8 -> 98.6 mm
- net /GPS_ANT_EN: track 44.8 -> 1.76 mm
- net 3V3_CONM: track 110.9 -> 71.8 mm
- net /CAN_SHDN: track 40.7 -> 2.56 mm
- net /CAN_500_L: track 43.4 -> 5.31 mm
- net /CAN_500_H: track 42.5 -> 5.68 mm
- net /CAN_RXD: track 37.4 -> 1.74 mm
- net /NRESET: track 35.2 -> 1.28 mm, vias 4 -> 1
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- added copper zone on F.Cu, net (none)
- added copper zone on F.Cu, net 4V7_BOOST
- added copper zone on F.Cu, net Net-(U18-SW)
- added copper zone on F.Cu, net VBAT
- removed copper zone on B.Cu, net 4V7_BOOST
- removed copper zone on In3.Cu, net GND
- removed copper zone on In4.Cu, net GND
- removed copper zone on B.Cu, net Net-(U18-SW)
- removed copper zone on F.Cu, net Net-(U20-SW)
- removed copper zone on B.Cu, net VBAT
Other:
- board size 60 x 50 mm -> 189.4 x 81.8 mm
- copper layers 6 -> 4

Commit message: saved
Parts:
- removed C35: 47uF, Inductor_SMD:L_1206_3216Metric
- removed C36, C42: 100nF, Capacitor_SMD:C_0402_1005Metric
- removed C37: 33pF, Inductor_SMD:L_0402_1005Metric
- removed C38, C39, C40, C41: 22uF, Capacitor_SMD:C_0805_2012Metric
- removed L1: 2.2uH, Inductor_SMD:L_Bourns-SRN4018
- removed R18: 10k, Resistor_SMD:R_0402_1005Metric
- removed R19: 169k, Resistor_SMD:R_0402_1005Metric
- removed R20: 30k, Resistor_SMD:R_0402_1005Metric
- removed TP14, TP15: TestPoint, TestPoint:TestPoint_Pad_D1.0mm
- removed U14: TPS566242DRLR, TC-Power:TPS566242DRLR
- removed U7: LP5907MFX-3.3, Package_TO_SOT_SMD:SOT-23-5
- added C56: 100nF, Capacitor_SMD:C_0402_1005Metric, F.Cu at (212.4, 68.4)
- added C59: 10uF, Capacitor_SMD:C_0603_1608Metric, F.Cu at (195.1, 95.2)
- added C60: 100nF, Capacitor_SMD:C_0402_1005Metric, F.Cu at (196.5, 94.7)
- added C62: 33pF, Inductor_SMD:L_0402_1005Metric, F.Cu at (197.6, 94.7)
- added C63: 33pF, Inductor_SMD:L_0402_1005Metric, F.Cu at (196.6, 99.4)
- added C64: 1uF, Capacitor_SMD:C_0402_1005Metric, F.Cu at (206.0, 68.1)
- added C65: 1uF, Capacitor_SMD:C_0402_1005Metric, F.Cu at (211.3, 68.5)
- added D21: ESD56151W04, Diode_SMD:D_SOD-323, F.Cu at (199.2, 95.3)
- added D22: ESD56151W04, Diode_SMD:D_SOD-323, F.Cu at (199.1, 98.9)
- added JP4: SolderJumper_2_Open, Jumper:SolderJumper-2_P1.3mm_Open_RoundedPad1.0x1.5mm, F.Cu at (210.3, 110.3)
- added Q6: Q_NPN_BEC_BRT, Package_TO_SOT_SMD:SOT-23, F.Cu at (198.2, 106.2)
- added R26: 0, Resistor_SMD:R_0603_1608Metric, F.Cu at (197.5, 84.7)
- added R29: 4k7, Resistor_SMD:R_0402_1005Metric, F.Cu at (210.1, 108.0)
- added R34: 0, Resistor_SMD:R_0402_1005Metric, F.Cu at (209.7, 96.5)
- added R36: 0, Resistor_SMD:R_0402_1005Metric, F.Cu at (208.4, 96.5)
- added U20: LC79H, TC-RF-module:XCVR_LC79H, F.Cu at (206.1, 101.5)
- added U21: LP5907MFX-3.3, Package_TO_SOT_SMD:SOT-23-5, F.Cu at (208.7, 68.8)
- C116, C13, C2, C29, C32, C9, D1, D13, D19, J2, J3, L10, L13, L6, R100, R12, R4: moved to F.Cu
- C3: value 2.2uF -> 10uF; footprint Capacitor_SMD:C_0402_1005Metric -> Capacitor_SMD:C_0603_1608Metric
- C4: value 1uF -> 100nF
- C50: value 220uF -> 470uF
- JP1: moved to B.Cu
- moved L6 128.7 mm to (206.4, 113.6)
- moved J2 128.3 mm to (202.7, 117.4), turned to 90 degrees
- moved Q2 127.2 mm to (232.7, 104.9)
- moved C2 127.0 mm to (207.0, 112.0), turned to -90 degrees
- moved R4 127.0 mm to (205.9, 112.0), turned to 90 degrees
- moved D13 125.2 mm to (203.2, 114.8)
- moved C116 123.5 mm to (202.8, 113.3), turned to -90 degrees
- moved D11 122.9 mm to (222.1, 77.5), turned to 180 degrees
- moved L10 121.9 mm to (202.3, 111.8)
- moved R100 120.3 mm to (202.8, 110.3), turned to 90 degrees
- moved L13 118.7 mm to (202.4, 108.8)
- moved R25 108.8 mm to (185.8, 86.4), turned to 90 degrees
- moved JP1 107.6 mm to (205.5, 74.0)
- moved D14 102.0 mm to (219.6, 72.1), turned to 90 degrees
- moved C96 100.5 mm to (242.2, 78.8), turned to 180 degrees
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Connections:
- C3 pad 1: 5V0 -> VCC_LC760Z
- C4 pad 1: 3V3_ANT -> GND
- C4 pad 2: GND -> VCC_LC760Z
- J6 pad 42: 4V0 -> /VBAT_RF
- J6 pad 43: 4V0 -> /VBAT_RF
- R7 pad 2: VDD_EXT -> GND
- U25 pad 17: /GPS_ANT_EN -> unconnected-(U25-IO13-Pad17)
- U25 pad 27: /GNSS_RST_3V3 -> /GNSS_RESET
- U25 pad 38: /GNSS_RXD_3V3 -> /GNSS_RXD
- U25 pad 41: /GNSS_TXD_3V3 -> /GNSS_TXD
- U25 pad 44: /GNSS_EN_3V3 -> /GNSS_EN
Routing:
- net GND: track 221.9 -> 53.7 mm
- net 4V0: track 130.4 -> 47.3 mm
- net /RXD0: track 58.6 -> 19.5 mm
- net (no net): track 100.6 -> 137.2 mm, vias 15 -> 25
- net /SIM_VDD: track 10.2 -> 39.5 mm
- net /USB_VBUS: track 34.2 -> 60.2 mm, vias 0 -> 2
- net /SIM_DATA: track 26.5 -> 48.8 mm
- net /DCD_3V3: track 25.7 -> 40.6 mm
- net /GNSS_EN_3V3: track 14.6 -> 0.00 mm, vias 3 -> 0
- net /MODEM_RI_3V3: track 6.72 -> 21.1 mm, vias 1 -> 3
- net Net-(J6A-USB_DP): track 19.9 -> 33.5 mm, vias 0 -> 2
- net /MODEM_DTR_3V3: track 8.41 -> 21.5 mm
- net 5V0: track 77.2 -> 64.2 mm
- net /CTS_3V3: track 23.6 -> 36.3 mm, vias 1 -> 3
- net VDD_EXT: track 23.3 -> 36.0 mm
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Other:
- board text added: "E4C"
- board text added: "ORANGE LITE"
- board text removed: "ORANGE LITE V3"

Commit message: saved
Parts:
- removed the J7 at (63.6, 72.1)
- moved C100 14.3 mm to (168.5, 93.3)
- moved R36 6.18 mm to (212.7, 101.0), turned to 0 degrees
- moved U16 5.42 mm to (165.7, 96.7), turned to 0 degrees
- moved C82 5.28 mm to (156.1, 108.9)
- moved C78 5.28 mm to (156.1, 105.7)
- moved C80 5.28 mm to (156.2, 107.3)
- moved C81 5.28 mm to (159.3, 108.8)
- moved C77 5.28 mm to (159.2, 105.7)
- moved C79 5.28 mm to (159.2, 107.3)
- moved U15 5.26 mm to (165.7, 93.3), turned to 0 degrees
- moved R29 4.65 mm to (209.7, 112.7)
- moved R34 4.54 mm to (212.7, 99.9), turned to 0 degrees
- moved CP2 4.47 mm to (194.3, 82.2), turned to 0 degrees
- moved C28 4.42 mm to (190.6, 87.0)
- moved C32 4.10 mm to (194.9, 87.0), turned to 90 degrees
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Routing:
- net 4V0: track 47.3 -> 81.7 mm
- net 5V0_BUCK: track 98.6 -> 129.8 mm
- net 5V0: track 64.2 -> 95.4 mm
- net Net-(C83-Pad1): track 28.3 -> 56.3 mm
- net V_EXT: track 15.1 -> 38.5 mm
- net VIN: track 19.6 -> 33.4 mm
- net Net-(D10-K): track 3.86 -> 7.99 mm
- net /GNSS_BOOT: track 0.00 -> 3.40 mm
- net Net-(U6-EN): track 4.28 -> 7.27 mm
- net Net-(U18-FB): track 3.05 -> 5.96 mm
- net Net-(U6-SS): track 2.14 -> 4.38 mm
- net Net-(C81-Pad2): track 1.59 -> 3.17 mm
- net Net-(C77-Pad2): track 1.55 -> 3.10 mm
- net Net-(C79-Pad2): track 1.53 -> 3.05 mm
