File: orange_compact.kicad_sch (KiCad schematic)
At the start: 221 parts, among them IC1 MCP25625-E_ML, IC3 MIC5317-1.8YD5-TR, IC4 MAX13487EESA+T, IC5 MC74HC4060A, J4 Conn_Coaxial, J5 Conn_01x08_Pin, J6 USB_B_Micro, Q2 MMBT3904, Q3 MMBT3904, Q5 MMBT3904, Q6 BC846A,215, Q7 BC846A,215, U1 EG9xQ, U12 LM3671MF-3.3/NOPB, U13 LIS2DH12TR, U2 MDBT50Q-1M, U20 TPS566242DRLR, U3 FDMC86139P, U4 LM5012DDAR, U5 TXB0108DQSR, U6 MX25R6435FZNIL0, U8 1NCE IoT SIMs Chip, U9 USBLC6-2SC6, Y1 16MHz

Commit message: saved
Parts:
- added C11, C2, C3: DNP, Capacitor_SMD:C_0402_1005Metric, symbol Device:C_Small
- added C24: 4.7uF, Capacitor_SMD:C_0603_1608Metric, symbol Device:C_Small
- added C4: 24pF, Capacitor_SMD:C_0402_1005Metric, symbol Device:C_Small
- added C46: 100nF, Capacitor_SMD:C_0603_1608Metric, symbol Device:C
- added J1: U.FL-R-SMT-1-GNSS_ANT, TC-Connector:coax-u.fl, symbol Connector:Conn_Coaxial
- added L6: 47nH, Inductor_SMD:L_0402_1005Metric, symbol Device:L_Small
- added R4: 10, Resistor_SMD:R_0402_1005Metric, symbol Device:R
- added U6: SIP32408DNP-T1-GE4, TC-ICs:SON50P120X160X60-5N(TDFN-4), symbol TC-ICs:SiP32408
Connections:
- net GND: now also C11.2, C2.2, C24.2, C3.2, C46.2, J1.2 (Ext), U6.2 (GND), U6.5 (GND)
- net GNSS_ANT: now also C3.1, C4.1
- new net: L6.1, R4.1
- new net: C11.1, C4.2, J1.1 (In), L6.2
- new net 3V3: C24.1, U6.1 (IN)
- new net 3V3_ANT: C2.1, C46.1, R4.2, U6.4 (OUT)
- new net GPS_ANT_EN: U6.3 (EN)
Other:
- note added: "GPS antenna an PI-network"
- note added: "GPS antenna power filter?"
- moved on the sheet: C116, D13, J4, L10, L13, R100

Commit message: SAVED
Parts:
- removed C11, C3: DNP, Capacitor_SMD:C_0402_1005Metric, symbol Device:C_Small
- removed C4: 24pF, Capacitor_SMD:C_0402_1005Metric, symbol Device:C_Small
- removed J1: U.FL-R-SMT-1-GNSS_ANT, TC-Connector:coax-u.fl, symbol Connector:Conn_Coaxial
Connections:
- net 3V3 is gone; now on net 3V3_ALWAYS_ON: C24.1, U6.1 (IN)
- net GPS_ANT_EN: now also U2.49 (P0.25)
- net at C116.2, D13.2 (A2), J4.1 (In): now also L6.2
- no-connect marks 60 -> 59
Other:
- note removed: "GPS antenna an PI-network"
- moved on the sheet: C116, C24, C46, D13, FID1, FID2, H1, H2, H3, H4, J4, L10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

Commit message: Added gnss power
Parts:
- removed C24: 4.7uF, Capacitor_SMD:C_0603_1608Metric, symbol Device:C_Small
- removed C46: 100nF, Capacitor_SMD:C_0603_1608Metric, symbol Device:C
- removed U6: SIP32408DNP-T1-GE4, TC-ICs:SON50P120X160X60-5N(TDFN-4), symbol TC-ICs:SiP32408
- added C3: 2.2uF, Capacitor_SMD:C_0402_1005Metric, symbol Device:C_Small
- added C4: 1uF, Capacitor_SMD:C_0402_1005Metric, symbol Device:C
- added U7: LP5907MFX-3.3, Package_TO_SOT_SMD:SOT-23-5, symbol Regulator_Linear:LP5907MFX-3.3
- C116: value 33nF -> 24pf
- C2: value DNP -> 100pf
- IC3: footprint SOT95P280X130-5N -> TC-ICs:SOT95P280X130-5N; symbol MIC5317-1_8YM5:MIC5317-1.8YM5 -> TC-ICs:MIC5317-1.8YM5; Height (none) -> 1.3; Manufacturer_Part_Number (none) -> MIC5317-1.8YM5
- IC5: symbol CD4060BPWR:CD4060BPWR -> TC-ICs:CD4060BPWR; Arrow Part Number (none) -> CD4060BPWR; Arrow Price/Stock (none) -> https://www.arrow.com/en/products/cd4060bpwr/texas-instrume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; Height (none) -> 1.2; Manufacturer_Name (none) -> Texas Instruments; Manufacturer_Part_Number (none) -> CD4060BPWR; Mouser Part Number (none) -> 595-CD4060BPWR; Mouser Price/Stock (none) -> https://www.mouser.co.uk/ProductDetail/Texas-Instruments/CD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
- L6: value 47nH -> 51nH
Connections:
- net 3V3_ANT: now also C4.1, U7.5 (OUT)
- net 5V0: now also C3.1, U7.1 (IN)
- net GND: now also C3.2, C4.2, U7.2 (GND)
- net GPS_ANT_EN: now also U7.3 (EN)
Other:
- note removed: "GPS antenna power filter?"

Commit message: update bom info
Parts:
- IC5: value MC74HC4060A -> CD4060BPWR; MPN MC74HC4060A -> CD4060BPWR
- L1: value L_Ferrite_Coupled_1243 -> CMA0805A681R-1A
- U1: value EG9xQ -> EG916QGLLG-N03-SGNSA; MPN EG91xQ -> EG916QGLLG-N03-SGNSA
Changed lines of the file:
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@@
 				)
 				(justify left)
-				(hide yes)
 			)
 		)
@@
 			)
 		)
-		(property "Value" "MC74HC4060A"
+		(property "Value" "CD4060BPWR"
 			(at 345.44 99.06 0)
 			(effects
@@
 			)
 		)
-		(property "MPN" "MC74HC4060A"
+		(property "MPN" "CD4060BPWR"
 			(at 355.6 699.06 0)
 			(effects
@@
 			)
 		)
-		(property "Value" "L_Ferrite_Coupled_1243"
+		(property "Value" "CMA0805A681R-1A"
 			(at 459.105 201.93 0)
 			(effects
@@
 			)
 		)
-		(property "Value" "EG9xQ"
+		(property "Value" "EG916QGLLG-N03-SGNSA"
 			(at 729.615 254.635 0)
 			(effects
@@
 			)
 		)
-		(property "Description" "\nLTE Cat 1 module\n"
+		(property "Description" "LTE Cat 1 module"
 			(at 731.52 247.65 0)
 			(effects
@@
 			)
 		)
-		(property "MPN" "EG91xQ"
+		(property "MPN" "EG916QGLLG-N03-SGNSA  "
 			(at 731.52 273.05 0)
 			(effects

Commit message: save 11/9
Parts:
- removed C13: 100nF, Capacitor_SMD:C_0402_1005Metric, symbol Device:C_Small
- removed C14: 1uF, Capacitor_SMD:C_0402_1005Metric, symbol Device:C_Small
- removed D1: SMCJ75A, digikey-footprints:DO-214AB, symbol Diode:1N62xxCA
- removed D5: MM3Z18VT1G, Diode_SMD:D_SOD-323F, symbol Diode:MM3Zxx
- removed IC3: MIC5317-1.8YD5-TR, TC-ICs:SOT95P280X130-5N, symbol TC-ICs:MIC5317-1.8YM5
- removed IC5: CD4060BPWR, SOP65P640X120-16N, symbol TC-ICs:CD4060BPWR
- removed Q5: MMBT3904, Package_TO_SOT_SMD:SOT-23, symbol Transistor_BJT:MMBT3904
- removed R19: 182k, Resistor_SMD:R_0805_2012Metric, symbol Device:R_Small
- removed R23: 220k, Resistor_SMD:R_0805_2012Metric, symbol Device:R_Small
- removed R23: 41k2, Resistor_SMD:R_0603_1608Metric, symbol Device:R_Small
- removed R23: 49k9, Resistor_SMD:R_0603_1608Metric, symbol Device:R_Small
- removed R23: 158k, Resistor_SMD:R_0603_1608Metric, symbol Device:R_Small
- removed R23: 20k, Resistor_SMD:R_1206_3216Metric, symbol Device:R_Small
- removed R23 (x2): 120k, Resistor_SMD:R_0805_2012Metric, symbol Device:R_Small
- removed R50: 10k, Resistor_SMD:R_0402_1005Metric, symbol Device:R
- removed U12: LM3671MF-3.3/NOPB, Package_TO_SOT_SMD:SOT-23-5, symbol TC-Power:LM3671MFX-1.8
- added C100, C101, C105, C110, C111, C112, C113, C55: 100nF, Capacitor_SMD:C_0402_1005Metric, symbol Device:C_Small
- added C102: 10UF, Capacitor_SMD:C_0805_2012Metric, symbol Device:C
- added C103, C104: 47UF, Capacitor_SMD:C_0805_2012Metric, symbol Device:C
- added C106, C107: 1uF, Capacitor_SMD:C_0603_1608Metric, symbol Device:C
- added C108, C109: 10UF, Capacitor_SMD:C_0603_1608Metric, symbol Device:C
- added C11: 4.7u, Capacitor_SMD:C_2220_5750Metric, symbol Device:C_Small
- added C114: 1nF, Capacitor_SMD:C_0402_1005Metric, symbol Device:C_Small
- added C24: 8.2nf, Capacitor_SMD:C_0402_1005Metric, symbol Device:C_Small
- added C46: 0.1uF, Capacitor_SMD:C_0402_1005Metric, symbol Device:C_Small
- added C47: 270pF, Capacitor_SMD:C_0201_0603Metric, symbol Device:C_Small
- added C57, C76: 47uF, Capacitor_SMD:C_1210_3225Metric, symbol Device:C_Small
- added C59, C97, C98, C99: 1uF, Capacitor_SMD:C_0402_1005Metric, symbol Device:C_Small
- added C77, C78: 100PF, Capacitor_SMD:C_0603_1608Metric, symbol Device:C
- added C79, C80: 1nF, Capacitor_SMD:C_0603_1608Metric, symbol Device:C
- added C81, C82: 10nF, Capacitor_SMD:C_0603_1608Metric, symbol Device:C
- added C83, C88, C89, C94: 100nF, Capacitor_SMD:C_0603_1608Metric, symbol Device:C
- added C90, C91: 220uF, Capacitor_SMD:C_Elec_6.3x7.7, symbol Device:C_Polarized
- added C92, C93: 10u, Capacitor_SMD:C_0805_2012Metric, symbol Device:C_Small
- added C95, C96: 1uF, Capacitor_SMD:C_0402_1005Metric, symbol Device:C
- added D10: D_Schottky, Package_TO_SOT_SMD:TO-277A_alt, symbol Device:D_Schottky
- added D12: SM712_SOT23, Package_TO_SOT_SMD:SOT-323_SC-70, symbol Diode:SM712_SOT23
- added D6: SMCJ75A, digikey-footprints:DO-214AB, symbol Diode:1N62xxCA
- added D8: MM3Z18VT1G, Diode_SMD:D_SOD-323F, symbol Diode:MM3Zxx
- added D9: D_Schottky, Diode_SMD:D_PowerDI-5, symbol Device:D_Schottky
- added IC2: MIC5317-1.8YD5-TR, TC-ICs:SOT95P280X130-5N, symbol TC-ICs:MIC5317-1.8YM5
- added IC3: CD4060BPWR, SOP65P640X120-16N, symbol TC-ICs:CD4060BPWR
- added IC5: MCP73833T-FCI/MF, TC-ICs:SON50P300X300X100-11N-D, symbol TC-ICs:MCP73833-CNI_MF
- added J1: Battery, Connector_Molex:Molex_PicoBlade_53048-0310_1x03_P1.25mm_Horizontal, symbol Connector:Conn_01x03_Male
- added JP2: Jumper_2_Bridged, Jumper:SolderJumper-2_P1.3mm_Bridged2Bar_RoundedPad1.0x1.5mm, symbol Jumper:Jumper_2_Bridged
- added L11, L12: 1uH, Inductor_SMD:L_Coilcraft_XAL4020-XXX, symbol Device:L
- added L14: L_Ferrite_Coupled_1243, Inductor_SMD:L_CommonModeChoke_Laird_CMA0805, symbol Device:L_Ferrite_Coupled_1243
- added L7: 2.7UH, TC-DC-DC:IND_1255AY-2R7N=P3, symbol Device:L_Small
- added L8, L9: 33UH, Inductor_SMD:L_Changjiang_FNR5040S, symbol Device:L_Small
- added Q1: MMBT3904, Package_TO_SOT_SMD:SOT-23, symbol Transistor_BJT:MMBT3904
- added R11: 20k, Resistor_SMD:R_1206_3216Metric, symbol Device:R_Small
- added R14: 220k, Resistor_SMD:R_0805_2012Metric, symbol Device:R_Small
- added R15: 68K, Resistor_SMD:R_0402_1005Metric, symbol Device:R_Small
- added R17, R18: 120k, Resistor_SMD:R_0805_2012Metric, symbol Device:R_Small
- added R19: 10k, Resistor_SMD:R_0402_1005Metric, symbol Device:R
- added R20: 41k2, Resistor_SMD:R_0603_1608Metric, symbol Device:R_Small
- added R21: 182k, Resistor_SMD:R_0805_2012Metric, symbol Device:R_Small
- added R22: 12K, Resistor_SMD:R_0402_1005Metric, symbol Device:R_Small
- added R27: 412K, Resistor_SMD:R_0402_1005Metric, symbol Device:R_Small
- added R28, R85: 51K, Resistor_SMD:R_0402_1005Metric, symbol Device:R_Small
- added R29: 158k, Resistor_SMD:R_0603_1608Metric, symbol Device:R_Small
- added R49: 49k9, Resistor_SMD:R_0603_1608Metric, symbol Device:R_Small
- added R5: 10.5K, Resistor_SMD:R_0402_1005Metric, symbol Device:R_Small
- added R50: 0, Resistor_SMD:R_0402_1005Metric, symbol Device:R_Small
- added R79: 649K, Resistor_SMD:R_0402_1005Metric, symbol Device:R_Small
- added R80: 100K, Resistor_SMD:R_0402_1005Metric, symbol Device:R_Small
- added R81, R82: 4K7, Resistor_SMD:R_0603_1608Metric, symbol Device:R_Small
- added R83: 2k, Resistor_SMD:R_0603_1608Metric, symbol Device:R_Small
- added R84: 3.9K, Resistor_SMD:R_0402_1005Metric, symbol Device:R_Small
- added R86: 4K, Resistor_SMD:R_0402_1005Metric, symbol Device:R_Small
- added R87: 0.5, Resistor_SMD:R_0603_1608Metric, symbol Device:R_Small
- added R88, R89: 0, Resistor_SMD:R_0402_1005Metric, symbol Device:R
- added R90, R91: 2k8, Resistor_SMD:R_0402_1005Metric, symbol Device:R_Small
- added TH1: DNP, Resistor_SMD:R_0603_1608Metric, symbol Device:Thermistor_NTC
- added U10: LP5907MFX-3.3, Package_TO_SOT_SMD:SOT-23-5, symbol Regulator_Linear:LP5907MFX-3.3
- added U11: LM3671MF-3.3/NOPB, Package_TO_SOT_SMD:SOT-23-5, symbol TC-Power:LM3671MFX-1.8
- added U12: AMS1117-1.8, Package_TO_SOT_SMD:SOT-223-3_TabPin2, symbol Regulator_Linear:AMS1117-1.8
- added U14: LP5907MFX-1.8, Package_TO_SOT_SMD:SOT-23-5, symbol Regulator_Linear:LP5907MFX-1.8
- added U15, U16: LM66100DCKR, Package_TO_SOT_SMD:SOT-363_SC-70-6, symbol TC-ICs:LM66100
- added U17: TPS3828-33DBVRG4, Package_TO_SOT_SMD:SOT-23-5, symbol TC-ICs:TPS3828-33DBVRG4
- added U18: TPS61022, Package_DFN_QFN:Texas_RWU0007A_VQFN-7_2x2mm_P0.5mm, symbol Converter_DCDC:TPS61022
- added U21: SN74LVC1G14DBV, Package_TO_SOT_SMD:SOT-23-5, symbol 74xGxx:SN74LVC1G14DBV
- added U22: TP4056, TC-ICs:SO08-PAD-300, symbol TC-ICs:TP4056
- added U23: MCP2515-xST, Package_SO:TSSOP-20_4.4x6.5mm_P0.65mm, symbol Interface_CAN_LIN:MCP2515-xST
- added U24: MCP2562-E-MF, Package_DFN_QFN:DFN-8-1EP_3x3mm_P0.65mm_EP1.55x2.4mm, symbol Interface_CAN_LIN:MCP2562-E-MF
- added U25: MCP2562-E/MF, Package_DFN_QFN:DFN-8-1EP_3x3mm_P0.65mm_EP1.55x2.4mm, symbol Interface_CAN_LIN:MCP2562-E-MF
- added U6: LMR14030SDDAR, TC-DC-DC:LMR14030DDAR_SOIC8, symbol TC-ICs:LMR14030SDDAR
- C23: value 2.2n -> 100nF; MPN GRM155R72A222KA01D -> CL05B104KP5NNNC
- C25: value 100p -> 47u; footprint Capacitor_SMD:C_0603_1608Metric -> Capacitor_SMD:C_1206_3216Metric; MPN GRM1885C2A101JA01D -> CL31A476MPHNNNE; desc (none) -> 10V
- C26: value 3.3n -> 2.2n; MPN GRM155R72A332KA01D -> GRM155R72A222KA01D
- C27: value 22u -> 100p; MPN C1608X5R1A226M080AC -> GRM1885C2A101JA01D
- C28: value 22u -> 3.3n; footprint Capacitor_SMD:C_0603_1608Metric -> Capacitor_SMD:C_0402_1005Metric; MPN C1608X5R1A226M080AC -> GRM155R72A332KA01D
- C53: value 47u -> 22u; footprint Capacitor_SMD:C_1206_3216Metric -> Capacitor_SMD:C_0603_1608Metric; MPN CL31A476MPHNNNE -> C1608X5R1A226M080AC; desc 10V -> (none)
- C56: value 100nF -> 22u; footprint Capacitor_SMD:C_0402_1005Metric -> Capacitor_SMD:C_0603_1608Metric; MPN CL05B104KP5NNNC -> C1608X5R1A226M080AC
- R2: value 1M -> 100k; MPN RC0402FR-071ML -> 667-ERJ-2RKF1003X
- R3: value 100k -> 1M; MPN 667-ERJ-2RKF1003X -> RC0402FR-071ML
- R34: value 100k -> 220k; MPN 667-ERJ-2RKF1003X -> ERJ-2GEJ224X
- R52: value 220k -> 100k; MPN ERJ-2GEJ224X -> 667-ERJ-2RKF1003X
Connections:
- net +1V8: now also C75.1, C99.1, IC2.5 (VOUT), U14.5 (OUT); no longer C74.1
- net 3V3_ALWAYS_ON: now also C74.1, C101.1, C105.1, C112.2, C55.1, C96.1, C98.1, IC2.1 (VIN), IC3.16 (VDD), R81.2, R82.2, U10.5 (OUT), U11.4 (FB), U14.1 (IN), U17.3 (~{MR}), U17.5 (VDD), U21.5 (VCC), U25.5 (Vio); no longer C75.1
- net 5V0: now also C28.2, C53.1, C56.1, C113.2, C95.1, R29.1, U10.1 (IN), U10.3 (EN), U11.1 (VIN), U15.6 (VOUT), U16.6 (VOUT), U25.3 (VDD); no longer C26.2, C27.1, C28.1
- net GND: now also C23.2, C25.2, R2.2, R52.2, C100.2, C101.2, C102.2, C103.2, C104.2, C105.2, C106.2, C107.2, C108.2, C109.2, C11.2, C110.2, C111.2, C112.1, C113.1, C114.2, C24.2, C55.2, C57.2, C76.2, C78.2, C80.2, C82.2, C83.2, C88.2, C89.2, C90.2, C91.2, C92.2, C93.2, C94.2, C95.2, C96.2, C98.2, C99.2, D12.3 (common), D6.1 (A1), D9.2 (A), IC2.2 (GND), IC3.8 (VSS), IC5.11 (EP), IC5.5 (VSS), J1.1 (Pin_1), Q1.2 (E), R11.2, R17.2, R18.2, R20.2, R22.2, R28.2, R49.2, R5.2, R80.2, R83.2, R85.2, R86.2, TH1.2, U10.2 (GND), U11.2 (GND), U14.2 (GND), U15.2 (GND), U16.2 (GND), U17.2 (GND), U18.1 (GND), U18.6 (MODE), U21.3 (GND), U22.3 (GND), U22.PAD (GND), U25.2 (VSS), U25.9 (PAD), U6.7 (GND), U6.9 (EXP), U6.V1 (EXP), U6.V2 (EXP), U6.V3 (EXP), U6.V4 (EXP), U6.V5 (EXP), U6.V6 (EXP); no longer C27.2, C28.2, R3.2, R34.2
- net GNSS_EN_3V3: now also IC2.3 (EN), U14.3 (EN)
- net VIN: now also C11.1, C92.1, C93.1, C94.1, L9.2, R27.1, U6.2 (VIN)
- net WDI: now also R52.1, IC3.12 (RESET), R50.2; no longer R34.1
- net WDO: now also R2.1, IC3.3 (Q14), JP2.2 (B), R19.1, R27.2, R28.1, U6.3 (EN); no longer R3.1
- net at C19.1, C20.1, FB1.1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: now also D8.1 (K), R14.1
- net at U3.4 (G): now also D8.2 (A), R11.1, R14.2
- net at U4.4 (RON): now also R20.1
- net at D7.1 (K), L3.1, U4.8 (SW): now also C26.1, R21.1; no longer C23.1
- net at C25.1: now also R16.2, U4.3 (ULVO), Q1.3 (C), R17.1, R18.1; no longer C26.1
- net at F1.2, U3.5 (D), U3.6 (D)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: now also D6.2 (A2)
- net at U4.5 (FB): now also C27.2, R29.2, R49.1; no longer C25.2
- net at U4.7 (BST): now also C26.2; no longer C23.2
- net at L5.1: now also U11.5 (SW)
- net at R46.2: now also U11.3 (EN)
- new net: C81.2, C82.1
- new net: R86.1, U22.2 (PROG)
- new net: C108.1, C110.1, R84.1, R87.2, U22.4 (VCC), U22.8 (CE)
- new net: C24.1, U6.6 (SS)
- new net: C79.2, C80.1
- new net: R5.1, U6.4 (RT/SYNC)
- new net: C27.1, C28.1, R21.2
- new net: C47.2, R15.2, R22.1, U6.5 (FB)
- new net: L14.4, R89.2, U25.6 (CANL)
- new net: C59.2, R3.1, R34.1
- new net: IC3.11 ([Phi]I), R3.2
- new net: R79.2, R80.1, U18.4 (FB)
- new net: IC5.6 (PROG), R83.1
- new net: C77.2, C78.1
- new net: C59.1, IC3.9 ([Phi]O)
- new net: IC3.10 (~{[Phi]O}), R34.2
- new net: D10.1 (K), L8.1
- new net: C83.1, C88.1, C89.1, C90.1, C91.1, L8.2, L9.1
- new net: C114.1, R90.2, R91.1
- new net: C46.2, D9.1 (K), L7.1, U6.8 (SW)
- new net: L14.1, R88.2, U25.7 (CANH)
- new net: C46.1, U6.1 (BOOT)
- new net: JP2.1 (A), U17.1 (~{RESET})
- new net: C23.1, Q1.1 (B), R19.2
- new net: R50.1, U17.4 (WDI)
- new net: L11.2, U18.2 (SW)
- new net 4V7_BOOST: C100.1, C103.1, C104.1, R79.1, U15.3 (~{CE}), U16.1 (VIN), U18.3 (VOUT)
- new net 5V0_BUCK: C106.1, C47.1, C57.1, C76.1, IC5.1 (VDD_1), IC5.2 (VDD_2), L7.2, R15.1, R87.1, U15.1 (VIN), U16.3 (~{CE}), U21.2
- new net BOOST_EN: U18.5 (EN), U21.4
- new net CAN_250_H: D12.2 (A2), L14.2, R88.1, R90.1
- new net CAN_250_L: D12.1 (A1), L14.3, R89.1, R91.2
- new net CAN_SHDN: U25.8 (SHDN)
- new net CHARGER_STAT_1: IC5.3 (STAT1), R81.1
- new net CHARGER_STAT_2: IC5.4 (STAT2), R82.1
- new net NTC: IC5.8 (THERM), J1.3 (Pin_3), R84.2, R85.1, TH1.1, U22.1 (TEMP)
- new net VBAT: C102.1, C107.1, C109.1, C111.1, IC5.10 (VBAT_2), IC5.9 (VBAT_1), J1.2 (Pin_2), L11.1, U18.7 (VIN), U22.5 (BAT)
- new net V_EXT: C77.1, C79.1, C81.1, D10.2 (A)
- no-connect marks 59 -> 64
Other:
- note added: "10k (103A) Normaly inside battery"
- note added: "15uA OPEN-DRAIN ACTIVE-LOW 1RMB SMALL SIZE"
- note added: "2k = 500mA max charge current"
- note added: "4V0 Buck GOOD TO KEEP CHEAP AND POWERFUL"
- note added: "4k = 300mA max charge current Rprog = 1200/Ibat"
- note added: "ACAP to input"
- note added: "Add this enable control from the external DCDC, avoid the booster to affect the charging."
- note added: "BECOME SO EXPENSIVE AGAIN"
- note added: "Battery charger"
- note added: "Battery interface"
- note added: "CAN-MS 500k"
- note added: "CD4060 is a 14 bit counter with internal oscillator Oscillator setup with C and R as below: f = 1 / ( 2.5 x R x C) f = 1 / (2.5 * 220k * 1u) = 1.8Hz 1/1.8Hz = 0.55 sec 0b10000000000000 = 8192 0.55sec * 8192 = ~75min Q13 is turned HIGH after around 75min toggle WDI will reset counter Power cycle will reset counter SHALL WE KEEP IT?"
- note added: "F2 Keep cold res low High cold res will cause isses with the booster"
- note added: "For LM3671MF-3.3 Efficiency 85% when Vin=5v Vout=3.3 @10mA 80% when Vin=5v Vout=3.3 @1mA 60% when Vin=5v Vout=3.3 @0.1mA price =8RMB@JLC shall we remove it? LDO efficiency =~60%"
- note added: "NTC 3380K 10K nominal resistor"
- note added: "ORing source selection circuit"
- note added: "R87 for pre-thermal release for internal LDO of TP4056"
- note added: "Shall we need it? Iq OF BOOST when it has no load = 0.9~3uA Ishundown when it's disable = 0.25~0.6uA the consideration is that whether Iq affect the charging chip or not."
- note added: "ULVO Configuration Ven 1.2V Ien 1uA Ihys = 3.6uA Rent = (Vstart- Vstop)/ Ihys Renb = Ven/((Vstart-Ven)/Rent + Ien)"
- note added: "Vin -> buck Vbat -> boost"
- note added: "Vstart = 10.5v *Vstop = 9V Rent = (10.5V- 9V)/ 3.6uA = ~416.6K, we take 412K Vhys= 412K*3.6uA = 1.48v So Vstop = 10.5v-1.48v = 9.02V Renb = Ven/((Vstart-Ven)/Rent + Ien) = 51k"
- note removed: "4V0 Buck"
- note removed: "CD4060 is a 14 bit counter with internal oscillator Oscillator setup with C and R as below: f = 1 / ( 2.5 x R x C) f = 1 / (2.5 * 220k * 1u) = 1.8Hz 1/1.8Hz = 0.55 sec 0b10000000000000 = 8192 0.55sec * 8192 = ~75min Q13 is turned HIGH after around 75min toggle WDI will reset counter Power cycle will reset counter"
- moved on the sheet: C35, C37, C39, C42, C43, C50, C51, C52, L4, R36, R40, R41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

Commit message: done before delete nrf
Parts:
- removed U25: MCP2562-E/MF, Package_DFN_QFN:DFN-8-1EP_3x3mm_P0.65mm_EP1.55x2.4mm, symbol Interface_CAN_LIN:MCP2562-E-MF
- added C115: 100nF, Capacitor_SMD:C_0402_1005Metric, symbol Device:C_Small
- added C117: 10uF, Capacitor_SMD:C_0603_1608Metric, symbol Device:C_Small
- added J4: Conn_01x03_Pin, Connector_PinHeader_1.27mm:PinHeader_1x02_P1.27mm_Vertical_SMD_Pin1Left, symbol Connector:Conn_01x02_Pin
- added R92: 120, Resistor_SMD:R_0402_1005Metric, symbol Device:R_Small
- added R93: 100k, Resistor_SMD:R_0603_1608Metric, symbol Device:R_Small
- added R94: 330k, Resistor_SMD:R_0603_1608Metric, symbol Device:R_Small
- added TP3: T_BAT, TestPoint:TestPoint_Pad_D1.0mm, symbol Connector:TestPoint
- added U25: ESP32-S3-MINI-1, RF_Module:ESP32-S2-MINI-1, symbol RF_Module:ESP32-S3-MINI-1
- added U26: MCP2562-E/MF, Package_DFN_QFN:DFN-8-1EP_3x3mm_P0.65mm_EP1.55x2.4mm, symbol Interface_CAN_LIN:MCP2562-E-MF
Connections:
- net 3V3_ALWAYS_ON: now also C117.1, U25.3 (3V3), U25.45 (EN), U26.5 (Vio)
- net 5V0: now also U26.3 (VDD)
- net ACC_INT: now also U25.34 (IO38)
- net AUX_LED: now also U25.4 (IO0)
- net CAN_250_H: now also J4.2 (Pin_2)
- net CAN_250_L: now also R92.2
- net CAN_SHDN: now also U25.37 (IO41), U26.8 (SHDN)
- net CONN_LED: now also U25.29 (IO34)
- net CTS_3V3: now also U25.10 (IO6)
- net DCD_3V3: now also U25.9 (IO5)
- net EBL: now also U25.5 (IO1)
- net GND: now also C115.2, C117.2, R94.2, U25.1 (GND), U25.2 (GND), U25.42 (GND), U25.43 (GND), U25.46 (GND), U25.47 (GND), U25.48 (GND), U25.49 (GND), U25.50 (GND), U25.51 (GND), U25.52 (GND), U25.53 (GND), U25.54 (GND), U25.55 (GND), U25.56 (GND), U25.57 (GND), U25.58 (GND), U25.59 (GND), U25.60 (GND), U25.61 (GND), U25.62 (GND), U25.63 (GND), U25.64 (GND), U25.65 (GND), U26.2 (VSS), U26.9 (PAD)
- net GNSS_EN_3V3: now also U25.44 (IO46)
- net GNSS_RST_3V3: now also U25.27 (IO47)
- net GNSS_RXD_3V3: now also U25.38 (IO42)
- net GNSS_TXD_3V3: now also U25.41 (IO45)
- net GPS_ANT_EN: now also U25.17 (IO13)
- net MODEM_DTR_3V3: now also U25.26 (IO26)
- net MODEM_RI_3V3: now also U25.28 (IO33)
- net MODEM_RX_3V3: now also U25.16 (IO12)
- net MODEM_TX_3V3: now also U25.15 (IO11)
- net NRESET: now also U25.25 (IO21)
- net NRF_LED: now also U25.33 (IO37)
- net PWRKEY: now also U25.22 (IO18)
- net RS485_RX: now also U25.14 (IO10)
- net RS485_TX: now also U25.13 (IO9)
- net RTS_3V3: now also U25.11 (IO7)
- net SCL: now also U25.19 (IO15)
- net SDA: now also U25.18 (IO14)
- net STATUS_LED_3V3: now also U25.32 (IO36)
- net U20_EN: now also U25.20 (IO16)
- net UART_RS485_RE_SHDN: now also U25.12 (IO8)
- net VBAT: now also R93.1, TP3.1
- net WDI: now also U25.21 (IO17)
- net at L14.4, R89.2: now also U26.6 (CANL)
- net at L14.1, R88.2: now also U26.7 (CANH)
- new net: J4.1 (Pin_1), R92.1
- new net CAN_RXD: U25.35 (IO39), U26.4 (RXD)
- new net CAN_TXD: U25.36 (IO40), U26.1 (TXD)
- new net IBL: C115.1, R93.2, R94.1, U25.6 (IO2)
- new net JTAG_D+: U25.24 (IO20)
- new net JTAG_D-: U25.23 (IO19)
- no-connect marks 64 -> 68
Other:
- note added: "Internal Battery voltage Level (IBL) 2.6V - 4.3V"
- note added: "USB Built-in JTAG interface"
- note added: "Vout/Vin = 0.767"
- moved on the sheet: C1, C100, C101, C102, C103, C104, C105, C106, C107, C108, C109, C11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

Commit message: done before delete the old stuff
Parts:
- removed D21, D22: LED, LED_SMD:LED_0603_1608Metric, symbol Device:LED
- removed J4: Conn_01x03_Pin, Connector_PinHeader_1.27mm:PinHeader_1x02_P1.27mm_Vertical_SMD_Pin1Left, symbol Connector:Conn_01x02_Pin
- removed Q2 (x3): MMBT3904, Package_TO_SOT_SMD:SOT-23, symbol Transistor_BJT:MMBT3904
- removed R70, R73, R76: 4K7, Resistor_SMD:R_0402_1005Metric, symbol Device:R
- removed R71, R74, R77: 47K, Resistor_SMD:R_0402_1005Metric, symbol Device:R
- removed R72, R75: 750, Resistor_SMD:R_0603_1608Metric, symbol Device:R_Small
- removed R88, R89: 0, Resistor_SMD:R_0402_1005Metric, symbol Device:R
- removed R90, R91: 2k8, Resistor_SMD:R_0402_1005Metric, symbol Device:R_Small
- removed R92: 120, Resistor_SMD:R_0402_1005Metric, symbol Device:R_Small
- added C118: 100nF, Capacitor_SMD:C_0402_1005Metric, symbol Device:C_Small
- added D14, D15: LED, LED_SMD:LED_0603_1608Metric, symbol Device:LED
- added Q12, Q2, Q5: Q_NPN_BEC_BRT, Package_TO_SOT_SMD:SOT-23, symbol Device:Q_NPN_BEC_BRT
- added R70, R71: 750, Resistor_SMD:R_0603_1608Metric, symbol Device:R_Small
- added U29: TXB0108RGY, Package_DFN_QFN:Texas_RGY_R-PVQFN-N20_EP2.05x3.05mm, symbol Logic_LevelTranslator:TXB0108RGY
- added U30: TXB0104RUT, Package_DFN_QFN:Texas_R-PUQFN-N12, symbol Logic_LevelTranslator:TXB0104RUT
- C114: value 1nF -> 100nF; MPN 0402N102F500CT -> CL05B104KP5NNNC
Connections:
- net CAN_250_H is gone; now on net CAN_500_H: D12.2 (A2), L14.2
- net CAN_250_L is gone; now on net CAN_500_L: D12.1 (A1), L14.3
- net +1V8: now also C118.1, U30.11 (VCCB), U30.12 (OE)
- net 3V3_ALWAYS_ON: now also C114.1, U30.1 (VCCA)
- net GND: now also C118.2, Q12.2 (E), Q2.2 (E), Q5.2 (E), U30.6 (GND)
- net GNSS_EN_1V8: now also U30.7 (B4)
- net GNSS_EN_3V3: now also U30.5 (A4)
- net GNSS_RST_1V8: now also U30.8 (B3)
- net GNSS_RST_3V3: now also U30.4 (A3)
- net GNSS_RXD_1V8: now also U30.10 (B1)
- net GNSS_RXD_3V3: now also U30.2 (A1)
- net GNSS_TXD_1V8: now also U30.9 (B2)
- net GNSS_TXD_3V3: now also U30.3 (A2)
- net NET_LED: now also Q2.1 (B)
- net PPS_GNSS: now also Q12.1 (B)
- net PSM_IND: now also Q5.1 (B)
- net at R78.2: now also Q12.3 (C)
- net at D23.2 (A), JP3.2 (B): now also D14.2 (A), D15.2 (A)
- new net: D15.1 (K), R71.1
- new net: Q5.3 (C), R71.2
- new net: Q2.3 (C), R70.2
- new net: D14.1 (K), R70.1
- new net: U29.11 (GND), U29.21 (GND)
Other:
- moved on the sheet: C14, C15, D12, D23, JP1, Q2, R13, R58, R60, R64, R78, U5

Commit message: saved
Parts:
- removed C61: 100nF, Capacitor_SMD:C_0402_1005Metric, symbol Device:C_Small
- removed C69, C70, C72, C73: 1nF, Capacitor_SMD:C_0402_1005Metric, symbol Device:C_Small
- removed Q2 (x4): MMBT3904, Package_TO_SOT_SMD:SOT-23, symbol Transistor_BJT:MMBT3904
- removed Q6, Q7: BC846A,215, Package_TO_SOT_SMD:SOT-23, symbol Transistor_BJT:BC846
- removed R57: 47K, Resistor_SMD:R_0402_1005Metric, symbol Device:R
- removed R58 (x4): 10k, Resistor_SMD:R_0402_1005Metric, symbol Device:R_Small
- removed R60, R62, R66, R68: 4K7, Resistor_SMD:R_0402_1005Metric, symbol Device:R
- removed U5: TXB0108DQSR, Package_SON:USON-20_2x4mm_P0.4mm, symbol Logic_LevelTranslator:TXB0108DQSR
- removed U6: MX25R6435FZNIL0, Package_SON:WSON-8-1EP_6x5mm_P1.27mm_EP3.4x4mm, symbol TC-Flash:MX25R6435FZNIL0
- added C61, C69, C70: 0.1uF, Capacitor_SMD:C_0402_1005Metric, symbol Device:C
- added J4: USB_B_Micro, Connector_USB:USB_Micro-B_Molex-105017-0001, symbol Connector:USB_B_Micro
- added Q6, Q8: Q_NPN_BEC_BRT, Package_TO_SOT_SMD:SOT-23, symbol Device:Q_NPN_BEC_BRT
- added SW1, SW2: SW_Push, Button_Switch_SMD:SW_Push_SPST_NO_Alps_SKRK, symbol Switch:SW_Push
- added TP14, TP15, TP16, TP17, TP4, TP6: TestPoint, TestPoint:TestPoint_Pad_D1.0mm, symbol Connector:TestPoint
- C1, C106, C107, C12, C16, C17, C18, C19, C20, C21, C22, C23, C25, C26, C27, C28, C30, C31, C33, C34, C36, C38, C40, C41, C53, C55, C56, C59, C6, C7, C74, C75, C8, C97, D2, D26, D6, D7, D8, F1, FB1, IC1, IC2, IC3, IC5, L1, L2, L3, L5, Q1, R1, R11, R14, R16, R17, R18, R19, R2, R20, R21, R23, R24, R25, R26, R29, R3, R32, R34, R46, R49, R52, R81, R82, R83, R9, U11, U12, U2, U23, U24, U3, U4, Y1: now not fitted
- R54: value 4K7 -> 10k; MPN RK73H1ETTP4701F -> (none)
- R55: value 4K7 -> 0; MPN RK73H1ETTP4701F -> RMCF0402FT20R0; Tolerance (none) -> 1%
- R56: value 47K -> 0; MPN ERJ-2RKF4702X -> RMCF0402FT20R0; Tolerance (none) -> 1%
Connections:
- net +1V8: now also C114.1, U30.1 (VCCA); no longer C118.1, U30.11 (VCCB)
- net 3V3_ALWAYS_ON: now also C118.1, R54.1, U29.19 (V_{CCB}), U30.11 (VCCB); no longer C114.1, U25.45 (EN), U30.1 (VCCA)
- net AUX_LED: now also U25.7 (IO3); no longer U25.4 (IO0)
- net CTS_1V8: now also U29.5 (A4)
- net CTS_3V3: now also U29.16 (B4)
- net DCD_1V8: now also U29.6 (A5)
- net DCD_3V3: now also U29.15 (B5)
- net GND: now also U29.11 (GND), U29.21 (GND), C61.2, C69.2, C70.1, J4.5 (GND), J4.6 (Shield), Q6.2 (E), Q8.2 (E), SW1.1, SW2.1; no longer R56.1
- net GNSS_EN_1V8: now also U30.2 (A1); no longer U30.7 (B4)
- net GNSS_EN_3V3: now also U30.10 (B1); no longer U30.5 (A4)
- net GNSS_RST_1V8: now also U30.3 (A2); no longer U30.8 (B3)
- net GNSS_RST_3V3: now also U30.9 (B2); no longer U30.4 (A3)
- net GNSS_RXD_1V8: now also U30.5 (A4); no longer U30.10 (B1)
- net GNSS_RXD_3V3: now also U30.7 (B4); no longer U30.2 (A1)
- net GNSS_TXD_1V8: now also U30.4 (A3); no longer U30.9 (B2)
- net GNSS_TXD_3V3: now also U30.8 (B3); no longer U30.3 (A2)
- net JTAG_D+: now also J5.4 (Pin_4), R55.2, TP14.1
- net JTAG_D-: now also J5.3 (Pin_3), R56.2, TP15.1
- net MODEM_DTR_1V8: now also U29.8 (A7)
- net MODEM_DTR_3V3: now also U29.13 (B7)
- net MODEM_RI_1V8: now also U29.7 (A6)
- net MODEM_RI_3V3: now also U29.14 (B6)
- net MODEM_RX_1V8: now also U29.3 (A2)
- net MODEM_RX_3V3: now also U29.18 (B2)
- net MODEM_TX_1V8: now also U29.1 (A1)
- net MODEM_TX_3V3: now also U29.20 (B1)
- net NRESET: now also Q8.1 (B); no longer R55.2
- net PWRKEY: now also Q6.1 (B); no longer R54.2
- net RTS_1V8: now also U29.4 (A3)
- net RTS_3V3: now also U29.17 (B3)
- net STATUS_LED: now also U29.9 (A8)
- net STATUS_LED_3V3: now also U29.12 (B8)
- net SWDCLK: no longer J5.3 (Pin_3)
- net SWDIO: no longer J5.4 (Pin_4)
- net VDD_EXT: now also U29.10 (OE), U29.2 (V_{CCA})
- net at C65.2, U1.17 (~{RESET}): now also Q8.3 (C)
- net at R55.1: now also J4.3 (D+)
- net TXD0: now reaches U25.39 (TXD0)
- net TXD0: now also TP16.1
- net RXD0: now reaches U25.40 (RXD0)
- net RXD0: now also TP17.1
- net at C67.2, U1.15 (PWRKEY): now also Q6.3 (C)
- new net: J4.2 (D-), R56.1
- new net EN: C61.1, C69.1, R54.2, SW1.2, TP4.1, U25.45 (EN)
- new net IO0: C70.2, SW2.2, TP6.1, U25.4 (IO0)
- no-connect marks 68 -> 69
Other:
- note removed: "Ext flash"
- note removed: "GNSS ENABLE / RESET LVL SHIFTER 3V3 <-> 1V8"
- note removed: "GNSS UART LVL SHIFTER 3V3 <-> 1V8"
- note removed: "MAX BAUDRATE: 460 kbps."
- moved on the sheet: C114, C117, C118, C14, C58, C68, J6, R31, R32, R51, R58, R59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
