File: orange_compact.kicad_sch (KiCad schematic)
At the start: 266 parts, among them IC4 MAX13487EESA+T, J1 Battery, J4 Conn_Coaxial, J4 USB_B_Micro, J5 USB_B_Micro, J6 EG800, J7 Conn_01x11_Pin, Q1 Q_NPN_BEC_BRT, Q2 Q_NPN_BEC_BRT, Q3 Q_NPN_BEC_BRT, Q4 Q_NPN_BEC_BRT, Q5 Q_NPN_BEC_BRT, Q6 Q_NPN_BEC_BRT, SW1 SW_Push, SW2 SW_Push, U1 1NCE IoT SIMs Chip, U10 LP5907MFX-3.3, U11 TXB0108RGY, U12 LP5907MFX-1.8, U13 LIS2DH12TR, U14 TPS566242DRLR, U15 LM66100DCKR, U16 LM66100DCKR, U17 MIC29302WU, U18 TPS61022, U19 LTV-217, U2 TXB0102DCU, U20 LC79H, U21 LP5907MFX-3.3, U22 TP4056, U25 ESP32-S3-MINI-1, U26 MCP2562-E/MF, U27 LP5907MFX-3.3, U28 USBLC6-2SC6, U3 TXB0104RUT, U4 LP5907MFX-3.3, U5 LTV-217, U6 LMR14030SDDAR, U8 EG916QGLLG-N03-SGNSA, U9 USBLC6-2SC6

Commit message: saved
Parts:
- removed C53: 2.2uF, Capacitor_SMD:C_0603_1608Metric, symbol Device:C_Small
- removed C55: 1uF, Capacitor_SMD:C_0603_1608Metric, symbol Device:C
- removed R30: 0, Resistor_SMD:R_0402_1005Metric, symbol Device:R_Small
- removed TP14, TP15: TestPoint, TestPoint:TestPoint_Pad_D1.0mm, symbol Connector:TestPoint
- added C64, C65: 1uF, Capacitor_SMD:C_0402_1005Metric, symbol Device:C
- C50: value 220uF -> 470uF
Connections:
- net 5V0: now also C64.1
- net GND: now also C64.2, C65.2
- net VCC_LC760Z: now also C65.1
- no-connect marks 53 -> 54
Other:
- moved on the sheet: C116, C2, D13, J4, L10, L13, L6, R100, R4

Commit message: saved
Parts:
- removed C6: 2.2uF, Capacitor_SMD:C_0402_1005Metric, symbol Device:C_Small
- removed C7: 1uF, Capacitor_SMD:C_0402_1005Metric, symbol Device:C
- removed U4: LP5907MFX-3.3, Package_TO_SOT_SMD:SOT-23-5, symbol Regulator_Linear:LP5907MFX-3.3
- C119, C120, U27: now not fitted
- C19, C20, C25, C26, C27, C33, C34, C35, C36, C37, C38, C39, C40, C41, C42, CP1, D15, D20, D6, D8, L1, Q4, Q5, R11, R17, R19, R20, TP11, TP12, TP13, TP19, TP20, TP21, TP9, U12, U14, U3, U8: now not fitted; now left out of the parts list
Connections:
- net 3V3_ALWAYS_ON: now also C112.2, C14.1, JP3.1 (A), U11.19 (V_{CCB}), U26.5 (Vio)
- net 3V3_CONM: no longer C112.2, C14.1, JP3.1 (A), U11.19 (V_{CCB}), U26.5 (Vio)

Commit message: almost done
Parts:
- removed TP24: TestPoint, TestPoint:TestPoint_Pad_D1.0mm, symbol Connector:TestPoint
Changed lines of the file:
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@@
 	(wire
 		(pts
-			(xy 494.03 111.76) (xy 510.54 111.76)
-		)
-		(stroke
-			(width 0)
-			(type default)
-		)
-	)
-	(wire
-		(pts
 			(xy 336.55 223.52) (xy 336.55 228.6)
 		)
@@
 		)
 		(instances
-			(project ""
+			(project "orange_compact"
 				(path "/e63e39d7-6ac0-4ffd-8aa3-1841a4541b55"
 					(reference "U22")
@@
 		)
 		(instances
-			(project ""
+			(project "orange_compact"
 				(path "/e63e39d7-6ac0-4ffd-8aa3-1841a4541b55"
 					(reference "JP2")
@@
 		)
 		(instances
-			(project ""
+			(project "orange_compact"
 				(path "/e63e39d7-6ac0-4ffd-8aa3-1841a4541b55"
 					(reference "C43")
@@
 		)
 		(instances
-			(project ""
+			(project "orange_compact"
 				(path "/e63e39d7-6ac0-4ffd-8aa3-1841a4541b55"
 					(reference "U25")
@@
 		)
 		(instances
-			(project ""
+			(project "orange_compact"
 				(path "/e63e39d7-6ac0-4ffd-8aa3-1841a4541b55"
 					(reference "U6")
@@
 		)
 		(instances
-			(project ""
+			(project "orange_compact"
 				(path "/e63e39d7-6ac0-4ffd-8aa3-1841a4541b55"
 					(reference "U20")
@@
 	)
 	(symbol
-		(lib_id "Connector:TestPoint")
-		(at 510.54 111.76 270)
-		(unit 1)
-		(exclude_from_sim no)
-		(in_bom yes)
-		(on_board yes)
-		(dnp no)
-		(fields_autoplaced yes)
-		(property "Reference" "TP24"
-			(at 515.62 111.125 90)
-			(effects
-				(font
-					(size 1.27 1.27)
-				)
-				(justify left)
-			)
-		)
-		(property "Value" "TestPoint"
-			(at 515.62 113.665 90)
-			(effects
-				(font
-					(size 1.27 1.27)
-				)
-				(justify left)
-			)
-		)
-		(property "Footprint" "TestPoint:TestPoint_Pad_D1.0mm"
-			(at 510.54 116.84 0)
-			(effects
-				(font
-					(size 1.27 1.27)
-				)
-				(hide yes)
-			)
-		)
-		(property "Datasheet" "~"
-			(at 510.54 116.84 0)
-			(effects
-				(font
-					(size 1.27 1.27)
-				)
-				(hide yes)
-			)
-		)
-		(property "Description" ""
-			(at 510.54 111.76 0)
-			(effects
-				(font
-					(size 1.27 1.27)
-				)
-				(hide yes)
-			)
-		)
-		(property "Field5" ""
-			(at 510.54 111.76 0)
-			(effects
-				(font
-					(size 1.27 1.27)
-				)
-				(hide yes)
-			)
-		)
-		(pin "1"
-		)
-		(instances
-			(project "orange_compact"
-				(path "/e63e39d7-6ac0-4ffd-8aa3-1841a4541b55"
-					(reference "TP24")
-					(unit 1)
-				)
-			)
-		)
-	)
-	(symbol
 		(lib_id "Device:C_Small")
 		(at 1397 125.73 0)
@@
 		)
 		(instances
-			(project ""
+			(project "orange_compact"
 				(path "/e63e39d7-6ac0-4ffd-8aa3-1841a4541b55"
 					(reference "U2")
@@
 		)
 		(instances
-			(project ""
+			(project "orange_compact"
 				(path "/e63e39d7-6ac0-4ffd-8aa3-1841a4541b55"
 					(reference "C90")
@@
 		)
 		(instances
-			(project ""
+			(project "orange_compact"
 				(path "/e63e39d7-6ac0-4ffd-8aa3-1841a4541b55"
 					(reference "H4")
@@
 		)
 		(instances
-			(project ""
+			(project "orange_compact"
 				(path "/e63e39d7-6ac0-4ffd-8aa3-1841a4541b55"
 					(reference "U17")
@@
 		)
 		(instances
-			(project ""
+			(project "orange_compact"
 				(path "/e63e39d7-6ac0-4ffd-8aa3-1841a4541b55"
 					(reference "U18")
@@
 		)
 		(instances
-			(project ""
+			(project "orange_compact"
 				(path "/e63e39d7-6ac0-4ffd-8aa3-1841a4541b55"
 					(reference "J7")
@@
 		)
 		(instances
-			(project ""
+			(project "orange_compact"
 				(path "/e63e39d7-6ac0-4ffd-8aa3-1841a4541b55"
 					(reference "L11")
@@
 		)
 		(instances
-			(project ""
+			(project "orange_compact"
 				(path "/e63e39d7-6ac0-4ffd-8aa3-1841a4541b55"
 					(reference "J6")
@@
 	)
 	(symbol
-		(lib_id "power:+1V8")
-		(at 494.03 111.76 0)
-		(unit 1)
-		(exclude_from_sim no)
-		(in_bom yes)
-		(on_board yes)
-		(dnp no)
-		(fields_autoplaced yes)
-		(property "Reference" "#PWR06"
-			(at 494.03 115.57 0)
-			(effects
-				(font
-					(size 1.27 1.27)
-				)
-				(hide yes)
-			)
-		)
-		(property "Value" "+1V8"
-			(at 494.03 107.95 0)
-			(effects
-				(font
-					(size 1.27 1.27)
-				)
-			)
-		)
-		(property "Footprint" ""
-			(at 494.03 111.76 0)
-			(effects
-				(font
-					(size 1.27 1.27)
-				)
-				(hide yes)
-			)
-		)
-		(property "Datasheet" ""
-			(at 494.03 111.76 0)
-			(effects
-				(font
-					(size 1.27 1.27)
-				)
-				(hide yes)
-			)
-		)
-		(property "Description" ""
-			(at 494.03 111.76 0)
-			(effects
-				(font
-					(size 1.27 1.27)
-				)
-				(hide yes)
-			)
-		)
-		(pin "1"
-		)
-		(instances
-			(project "orange_compact"
-				(path "/e63e39d7-6ac0-4ffd-8aa3-1841a4541b55"
-					(reference "#PWR06")
-					(unit 1)
-				)
-			)
-		)
-	)
-	(symbol
 		(lib_id "power:GND")
 		(at 193.04 304.8 0)
@@
 		)
 		(instances
-			(project ""
+			(project "orange_compact"
 				(path "/e63e39d7-6ac0-4ffd-8aa3-1841a4541b55"
 					(reference "J6")

Commit message: saved
Parts:
- removed C19, C20, C25, C36, C42: 100nF, Capacitor_SMD:C_0402_1005Metric, symbol Device:C_Small
- removed C26, C37: 33pF, Inductor_SMD:L_0402_1005Metric, symbol Device:C_Small
- removed C27: 10pF, Capacitor_SMD:C_0402_1005Metric, symbol Device:C_Small
- removed C33, C34: 1uF, Capacitor_SMD:C_0402_1005Metric, symbol Device:C_Small
- removed C35: 47uF, Inductor_SMD:L_1206_3216Metric, symbol Device:C_Small
- removed C38, C39, C40, C41: 22uF, Capacitor_SMD:C_0805_2012Metric, symbol Device:C_Small
- removed CP1: 100u, Capacitor_Tantalum_SMD:CP_EIA-6032-28_Kemet-C, symbol Device:C_Polarized
- removed D15, D20: LED, LED_SMD:LED_0603_1608Metric, symbol Device:LED
- removed D6, D8: D4V5H1BS2LP-7B, Diode_SMD:D_0402_1005Metric, symbol Device:D_Zener
- removed L1: 2.2uH, Inductor_SMD:L_Bourns-SRN4018, symbol Device:L
- removed Q4, Q5: Q_NPN_BEC_BRT, Package_TO_SOT_SMD:SOT-23, symbol Device:Q_NPN_BEC_BRT
- removed R11, R17: 750, Resistor_SMD:R_0603_1608Metric, symbol Device:R_Small
- removed R18: 10k, Resistor_SMD:R_0402_1005Metric, symbol Device:R
- removed R19: 169k, Resistor_SMD:R_0402_1005Metric, symbol Device:R
- removed R20: 30k, Resistor_SMD:R_0402_1005Metric, symbol Device:R
- removed TP11: gnss_en, TestPoint:TestPoint_Pad_D1.0mm, symbol Connector:TestPoint
- removed TP12, TP20, TP21, TP9: TestPoint, TestPoint:TestPoint_Pad_D1.0mm, symbol Connector:TestPoint
- removed TP13: gnss_tx, TestPoint:TestPoint_Pad_D1.0mm, symbol Connector:TestPoint
- removed TP19: gnss_rx, TestPoint:TestPoint_Pad_D1.0mm, symbol Connector:TestPoint
- removed U12: LP5907MFX-1.8, Package_TO_SOT_SMD:SOT-23-5, symbol Regulator_Linear:LP5907MFX-1.8
- removed U14: TPS566242DRLR, TC-Power:TPS566242DRLR, symbol TC-Power:TPS566242DRLR
- removed U3: TXB0104RUT, Package_DFN_QFN:Texas_R-PUQFN-N12, symbol Logic_LevelTranslator:TXB0104RUT
- removed U8: EG916QGLLG-N03-SGNSA, TC-RF-module:XCVR_EG9xQ, symbol RF_Module:EG91xQ
- C1, C102, C103, C104, C108, C109, C110, C111, C13, C14, C5, C9, D16, IC4, L10, L11, L13, R2, R25, R3, R32, R34, R35, R36, R37, R38, R39, R79, R80, R84, R85, R86, R87, TP25, TP26, U15, U16, U18, U2: DNP (none) -> 1; now in the parts list
- C10, C11, C112, C113, C116, C117, C12, C14, C15, C16, C17, C18, C21, C22, C23, C24, C28, C29, C3, C30, C4, C43, C44, C45, C46, C47, C50, C51, C52, C56, C57, C58, C59, C60, C61, C62, C63, C64, C65, C76, C77, C78, C79, C8, C80, C81, C82, C83, C88, C89, C90, C91, C92, C93, C94, C95, C96, CP2, D1, D10, D11, D12, D13, D14, D18, D19, D2, D3, D4, D5, D7, D9, J4, J5, L6, L7, L8, L9, Q1, Q2, Q3, Q6, R1, R10, R100, R12, R13, R14, R15, R16, R21, R22, R23, R24, R27, R28, R29, R31, R32, R34, R36, R37, R38, R5, R54, R6, R65, R7, R8, R9, SW1, SW2, U1, U10, U11, U13, U17, U20, U25, U26, U28, U6, U9: DNP (none) -> 0
- C100, C115, C72, C73, D17, H1, H2, H3, H4, J1, JP1, JP3, JP4, L15, R57, R60, R61, R93, R94, TP1, TP10, TP16, TP17, TP18, TP2, TP22, TP23, TP27, TP28, TP3, TP4, TP5, TP6, TP7, TP8, U19, U5: DNP (none) -> 1; now not fitted
- C119, C120, U27: DNP (none) -> 1
- C2: DNP (none) -> 0; MPN NC -> O402CG101J500NT
- C31: DNP (none) -> 0; MPN (none) -> CC0402BRNPO9BN3R9
- C32: DNP (none) -> 0; MPN (none) -> CC0402BRNPO9BN1R8
- D21, D22: DNP (none) -> 0; MPN (none) -> ESD56151W04
- FID1, FID2: DNP (none) -> 1; now not fitted; now in the parts list
- J6: value EG800 -> EG800K; DNP (none) -> 0; MPN (none) -> EG800K-EU
- J7: DNP (none) -> 0; MPN (none) -> C5368784(2.54mm-11P ZZ)
- JP2: value Jumper_2_Bridged -> 0; DNP (none) -> 0; MPN (none) -> FRC0805P000 TS
- R26: DNP (none) -> 0; MPN (none) -> FRC0603F0000TS
- R4: DNP (none) -> 0; MPN (none) -> 0402WGF100JTCE
- U21: DNP (none) -> 0; MPN (none) -> LP5907MFX-3.3/NOPB
- U22: DNP (none) -> 1; MPN TP4056 -> TP4056-42-ESOP8; now in the parts list
Connections:
- net 3V3_CONM is gone; now on net 3V3_ALWAYS_ON: C1.1, U2.3 (VCCA), U2.6 (OE)
- net 3V3_COMU_EN: no longer names the net of U25.12 (IO8)
- no-connect marks 54 -> 33
Other:
- note removed: "0.3A"
- note removed: "1.2A"
- note removed: "1.8V LDO (GNSS)"
- note removed: "4V0 Buck GOOD TO KEEP CHEAP AND POWERFUL"
- note removed: "GN916 module can be operated in stand-alone or all-in-one mode Stand-alone enables the GNSS part to be operated independently without turning on the CELL functionality. However this require more circuit around the module and if not nessesary it could be removed. Check datasheet for more info"
- note removed: "MODEM / GNSS MODULE"
- note removed: "Power supply buffer for modem"
- note removed: "Stand alone or all in one solution?"
- note removed: "Unlcear if needed"
- note removed: "VBAT_BB -> BaseBand 0.3A VBAT_RF -> RF POWER 1.3A Total 1.6A"
- moved on the sheet: C3, C4, C56, C59, C60, C62, C63, C64, C65, D21, D22, Q6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

Commit message: update bom info
Parts:
- C1, C100, C102, C103, C104, C108, C109, C110, C111, C115, C119, C120, C13, C14, C5, C72, C73, C9, D17, FID1, FID2, H1, H2, H3, H4, IC4, J1, JP1, JP3, JP4, L10, L11, L13, L15, R2, R25, R3, R32, R34, R35, R36, R37, R38, R39, R57, R60, R61, R79, R80, R84, R85, R86, R87, R93, R94, TP1, TP10, TP16, TP17, TP18, TP2, TP22, TP23, TP25, TP26, TP27, TP28, TP3, TP4, TP5, TP6, TP7, TP8, U15, U16, U18, U19, U2, U22, U27, U5: DNP 1 -> (none)
- C10, C11, C112, C113, C116, C117, C12, C14, C15, C16, C17, C18, C2, C21, C22, C23, C24, C28, C29, C3, C30, C31, C32, C4, C43, C44, C45, C46, C47, C50, C51, C52, C56, C57, C58, C59, C60, C61, C62, C63, C64, C65, C76, C77, C78, C79, C8, C80, C81, C82, C83, C88, C89, C90, C91, C92, C93, C94, C95, C96, CP2, D1, D10, D11, D12, D13, D14, D18, D19, D2, D21, D22, D3, D4, D5, D7, D9, J4, J5, J7, JP2, L6, L7, L8, L9, Q1, Q2, Q3, Q6, R1, R10, R100, R12, R13, R14, R15, R16, R21, R22, R23, R24, R26, R27, R28, R29, R31, R32, R34, R36, R37, R38, R4, R5, R54, R6, R65, R7, R8, R9, SW1, SW2, U1, U10, U11, U13, U17, U20, U21, U25, U26, U28, U6: DNP 0 -> (none)
- D16: DNP 1 -> (none); Price (none) -> 1
- J6: DNP 0 -> (none); Price None -> (none)
- U9: DNP 0 -> (none); now not fitted

Commit message: RIGHT BEFORE SMT
Parts:
- removed J4 (x2): Conn_Coaxial, TC-Connector:coax-u.fl, symbol Connector:Conn_Coaxial
- added J3, J8: IPEX, TC-Connector:IPEX1, symbol 0734120110:0734120110
- C1, C100, C102, C103, C104, C108, C109, C110, C111, C115, C119, C120, C13, C14, C5, C72, C73, D16, D17, IC4, J1, L11, L15, R2, R3, R32, R34, R35, R36, R37, R38, R39, R57, R60, R61, R79, R80, R84, R85, R86, R87, R93, R94, TP25, TP26, U15, U16, U18, U19, U2, U22, U27, U5, U9: now fitted
- JP2: symbol Jumper:Jumper_2_Bridged -> Device:R; now not fitted
- R25: MPN RMCF0402FT10K0 -> (none); now fitted
- U1: value 1NCE IoT SIMs Chip -> IoT SIMs Chip
Connections:
- net GND: now also J3.2, J3.3, J3.4, J8.2, J8.3, J8.4
- net RF_ANT_OUT: now also J8.1
- net at C116.2, D13.2 (A2), L6.2: now also J3.1
Other:
- moved on the sheet: JP2

Commit message: updated bom info based on JLC
Parts:
- C1, C100, C102, C103, C104, C108, C109, C110, C111, C115, C119, C120, C13, C14, C23, C5, C72, C73, D16, D17, IC4, J1, J4, J5, L11, L15, R14, R16, R2, R3, R32, R34, R35, R36, R37, R38, R39, R57, R60, R61, R79, R80, R84, R85, R86, R87, R93, R94, TP25, TP26, U15, U16, U18, U19, U2, U22, U27, U28, U5, U9: now not fitted
- C10, C12, C18, C29, C62, C63: JLCPCB Part # (none) -> C441758; MPN GRM1555C1E330JA01D // -> GRM1555C1E330JA01D
- C11: JLCPCB Part # (none) -> C381466; MPN GRM32ER71H475KA88L -> FS32X475K101EGG
- C112, C113, C14, C15, C22, C28, C4, C44, C56, C58, C60, C8: JLCPCB Part # (none) -> C1525; MPN CL05B104KP5NNNC -> CL05B104KO5NNNC
- C116: JLCPCB Part # (none) -> C161543; MPN 0402B333K160CT -> GRM1555C1H240JA01D
- C117, C3, C45, C59: JLCPCB Part # (none) -> C96446; MPN CL10A106MP8NNNC -> CL10A106MA8NRNC
- C14: JLCPCB Part # (none) -> C52923; MPN CC0402KRX5R6BB105 -> CL05A105KA5NQNC
- C16, C17: JLCPCB Part # (none) -> C15195; MPN C0402C103K8RACTU -> CL05B103KB5NNNC
- C2: JLCPCB Part # (none) -> C1546; MPN O402CG101J500NT -> 0402CG101J500NT
- C21: JLCPCB Part # (none) -> C170151; MPN CL05A225MQ5NNNC -> CL05A225KO5NQNC
- C24: JLCPCB Part # (none) -> C307436; MPN GRM155R71C103KA01D** -> CL05B822KB5NNNC
- C30: JLCPCB Part # (none) -> C32949; MPN CGA2B2C0G1H100D050BA -> CL05C100JB5NNNC
- C31: JLCPCB Part # (none) -> C1566; MPN CC0402BRNPO9BN3R9 -> 0402CG3R9C500NT
- C32: JLCPCB Part # (none) -> C1553; MPN CC0402BRNPO9BN1R8 -> 0402CG1R8C500NT
- C43, C50: JLCPCB Part # (none) -> C335982; MPN GVT1A477M0608CNVC -> RVT1A471M0607
- C46: JLCPCB Part # (none) -> C1525; MPN C1005X5R1H104K050BB -> CL05B104KO5NNNC
- C47: JLCPCB Part # (none) -> C237468; MPN GRM033R71C221KA01D** -> GRM033R71C221KA01D
- C51, C52, C83, C88, C89, C94: JLCPCB Part # (none) -> C77055; MPN CL10B104KB8NNNC -> GRM188R71H104KA93D
- C57, C76: JLCPCB Part # (none) -> C77101
- C61: JLCPCB Part # (none) -> C1525; MPN GRM188R71H104KA93D -> CL05B104KO5NNNC
- C64, C65, C95, C96: JLCPCB Part # (none) -> C52923; MPN (none) -> CL05A105KA5NQNC
- C77, C78: JLCPCB Part # (none) -> C14858; MPN CC0603JRNPO0BN101 -> CL10C101JB8NNNC
- C79, C80: JLCPCB Part # (none) -> C1588; MPN GCM155R72A102KA37D -> CL10B102KB8NNNC
- C81, C82: JLCPCB Part # (none) -> C57112; MPN CC0603KRX7R0BB103 -> 0603B103K500NT
- C90, C91: JLCPCB Part # (none) -> C127327; MPN 189RV0019 -> VES221M1CTR-0607
- C92, C93: JLCPCB Part # (none) -> C141033; MPN GRM21BR61H106KE43L -> C0805C106K8PAC7800
- CP2: JLCPCB Part # (none) -> C696808
- D1, D13: JLCPCB Part # (none) -> C434715; MPN AXGD10402 -> AXGD10402KR
- D10: JLCPCB Part # (none) -> C3020232
- D11: JLCPCB Part # (none) -> C316020
- D12, D18: JLCPCB Part # (none) -> C1973833
- D14, D3, D4: JLCPCB Part # (none) -> C2286; MPN QBLP601D-IB -> ESDCAN03-2BWY
- D19, D2, D7: JLCPCB Part # (none) -> C5244624
- D21, D22: JLCPCB Part # (none) -> C2841421; MPN ESD56151W04 -> TPESD56151W04
- D5: JLCPCB Part # (none) -> C965804; MPN QBLP601D-IG -> XL-1608UGC-04
- D9: JLCPCB Part # (none) -> C96113
- J3, J8: JLCPCB Part # (none) -> C2894919; MPN GT-RF1125A-01G -> HC-RF-IPEX0303-01
- J6: JLCPCB Part # (none) -> C22391110; MPN EG800K-EU -> ESDCAN03-2BWY
- J7: JLCPCB Part # (none) -> C5368784; MPN C5368784(2.54mm-11P ZZ) -> 2.54mm-11P ZZ
- JP2: JLCPCB Part # (none) -> #N/A; MPN FRC0805P000 TS -> #N/A; now fitted
- L6: JLCPCB Part # (none) -> C1329469; MPN MLK1005S47NJTD25 -> MLG1005S51NJTD25
- L7: JLCPCB Part # (none) -> C3222940
- L8, L9: JLCPCB Part # (none) -> C167973; MPN FNR5040S330MT -> FNR5040S330MT
- Q1, Q2, Q3, Q6: JLCPCB Part # (none) -> C5439972
- R1: JLCPCB Part # (none) -> C25756; MPN RMCF0402FT15K0 -> 0402WGF1502TCE
- R10, R65, R8, R9: JLCPCB Part # (none) -> C23241; MPN RC0603JR-07750RL -> ESDCAN03-2BWY
- R100, R12, R34, R36: JLCPCB Part # (none) -> C106231; MPN RMCF0402ZT0R00 -> RC0402FR-070RL
- R13: JLCPCB Part # (none) -> C25741; MPN 667-ERJ-2RKF1003X -> 0402WGF1003TCE
- R15: JLCPCB Part # (none) -> C36871; MPN (none) -> 0402WGF6802TCE
- R21: JLCPCB Part # (none) -> C25741; MPN (none) -> 0402WGF1003TCE
- R22: JLCPCB Part # (none) -> C25752; MPN (none) -> FRC0805P000 TS
- R23: JLCPCB Part # (none) -> C25792; MPN (none) -> 0402WGF4702TCE
- R24: JLCPCB Part # (none) -> C23138; MPN (none) -> ESDCAN03-2BWY
- R25, R54: JLCPCB Part # (none) -> C25744; MPN (none) -> 0402WGF1002TCE
- R26: JLCPCB Part # (none) -> C100044; MPN FRC0603F0000TS -> RC0603FR-070RL
- R27: JLCPCB Part # (none) -> C5126037; MPN (none) -> FRC0402F4123TS
- R28: JLCPCB Part # (none) -> C25794; MPN (none) -> 0402WGF5102TCE
- R29, R37, R38, R7: JLCPCB Part # (none) -> C25900; MPN RK73H1ETTP4701F -> 0402WGF4701TCE
- R31: JLCPCB Part # (none) -> C23137; MPN 0603WAF3303T5E -> ESDCAN03-2BWY
- R32: JLCPCB Part # (none) -> C25950; MPN RTT031102FTP -> 0603WAF1102T5E
- R4: JLCPCB Part # (none) -> C413044; MPN 0402WGF100JTCE -> ERJ2RKF10R0X
- R5: JLCPCB Part # (none) -> C25850; MPN CRCW040210K5FKED -> 0402WGF1052TCE
- R6: JLCPCB Part # (none) -> C11702; MPN PFR05S-102-FNH -> 0402WGF1001TCE
- SW1, SW2: JLCPCB Part # (none) -> C720477
- U1: JLCPCB Part # (none) -> #N/A; MPN (none) -> #N/A
- U10: JLCPCB Part # (none) -> C80670; MPN LP5907MFX-3.3 -> LP5907MFX-3.3/NOPB
- U11: JLCPCB Part # (none) -> C194701; MPN (none) -> TXB0108RGYR
- U13: JLCPCB Part # (none) -> C110926
- U17: JLCPCB Part # (none) -> C2995533; MPN (none) -> MIC29302WU(UMW)
- U20: JLCPCB Part # (none) -> C22234543; MPN (none) -> ESDCAN03-2BWY
- U21: JLCPCB Part # (none) -> C80670
- U25: JLCPCB Part # (none) -> C2913206; MPN ESP32-S3-MINI-1 -> ESP32-S3-MINI-1-N8
- U26: JLCPCB Part # (none) -> C635113
- U6: JLCPCB Part # (none) -> C182078

Commit message: updated bom
Parts:
- removed C3, C59: 10uF, Capacitor_SMD:C_0603_1608Metric, symbol Device:C
- removed C4: 100nF, Capacitor_SMD:C_0402_1005Metric, symbol Device:C_Small
- removed C63: 33pF, Inductor_SMD:L_0402_1005Metric, symbol Device:C
- removed D22: ESD56151W04, Diode_SMD:D_SOD-323, symbol Diode:SMAJ30CA
- removed JP4: SolderJumper_2_Open, Jumper:SolderJumper-2_P1.3mm_Open_RoundedPad1.0x1.5mm, symbol Jumper:SolderJumper_2_Open
- removed Q6: Q_NPN_BEC_BRT, Package_TO_SOT_SMD:SOT-23, symbol Device:Q_NPN_BEC_BRT
- removed R29: 4k7, Resistor_SMD:R_0402_1005Metric, symbol Device:R_Small
- removed R34, R36: 0, Resistor_SMD:R_0402_1005Metric, symbol Device:R_Small
- removed U20: LC79H, TC-RF-module:XCVR_LC79H, symbol TC-RF-Module:LC760Z
- C1, C100, C110, C111, C115, C13, C5, C72, C73: JLCPCB Part # (none) -> C1525; MPN CL05B104KP5NNNC -> CL05B104KO5NNNC; now fitted
- C102: JLCPCB Part # (none) -> C15850; MPN C0805C106K8PAC7800** -> CL21A106KAYNNNE; now fitted
- C103, C104: JLCPCB Part # (none) -> C98190; MPN LMK212BJ226MG-T** -> CL21A226MOQNNNE; now fitted
- C108, C109: JLCPCB Part # (none) -> C19702; MPN CL10A106MA8NRNC -> CL10A106KP8NNNC; now fitted
- C119, C120: JLCPCB Part # (none) -> C52923; MPN (none) -> CL05A105KA5NQNC; now fitted
- C13, C9, FID1, FID2: JLCPCB Part # (none) -> #N/A; MPN DNP -> #N/A; now fitted
- C14, C23: JLCPCB Part # (none) -> C52923; MPN CC0402KRX5R6BB105 -> CL05A105KA5NQNC; now fitted
- C46, C61: value 0.1uF -> 100nF
- D14, D3, D4: MPN ESDCAN03-2BWY -> KT-0603R
- D16: JLCPCB Part # (none) -> C316022; now fitted
- D17: JLCPCB Part # (none) -> C5186015; now fitted
- H1, H2, H3, H4, JP1, JP3, L10, L13, R37, TP1, TP10, TP16, TP17, TP18, TP2, TP22, TP23, TP25, TP26, TP27, TP28, TP3, TP4, TP5, TP6, TP7, TP8: JLCPCB Part # (none) -> #N/A; MPN (none) -> #N/A; now fitted
- IC4: JLCPCB Part # (none) -> C18347; now fitted
- J1: JLCPCB Part # (none) -> C2689907; MPN 53048-0310 -> 1.25T-3P-WP; now fitted
- J4, J5: JLCPCB Part # (none) -> C136000; MPN 1050170001 -> ’1050170001; now fitted
- J6: value EG800K -> EG800K-CN; MPN ESDCAN03-2BWY -> #N/A
- L11: JLCPCB Part # (none) -> C138582; MPN SPM5030T-1R0M -> SPM5030T-1R0M; now fitted
- L15: JLCPCB Part # (none) -> C394950; MPN MLZ1608A2R2WT000 -> CMH160808B2R2MT; now fitted
- R10, R65, R8, R9: MPN ESDCAN03-2BWY -> 0603WAF7500T5E
- R14, R16: JLCPCB Part # (none) -> C25089; MPN RMCF0402FT20R0 -> 0402WGF200JTCE; now fitted
- R2, R3, R60: JLCPCB Part # (none) -> C11702; MPN PFR05S-102-FNH -> 0402WGF1001TCE; now fitted
- R24: MPN ESDCAN03-2BWY -> 0603WAF3300T5E
- R31: MPN ESDCAN03-2BWY -> 0603WAF3303T5E
- R32, R34: JLCPCB Part # (none) -> C25744; MPN RMCF0402FT10K0 -> 0402WGF1002TCE; now fitted
- R35, R36: JLCPCB Part # (none) -> C25900; MPN RK73H1ETTP4701F -> 0402WGF4701TCE; now fitted
- R38, R39: JLCPCB Part # (none) -> C25139; MPN RC0402FR-0710RL -> 0402WGJ0100TCE; now fitted
- R57: JLCPCB Part # (none) -> C17798; MPN ERJ-PB6B6800V -> 0805W8F6800T5E; now fitted
- R61: JLCPCB Part # (none) -> C22796; MPN RT0603BRE07130RL -> 0603WAF1300T5E; now fitted
- R7: value 4k7 -> 4K7
- R79: JLCPCB Part # (none) -> C423143; MPN (none) -> 0402WGF6493TCE; now fitted
- R80: value 100K -> 100k; JLCPCB Part # (none) -> C25741; MPN (none) -> 0402WGF1003TCE; now fitted
- R84: JLCPCB Part # (none) -> C51721; MPN (none) -> 0402WGF3901TCE; now fitted
- R85: JLCPCB Part # (none) -> C25794; MPN (none) -> 0402WGF5102TCE; now fitted
- R86: JLCPCB Part # (none) -> C4908; MPN (none) -> 0402WGF1601TCE; now fitted
- R87: JLCPCB Part # (none) -> C44051; MPN (none) -> 0805W8F200LT5E; now fitted
- R93: JLCPCB Part # (none) -> C25803; MPN RMCF0603FT100KCT-ND -> 0603WAF1003T5E; now fitted
- R94: JLCPCB Part # (none) -> C23137; MPN RMCF0603FT330KCT-ND -> 0603WAF3303T5E; now fitted
- U15, U16: JLCPCB Part # (none) -> C2869734; now fitted
- U18: JLCPCB Part # (none) -> C915088; MPN (none) -> TPS61022RWUR; now fitted
- U19, U5: JLCPCB Part # (none) -> C481866; MPN LTV-217-TP1-C-G -> LTV-217-TP1-B-G; now fitted
- U2: JLCPCB Part # (none) -> C60709; MPN TXB0102DCU -> TXB0102DCUR; now fitted
- U22: JLCPCB Part # (none) -> C382139; MPN TP4056-42-ESOP8 -> TP4056; now fitted
- U27: JLCPCB Part # (none) -> C80670; MPN LP5907MFX-3.3 -> LP5907MFX-3.3/NOPB; now fitted
- U28, U9: JLCPCB Part # (none) -> C2827654; now fitted
Connections:
- net VCC_LC760Z is gone; now on net 3V3_ANT: C56.1, C60.2, C62.1, C65.1, D21.2 (A2), U21.5 (OUT)
- net GNSS_ANT: now also J6.2 (GNSS_ANT)
- net GNSS_RESET: no longer names the net of U25.27 (IO47)
- net GNSS_RXD: no longer names the net of U25.38 (IO42)
- net GNSS_TXD: no longer names the net of U25.41 (IO45)
- no-connect marks 33 -> 28
