File: roam_edge_xl.kicad_pcb (KiCad board)
At the start: 6 copper layers, 103 x 60 mm, 236 parts, among them IC4 MAX13487EESA+T, J1 Battery, J11 Conn_01x05_Pin, J2 USB_B_Micro, J3 IPEX, J4 USB_B_Micro, J5 DNP, J6 CA-L01, J7 SIM8060-6-0-14-00-A, J8 MX23A18NF1, J9 Conn_01x11_Pin, Q1 SQS201CENW-T1_GE3, Q4 Q_NPN_BEC_BRT, Q5 Q_NPN_BEC_BRT, Q6 Q_NPN_BEC_BRT, Q7 2N7002E, Q9 AO4407A, SW1 SW_Push, SW2 SW_Push, U1 NUP4202, U10 LP5907MFX-3.3, U11 TXB0108RGY, U12 CN809T, U13 LIS2DH12TR, U14 CN809L, U15 LM66100DCKR, U16 LM66100DCKR, U18 TPS61022, U19 LTV-217, U2 TXB0102DCU, U20 LC760Z, U21 LP5907MFX-3.3, U22 TP4056, U25 ESP32-S3-MINI-1, U26 TJA1051T/3, U27 LP5907MFX-3.3, U28 USBLC6-2SC6, U3 TPS566242DRLR, U4 EG1192L, U5 LTV-217, U6 W25Q128JVP, U7 EG915UEUAC-N05-SNNSA, U8 USBLC6-2SC6, U9 SQS201CENW-T1_GE3

Commit message: added CN809L
Parts:
- removed U12: CN809T, Package_TO_SOT_SMD:SOT-23-3
- removed U9: SQS201CENW-T1_GE3, SQS201CENW-T1_GE3:PDFN3333-8_L3.1-W3.2-P0.65-LS3.4-BL
- R62: value 4.7K -> 4K7
- U14: footprint Package_TO_SOT_SMD:SOT-23 -> Package_TO_SOT_SMD:SOT-23-3
- moved R56 59.4 mm to (51.3, 59.4), turned to 90 degrees
- moved R62 59.3 mm to (51.3, 61.4), turned to 90 degrees
- moved U14 59.1 mm to (54.0, 60.9)
Connections:
- L6 pad 1: Net-(C101-Pad1) -> unconnected-(L6-Pad1)
- R4 pad 1: Net-(C101-Pad1) -> unconnected-(R4-Pad1)
Routing:
- net 5V0: track 78.5 -> 104.0 mm
- net 3V3_ALWAYS_ON: track 119.5 -> 115.0 mm
- net Net-(U14-~{RESET}): track 0.00 -> 1.60 mm

Commit message: add 6pin connector for flasher board and done the whole design
Parts:
- J11: value Conn_01x05_Pin -> Conn_01x06_Pin; footprint Connector_PinHeader_2.54mm:PinHeader_1x05_P2.54mm_Vertical -> Connector_PinHeader_2.54mm:PinHeader_1x06_P2.54mm_Vertical
- U13: footprint LIS2DH12TR:PQFN50P200X200100-12N -> MotionSensor:LIS12DH
- moved G*** 19.0 mm to (63.5, 53.9)
- moved G*** 13.0 mm to (67.6, 58.7)
- moved D9 5.81 mm to (77.9, 102.2)
- moved Q9 5.78 mm to (77.8, 103.1)
- moved R41 5.40 mm to (73.7, 105.5)
- moved G*** 4.42 mm to (40.7, 65.5), turned to -90 degrees
- moved R24 4.26 mm to (73.3, 102.0), turned to -90 degrees
- moved J11 4.14 mm to (95.2, 103.4)
- moved C43 3.63 mm to (37.8, 61.8), turned to -90 degrees
- moved Q7 3.21 mm to (70.5, 101.2)
- moved R27 0.75 mm to (68.7, 103.7)
- moved J1 0.39 mm to (100.1, 95.2)
- moved C109 0.33 mm to (101.3, 99.1)
- moved C111 0.32 mm to (101.8, 97.1)
- moved CR1 0.32 mm to (54.4, 103.3)
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Connections:
- L6 pad 1: unconnected-(L6-Pad1) -> Net-(C101-Pad1)
- R4 pad 1: unconnected-(R4-Pad1) -> Net-(C101-Pad1)
Routing:
- net /IGN: track 59.9 -> 110.9 mm, vias 1 -> 5
- net GND: track 24.6 -> 2.60 mm, vias 259 -> 304
- net /GNSS_BOOT: track 13.3 -> 22.2 mm, vias 1 -> 2
- net /LID_OPEN_DET: track 26.4 -> 33.8 mm
- net V_EXT_P: track 91.1 -> 85.0 mm, vias 6 -> 7
- net /T6_OUT: track 95.1 -> 89.5 mm, vias 4 -> 5
- net /Flasher_Out: track 83.7 -> 78.7 mm
- net 3V3_ANT: track 12.9 -> 17.2 mm, vias 1 -> 2
- net 12V_MCU_OUT: track 78.1 -> 74.1 mm
- net /T6_SIG: track 68.2 -> 65.0 mm
- net Net-(Q7-G): track 5.13 -> 2.63 mm
- net 5V0: track 104.0 -> 105.1 mm
- net VBAT: track 41.2 -> 41.9 mm
- net Net-(Q1-G): track 20.6 -> 19.9 mm
- net Net-(F1-Pad2): track 17.4 -> 16.8 mm
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Other:
- board text added: "5V_BU"
- board text removed: "EBL"
