File: roam_edge_xl.kicad_pcb (KiCad board)
At the start: 6 copper layers, 103 x 60 mm, 234 parts, among them IC4 MAX13487EESA+T, J1 Battery, J11 Conn_01x06_Pin, J2 USB_B_Micro, J3 IPEX, J4 USB_B_Micro, J5 DNP, J6 CA-L01, J7 SIM8060-6-0-14-00-A, J8 MX23A18NF1, J9 Conn_01x11_Pin, Q1 SQS201CENW-T1_GE3, Q4 Q_NPN_BEC_BRT, Q5 Q_NPN_BEC_BRT, Q6 Q_NPN_BEC_BRT, Q7 2N7002E, Q9 AO4407A, SW1 SW_Push, SW2 SW_Push, U1 NUP4202, U10 LP5907MFX-3.3, U11 TXB0108RGY, U13 LIS2DH12TR, U14 CN809L, U15 LM66100DCKR, U16 LM66100DCKR, U18 TPS61022, U19 LTV-217, U2 TXB0102DCU, U20 LC760Z, U21 LP5907MFX-3.3, U22 TP4056, U25 ESP32-S3-MINI-1, U26 TJA1051T/3, U27 LP5907MFX-3.3, U28 USBLC6-2SC6, U3 TPS566242DRLR, U4 EG1192L, U5 LTV-217, U6 W25Q128JVP, U7 EG915UEUAC-N05-SNNSA, U8 USBLC6-2SC6

Commit message: updated silkscreen
Other:
- board text added: "V0.3"
- board text removed: "V0.2"
