File: roam_edge_xl.kicad_sch (KiCad schematic)
At the start: 234 parts, among them IC4 MAX13487EESA+T, J1 Battery, J11 Conn_01x05_Pin, J2 USB_B_Micro, J3 IPEX, J4 USB_B_Micro, J5 DNP, J6 CA-L01, J7 SIM8060-6-0-14-00-A, J8 MX23A18NF1, J9 Conn_01x11_Pin, Q1 SQS201CENW-T1_GE3, Q4 Q_NPN_BEC_BRT, Q5 Q_NPN_BEC_BRT, Q6 Q_NPN_BEC_BRT, Q7 2N7002E, Q9 AO4407A, SW1 SW_Push, SW2 SW_Push, U1 NUP4202, U10 LP5907MFX-3.3, U11 TXB0108RGY, U12 CN809T, U13 LIS2DH12TR, U14 CN809L, U15 LM66100DCKR, U16 LM66100DCKR, U18 TPS61022, U19 LTV-217, U2 TXB0102DCU, U20 LC760Z, U21 LP5907MFX-3.3, U22 TP4056, U25 ESP32-S3-MINI-1, U26 TJA1051T/3, U27 LP5907MFX-3.3, U28 USBLC6-2SC6, U3 TPS566242DRLR, U4 EG1192L, U5 LTV-217, U6 W25Q128JVP, U7 EG915UEUAC-N05-SNNSA, U8 USBLC6-2SC6, U9 SQS201CENW-T1_GE3

Commit message: updated Tamper switch design
Parts:
- Q1: footprint SQS201CENW-T1_GE3:PDFN3333-8_L3.1-W3.2-P0.65-LS3.4-BL -> PMOS_SQS201CENW:PDFN3333-8_L3.1-W3.2-P0.65-LS3.4-BL
- S1: footprint limit switch:SW-SMD_ESE11MV9T -> Tamper_Switch:ESE11MV9
Connections:
- net GND: no longer S1.2 (NO_2)
- net LID_OPEN_DET: now also S1.2 (NO_2)
- net V_EXT_P: now also CR2.1; no longer CR2.2, R5.1
- net at Q1.4 (G): now also CR2.2, R5.1; no longer CR2.1

Commit message: updated gps power input
Parts:
- added C101: 100nF, Capacitor_SMD:C_0402_1005Metric, symbol Device:C_Small
- C116: value 24pf -> 100pf; LCSC Part C161543 -> C1546; MPN GRM1555C1H240JA01D -> 0402CG101J500NT
- L6: value 51nH -> 68nH; LCSC Part C1329469 -> C32836; MPN MLG1005S51NJTD25 -> SDCL1005C68NJTDF
- R4: value 10 -> 0; LCSC Part C481926 -> C17168; MPN CRCW040210R0FKED -> 0402WGF0000TCE
Connections:
- net 3V3_ANT: now also C101.1
- net GND: now also C101.2

Commit message: modified the antenna routing
Connections:
- net 3V3_ANT: no longer C101.1, C2.1
- net at L6.1, R4.1: now also C101.1, C2.1

Commit message: added CN809L
Parts:
- removed U12: CN809T, Package_TO_SOT_SMD:SOT-23-3, symbol Power_Supervisor:LM809
- removed U9: SQS201CENW-T1_GE3, SQS201CENW-T1_GE3:PDFN3333-8_L3.1-W3.2-P0.65-LS3.4-BL, symbol SQS201CENW-T1_GE3:SQS201CENW-T1_GE3
- R62: value 4.7K -> 4K7; LCSC Part (none) -> C25900
- U14: footprint Package_TO_SOT_SMD:SOT-23 -> Package_TO_SOT_SMD:SOT-23-3; LCSC Part (none) -> C840517; MPN (none) -> CN809L
Connections:
- net at C101.1, C2.1: no longer L6.1, R4.1

Commit message: add 6pin connector for flasher board and done the whole design
Parts:
- removed J11: Conn_01x05_Pin, Connector_PinHeader_2.54mm:PinHeader_1x05_P2.54mm_Vertical, symbol Connector:Conn_01x05_Pin
- added J11: Conn_01x06_Pin, Connector_PinHeader_2.54mm:PinHeader_1x06_P2.54mm_Vertical, symbol Connector:Conn_01x06_Pin
- U13: footprint LIS2DH12TR:PQFN50P200X200100-12N -> MotionSensor:LIS12DH
Connections:
- net 12V_MCU_OUT: now also J11.5 (Pin_5)
- net 5V0: now also J11.4 (Pin_4)
- net Flasher_Out: now also J11.3 (Pin_3)
- net GND: now also J11.1 (Pin_1)
- net IGN: now also J11.6 (Pin_6)
- net V_EXT_P: now also J11.2 (Pin_2)
- net at L6.1: now also C101.1, C2.1, R4.1
Changed lines of the file:
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@@
 	)
 	(junction
+		(at 807.72 179.07)
+		(diameter 0)
+		(color 0 0 0 0)
+	)
+	(junction
 		(at 113.03 204.47)
 		(diameter 0)
@@
 	(wire
 		(pts
-			(xy 732.79 551.18) (xy 762 551.18)
+			(xy 736.6 551.18) (xy 762 551.18)
 		)
 		(stroke
@@
 	(wire
 		(pts
-			(xy 817.88 179.07) (xy 822.96 179.07)
+			(xy 817.88 179.07) (xy 833.12 179.07)
 		)
 		(stroke
@@
 	(wire
 		(pts
+			(xy 737.87 541.02) (xy 762 541.02)
+		)
+		(stroke
+			(width 0)
+			(type default)
+		)
+	)
+	(wire
+		(pts
 			(xy 116.84 353.06) (xy 153.67 353.06)
 		)
@@
 	(wire
 		(pts
+			(xy 756.92 546.1) (xy 762 546.1)
+		)
+		(stroke
+			(width 0)
+			(type default)
+		)
+	)
+	(wire
+		(pts
 			(xy 960.12 347.98) (xy 960.12 355.6)
 		)
@@
 	(wire
 		(pts
+			(xy 753.11 543.56) (xy 756.92 543.56)
+		)
+		(stroke
+			(width 0)
+			(type default)
+		)
+	)
+	(wire
+		(pts
 			(xy 127 342.9) (xy 153.67 342.9)
 		)
@@
 	(wire
 		(pts
-			(xy 833.12 179.07) (xy 830.58 179.07)
-		)
-		(stroke
-			(width 0)
-			(type default)
-		)
-	)
-	(wire
-		(pts
 			(xy 1023.62 374.65) (xy 1031.24 374.65)
 		)
@@
 	(wire
 		(pts
-			(xy 762 543.56) (xy 762 546.1)
-		)
-		(stroke
-			(width 0)
-			(type default)
-		)
-	)
-	(wire
-		(pts
 			(xy 980.44 60.325) (xy 980.44 62.23)
 		)
@@
 	(wire
 		(pts
-			(xy 753.11 543.56) (xy 762 543.56)
-		)
-		(stroke
-			(width 0)
-			(type default)
-		)
-	)
-	(wire
-		(pts
 			(xy 487.68 398.78) (xy 487.68 402.59)
 		)
@@
 	(wire
 		(pts
+			(xy 756.92 543.56) (xy 756.92 546.1)
+		)
+		(stroke
+			(width 0)
+			(type default)
+		)
+	)
+	(wire
+		(pts
 			(xy 57.15 487.68) (xy 64.77 487.68)
 		)
@@
 	(wire
 		(pts
+			(xy 762 541.02) (xy 762 543.56)
+		)
+		(stroke
+			(width 0)
+			(type default)
+		)
+	)
+	(wire
+		(pts
 			(xy 377.19 316.23) (xy 379.73 316.23)
 		)
@@
 	(wire
 		(pts
+			(xy 805.18 179.07) (xy 807.72 179.07)
+		)
+		(stroke
+			(width 0)
+			(type default)
+		)
+	)
+	(wire
+		(pts
 			(xy 737.235 316.23) (xy 751.205 316.23)
 		)
@@
 		)
 	)
+	(label "IGN"
+		(at 737.87 541.02 0)
+		(effects
+			(font
+				(size 1.27 1.27)
+			)
+			(justify left bottom)
+		)
+	)
 	(label "GNSS_TXD"
 		(at 208.28 358.14 180)
@@
 	)
 	(label "Flasher_Out"
-		(at 740.41 551.18 0)
+		(at 736.6 551.18 0)
 		(effects
 			(font
@@
 	)
 	(symbol
+		(lib_id "Connector:Conn_01x06_Pin")
+		(at 767.08 551.18 180)
+		(unit 1)
+		(body_style 1)
+		(exclude_from_sim no)
+		(in_bom yes)
+		(on_board yes)
+		(in_pos_files yes)
+		(dnp no)
+		(fields_autoplaced yes)
+		(property "Reference" "J11"
+			(at 768.35 548.6399 0)
+			(show_name no)
+			(do_not_autoplace no)
+			(effects
+				(font
+					(size 1.27 1.27)
+				)
+				(justify right)
+			)
+		)
+		(property "Value" "Conn_01x06_Pin"
+			(at 768.35 551.1799 0)
+			(show_name no)
+			(do_not_autoplace no)
+			(effects
+				(font
+					(size 1.27 1.27)
+				)
+				(justify right)
+			)
+		)
+		(property "Footprint" "Connector_PinHeader_2.54mm:PinHeader_1x06_P2.54mm_Vertical"
+			(at 767.08 551.18 0)
+			(hide yes)
+			(show_name no)
+			(do_not_autoplace no)
+			(effects
+				(font
+					(size 1.27 1.27)
+				)
+			)
+		)
+		(property "Datasheet" ""
+			(at 767.08 551.18 0)
+			(hide yes)
+			(show_name no)
+			(do_not_autoplace no)
+			(effects
+				(font
+					(size 1.27 1.27)
+				)
+			)
+		)
+		(property "Description" "Generic connector, single row, 01x06, script generated"
+			(at 767.08 551.18 0)
+			(hide yes)
+			(show_name no)
+			(do_not_autoplace no)
+			(effects
+				(font
+					(size 1.27 1.27)
+				)
+			)
+		)
+		(pin "3"
+		)
+		(pin "2"
+		)
+		(pin "4"
+		)
+		(pin "1"
+		)
+		(pin "5"
+		)
+		(pin "6"
+		)
+		(instances
+			(project "roam_edge_xl"
+				(path "/e63e39d7-6ac0-4ffd-8aa3-1841a4541b55"
+					(reference "J11")
+					(unit 1)
+				)
+			)
+		)
+	)
+	(symbol
 		(lib_id "Connector:TestPoint")
 		(at 510.54 119.38 270)
@@
 	)
 	(symbol
-		(lib_id "Connector:Conn_01x05_Pin")
-		(at 767.08 551.18 180)
-		(unit 1)
-		(body_style 1)
-		(exclude_from_sim no)
-		(in_bom yes)
-		(on_board yes)
-		(in_pos_files yes)
-		(dnp no)
-		(fields_autoplaced yes)
-		(property "Reference" "J11"
-			(at 768.35 549.9099 0)
-			(show_name no)
-			(do_not_autoplace no)
-			(effects
-				(font
-					(size 1.27 1.27)
-				)
-				(justify right)
-			)
-		)
-		(property "Value" "Conn_01x05_Pin"
-			(at 768.35 552.4499 0)
-			(show_name no)
-			(do_not_autoplace no)
-			(effects
-				(font
-					(size 1.27 1.27)
-				)
-				(justify right)
-			)
-		)
-		(property "Footprint" "Connector_PinHeader_2.54mm:PinHeader_1x05_P2.54mm_Vertical"
-			(at 767.08 551.18 0)
-			(hide yes)
-			(show_name no)
-			(do_not_autoplace no)
-			(effects
-				(font
-					(size 1.27 1.27)
-				)
-			)
-		)
-		(property "Datasheet" ""
-			(at 767.08 551.18 0)
-			(hide yes)
-			(show_name no)
-			(do_not_autoplace no)
-			(effects
-				(font
-					(size 1.27 1.27)
-				)
-			)
-		)
-		(property "Description" "Generic connector, single row, 01x05, script generated"
-			(at 767.08 551.18 0)
-			(hide yes)
-			(show_name no)
-			(do_not_autoplace no)
-			(effects
-				(font
-					(size 1.27 1.27)
-				)
-			)
-		)
-		(property "LCSC" ""
-			(at 767.08 551.18 0)
-			(hide yes)
-			(show_name no)
-			(do_not_autoplace no)
-			(effects
-				(font
-					(size 1.27 1.27)
-				)
-			)
-		)
-		(pin "2"
-		)
-		(pin "1"
-		)
-		(pin "5"
-		)
-		(pin "4"
-		)
-		(pin "3"
-		)
-		(instances
-			(project "roam_edge_xl"
-				(path "/e63e39d7-6ac0-4ffd-8aa3-1841a4541b55"
-					(reference "J11")
-					(unit 1)
-				)
-			)
-		)
-	)
-	(symbol
 		(lib_id "TC-RF-Module:LC760Z")
 		(at 1005.84 445.77 0)
@@
 			)
 		)
-		(property "Footprint" "LIS2DH12TR:PQFN50P200X200100-12N"
+		(property "Footprint" "MotionSensor:LIS12DH"
 			(at 276.86 297.18 0)
 			(hide yes)
